File: hardware/kicad/cryocooler.kicad_sch (KiCad schematic)
At the start: 16 parts, among them J1 USB_C, SW1 RESET, SW2 BOOT, U1 ESP32-S3-WROOM-2-N32R16V, U2 USBLC6-2SC6

Commit message: KiCad: cleaner layout, decoupling blocks, label directions, KiCad format fixes
- move IC decoupling caps into labelled blocks at the side of each sheet
- global labels show input/output direction per net
- no 4-way junctions (generator now checks and fails)
- generator output matches KiCad's saved format (hide property, junction
  and wire normalisation, lib symbol embedded fonts, multi-unit pins)
- hand-laid USB ESD protection as a pass-through

Co-Authored-By: Claude Sonnet 5.5 <noreply@anthropic.com>
Other:
- note added: "ESP32-S3 DECOUPLING CAPACITORS"
