File: hardware/kicad/cryocooler.kicad_sch (KiCad schematic)
At the start: 14 parts, among them J1 USB_C, SW1 RESET, SW2 BOOT, U1 ESP32-S3-WROOM-2-N32R16V, U2 USBLC6-2SC6

Commit message: WIP: restructure PCB for the Phoenix UCS 125-87 housing
Work in progress, layout not finished: about 90 parts still do not fit
their sections and the board is not routed.

- Right-angle connectors: Phoenix MSTBA 2,5 / MC 1,5, JST XH side entry,
  Hirose DF13, Molex 505448-0871 (new footprint from the Molex drawing)
- Datasheet and product links on every symbol (tools/part_links.py)
- Test points so every IC has one on its own nets
- gen_pcb.py: 100 x 62 mm two-sided board, housing holes and restricted
  corners, ESP32 antenna notch, one section per sheet, board ID block,
  ESP32 pin names, pin-1 marks, blue mask
- Housing drawings in hardware/housing/

Co-Authored-By: Claude Opus 5.5 <noreply@anthropic.com>
Parts:
- added C5: 4.7uF, Capacitor_SMD:C_0805_2012Metric, symbol Device:C
- C1: Product (none) -> https://www.digikey.com/en/products/result?keywords=CL21A10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
- C2, C4: Product (none) -> https://www.digikey.com/en/products/result?keywords=C0603C1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
- C3: Product (none) -> https://www.digikey.com/en/products/result?keywords=08055C1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
- J1: Product (none) -> https://www.digikey.com/en/products/result?keywords=USB4105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
- R1, R2: Product (none) -> https://www.digikey.com/en/products/result?keywords=AR0603F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
- R3, R4: Product (none) -> https://www.digikey.com/en/products/result?keywords=CR0603-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
- SW1, SW2: Product (none) -> https://www.digikey.com/en/products/result?keywords=TL3342F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
- TP1: renamed from C5; value 4.7uF -> USB_VBUS; footprint Capacitor_SMD:C_0805_2012Metric -> TestPoint:TestPoint_Pad_D1.5mm; symbol Device:C -> Connector:TestPoint
- U1: Product (none) -> https://www.digikey.com/en/products/result?keywords=ESP32-S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
- U2: Product (none) -> https://www.digikey.com/en/products/result?keywords=USBLC6-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
Connections:
- net GND: now also C5.2; no longer TP1.2
- net USB_VBUS: now also C5.1

Commit message: Lay out the board for the Phoenix UCS 145-125 housing
Move to a 120 x 100 mm, 4-layer, blue-mask board for the UCS 145-125-F-CCD
7035 housing: housing mounting holes and restricted corners, ESP32 antenna
over a routed notch, one labelled section per schematic sheet with almost
every part on top. Placed, routed and cleaned up: DRC 0 errors, 0
unconnected, 0 schematic-parity issues; ERC 0; 193/193 datasheet rules.

- AGENTS.md: test points go on the same side as the part they test, close
  to it
- gen_pcb: test points held to their IC's side and within 8 mm; silkscreen
  check measures text by ink and also fails on pads, part outlines, section
  lines and pin-1 dots; titles along or up a border; connector labels and
  ESP32 pin names reserved before the passives; pin-1 dots only where the
  footprint has no mark; footprints carry the schematic's library links and
  fields; mounting holes are board-only H1-H4
- fix_route: generic clean-up (no old-board coordinate edits); removes GND
  vias in keep-outs or on foreign pads, links stranded ground pads, nudges
  squeezed tracks, handles back-side pour islands
- kicad_dru: fix the rule file (an invalid USB-C rule made KiCad ignore it);
  housing-corner and antenna keep-out part rules
- schematic: pad test points excluded from the BOM
- README / fabrication README updated for the new board

Co-Authored-By: Claude Opus 5.5 <noreply@anthropic.com>
Parts:
- TP1: now left out of the parts list
Changed lines of the file:
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@@
 		(body_style 1)
 		(exclude_from_sim no)
-		(in_bom yes)
+		(in_bom no)
 		(on_board yes)
 		(in_pos_files yes)
