File: hardware/kicad/cryocooler.kicad_pcb (KiCad board)
At the start: 4 copper layers, 130 x 110 mm, 322 parts, among them J1 USB_C, J10 RTD PT1000 4-wire, J11 AMP OUT (+ / -), J12 CRYOCOOLER (+ / -), J13 COMPRESSOR RELAY / GND, J14 IMU LSM6DSOX module, J2 12V IN, J3 FAN (4-pin PWM), J4 PUMP (4-pin PWM), J5 ALPHACOOL ES FLOW (3-pin), J6 ALPHACOOL ES NTC 10k, J7 PANEL BUTTON, J8 AMP REM / GND, J9 AMP SIGNAL IN / GND, Q1 IRF4905S, Q10 BSS138, Q11 BSS138, Q12 BSS138, Q2 BSS138, Q3 BSS138, Q4 BSS138, Q5 BSS138, Q6 BSS84, Q7 BSS138, Q8 BSS84, Q9 BSS138, SW1 RESET, SW2 BOOT, SW3 POWER, U1 ESP32-S3-WROOM-2-N32R16V, U10 EMC2303-x-KP, U11 LTC2954CTS8-2, U12 LM4040DBZ-5, U13 CL25N8-G, U14 ADS1220IPW, U15 AP63205WU-7, U16 LD1117S33TR, U17 ISO7741DW, U18 ACS37800KMACTR-030B3-SPI, U2 USBLC6-2SC6, U20 ADP5071AREZ, U21 LT3097ADJC, U23 INA239AIDGSR, U24 74AHCT1G125, U25 SC18IS604PW, U26 74LVC1G125, U3 SG-8002CA-PH 25MHz, U4 AD9833BRMZ, U5 OPA1656ID, U6 AD633JRZ-R7, U7 MCP4921-E/SN, U8 LM4040DBZ-2.5, U9 OPA188ID

Commit message: Adding updated board
Other:
- board text added: "ACS37800"
- board text added: "AD633 JRZ-R7"
- board text added: "ADS 1220IPW"
- board text added: "ISO7741DW"
- board text added: "LD1117 S33TR"
- board text added: "MCP 4921"
- board text added: "OPA 1656ID"
- board text added: "OPA 188ID"
- board text added: "SC18IS 604PW"
- board text added: "SG- 8002CA"
Changed lines of the file:
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@@
 		(layer "Edge.Cuts")
+	)
+	(gr_text "AD633\nJRZ-R7"
+		(at 24 9 90)
+		(layer "F.SilkS")
+		(effects
+			(font
+				(size 0.7 0.7)
+				(thickness 0.12)
+			)
+		)
+	)
+	(gr_text "OPA\n1656ID"
+		(at 36 8 90)
+		(layer "F.SilkS")
+		(effects
+			(font
+				(size 0.7 0.7)
+				(thickness 0.12)
+			)
+		)
+	)
+	(gr_text "OPA\n188ID"
+		(at 36 22.5 90)
+		(layer "F.SilkS")
+		(effects
+			(font
+				(size 0.7 0.7)
+				(thickness 0.12)
+			)
+		)
+	)
+	(gr_text "MCP\n4921"
+		(at 47 22.5 90)
+		(layer "F.SilkS")
+		(effects
+			(font
+				(size 0.7 0.7)
+				(thickness 0.12)
+			)
+		)
+	)
+	(gr_text "ADS\n1220IPW"
+		(at 113 84 90)
+		(layer "F.SilkS")
+		(effects
+			(font
+				(size 0.7 0.7)
+				(thickness 0.12)
+			)
+		)
 	)
 	(gr_text "+"
@@
 		)
 	)
+	(gr_text "SG-\n8002CA"
+		(at 59 8 90)
+		(layer "F.SilkS")
+		(effects
+			(font
+				(size 0.8 0.8)
+				(thickness 0.12)
+			)
+		)
+	)
 	(gr_text "FAULT"
 		(at 81 15.925 90)
@@
 		)
 	)
+	(gr_text "SC18IS\n604PW"
+		(at 101 67.5 90)
+		(layer "F.SilkS")
+		(effects
+			(font
+				(size 0.8 0.8)
+				(thickness 0.12)
+			)
+		)
+	)
 	(gr_text "PWM"
 		(at 102.42 101.055 90)
@@
 				(thickness 0.12)
 			)
+		)
+	)
+	(gr_text "ACS37800"
+		(at 26 49 90)
+		(layer "F.SilkS")
+		(effects
+			(font
+				(size 0.9 0.9)
+				(thickness 0.12)
+			)
+		)
+	)
+	(gr_text "ISO7741DW"
+		(at 40 44.5 90)
+		(layer "F.SilkS")
+		(effects
+			(font
+				(size 0.9 0.9)
+				(thickness 0.12)
+			)
+		)
+	)
+	(gr_text "LD1117\nS33TR"
+		(at 79 83 90)
+		(layer "F.SilkS")
+		(effects
+			(font
+				(size 0.9 0.9)
+				(thickness 0.12)
+			)
