File: hardware/kicad/sheets/amp_current.kicad_sch (KiCad schematic)
At the start: 22 parts, among them J6 AMP OUT (+ / -), J7 CRYOCOOLER (+ / -), U18 ISO7741DW, U19 ACS37800KMACTR-030B3-SPI

Commit message: KiCad: cleaner layout, decoupling blocks, label directions, KiCad format fixes
- move IC decoupling caps into labelled blocks at the side of each sheet
- global labels show input/output direction per net
- no 4-way junctions (generator now checks and fails)
- generator output matches KiCad's saved format (hide property, junction
  and wire normalisation, lib symbol embedded fonts, multi-unit pins)
- hand-laid USB ESD protection as a pass-through

Co-Authored-By: Claude Sonnet 5.5 <noreply@anthropic.com>
Parts:
- C48: value 100nF -> 10uF; footprint Capacitor_SMD:C_0603_1608Metric -> Capacitor_SMD:C_0805_2012Metric
- C50: value 10uF -> 22uF; footprint Capacitor_SMD:C_0805_2012Metric -> Capacitor_SMD:C_1206_3216Metric
- C52: value 22uF -> 100nF; footprint Capacitor_SMD:C_1206_3216Metric -> Capacitor_SMD:C_0603_1608Metric
Connections:
- net +3V3: now also C52.1; no longer C48.1
- net +5V: now also C48.1, C49.1; no longer C50.1, C51.1
- net GND: now also C49.2, C52.2; no longer C50.2, C51.2
- net ISO_3V3: now also C50.1, C51.1; no longer C49.1, C52.1
- net ISO_GND: now also C50.2, C51.2; no longer C49.2, C52.2
Other:
- note added: "ACS37800 DECOUPLING CAPACITORS"
- note added: "ISO7741 VCC1 DECOUPLING CAPACITORS"
- note added: "ISO7741 VCC2 DECOUPLING CAPACITORS"
