File: hardware/kicad/sheets/amp_current.kicad_sch (KiCad schematic)
At the start: 22 parts, among them J6 AMP OUT (+ / -), J7 CRYOCOOLER (+ / -), U18 ISO7741DW, U19 ACS37800KMACTR-030B3-SPI

Commit message: Fixing the UUID issues
Parts:
- removed C48: 10uF, Capacitor_SMD:C_0805_2012Metric, symbol Device:C
- removed C53: 100nF, Capacitor_SMD:C_0603_1608Metric, symbol Device:C
- removed J7: CRYOCOOLER (+ / -), TerminalBlock_Phoenix:TerminalBlock_Phoenix_MKDS-1,5-2-5.08_1x02_P5.08mm_Horizontal, symbol Connector:Screw_Terminal_01x02
- removed R41, R42, R43: 10k, Resistor_SMD:R_0603_1608Metric, symbol Device:R_US
- removed R44: 100k, Resistor_SMD:R_0603_1608Metric, symbol Device:R_US
- removed R46: 1M, Resistor_SMD:R_1206_3216Metric, symbol Device:R_US
- removed U18: ISO7741DW, Package_SO:SOIC-16W_7.5x10.3mm_P1.27mm, symbol cryocooler:ISO7741DW
- added C46: 100nF, Capacitor_SMD:C_0603_1608Metric, symbol Device:C
- added J11: AMP OUT (+ / -), TerminalBlock_Phoenix:TerminalBlock_Phoenix_MKDS-1,5-2-5.08_1x02_P5.08mm_Horizontal, symbol Connector:Screw_Terminal_01x02
- added J12: CRYOCOOLER (+ / -), TerminalBlock_Phoenix:TerminalBlock_Phoenix_MKDS-1,5-2-5.08_1x02_P5.08mm_Horizontal, symbol Connector:Screw_Terminal_01x02
- added R48: 10k, Resistor_SMD:R_0603_1608Metric, symbol Device:R_US
- added R51: 4.02k, Resistor_SMD:R_0603_1608Metric, symbol Device:R_US
- added R52, R53: 1M, Resistor_SMD:R_1206_3216Metric, symbol Device:R_US
- added U17: ISO7741DW, Package_SO:SOIC-16W_7.5x10.3mm_P1.27mm, symbol cryocooler:ISO7741DW
- added U18: ACS37800KMACTR-030B3-SPI, Package_SO:SOIC-16W_7.5x10.3mm_P1.27mm, symbol cryocooler:ACS37800KMACTR-030B3-SPI
- C45: renamed from U19; value ACS37800KMACTR-030B3-SPI -> 10uF; footprint Package_SO:SOIC-16W_7.5x10.3mm_P1.27mm -> Capacitor_SMD:C_0805_2012Metric; symbol cryocooler:ACS37800KMACTR-030B3-SPI -> Device:C
- C47: renamed from R48; value 1M -> 22uF; footprint Resistor_SMD:R_1206_3216Metric -> Capacitor_SMD:C_1206_3216Metric; symbol Device:R_US -> Device:C
- C48: renamed from J6; value AMP OUT (+ / -) -> 100nF; footprint TerminalBlock_Phoenix:TerminalBlock_Phoenix_MKDS-1,5-2-5.08_1x02_P5.08mm_Horizontal -> Capacitor_SMD:C_0603_1608Metric; symbol Connector:Screw_Terminal_01x02 -> Device:C
- C50: value 22uF -> 100nF; footprint Capacitor_SMD:C_1206_3216Metric -> Capacitor_SMD:C_0603_1608Metric
- C51: value 100nF -> 1uF; footprint Capacitor_SMD:C_0603_1608Metric -> Capacitor_SMD:C_0805_2012Metric
- R47, R49: value 1M -> 10k; footprint Resistor_SMD:R_1206_3216Metric -> Resistor_SMD:R_0603_1608Metric
- R50: renamed from R45; value 4.02k -> 100k
- R54: renamed from C54; value 1uF -> 1M; footprint Capacitor_SMD:C_0805_2012Metric -> Resistor_SMD:R_1206_3216Metric; symbol Device:C -> Device:R_US
- R55: renamed from C55; value 100nF -> 1M; footprint Capacitor_SMD:C_0603_1608Metric -> Resistor_SMD:R_1206_3216Metric; symbol Device:C -> Device:R_US
Connections:
- net +3V3: now also C49.1, R47.1, R49.1, R48.1, U17.1 (VCC1), U17.7 (EN1); no longer C52.1
- net +5V: now also C45.1, R50.1, C46.1; no longer C49.1
- net ACS_CS: now also R47.2, U17.5 (INC)
- net ACS_MISO: now also U17.6 (OUTD)
- net ACS_MOSI: now also R49.2, U17.3 (INA)
- net ACS_SCK: now also R48.2, U17.4 (INB)
- net GND: now also C45.2, C46.2, U17.2 (GND1), U17.8 (GND1); no longer C52.2
- net ISO_3V3: now also C47.1, C48.1, C52.1, U17.10 (EN2), U17.16 (VCC2), U18.13 (VCC); no longer C45.13 (VCC), R54.1, R55.1
- net ISO_CS: now also U17.12 (OUTC), U18.9 (~{CS}); no longer C45.9 (~{CS})
- net ISO_GND: now also C47.2, C52.2, J11.2 (Pin_2), J12.2 (Pin_2), R51.2, U17.15 (GND2), U17.9 (GND2), U18.14 (GND), U18.15 (VINN); no longer C45.14 (GND), C45.15 (VINN), R50.2, R54.2, R55.2
- net ISO_MISO: now also U17.11 (IND), U18.12 (MISO); no longer C45.12 (MISO)
- net ISO_MOSI: now also U17.14 (OUTA), U18.10 (MOSI); no longer C45.10 (MOSI)
- net ISO_SCK: now also U17.13 (OUTB), U18.11 (SCLK); no longer C45.11 (SCLK)
- net at PS1.8 (EN): now also R50.2
- new net: R51.1, R52.1, U18.16 (VINP)
- new net: R52.2, R53.1
- new net: R54.2, R55.1
- new net: J12.1 (Pin_1), R55.2, U18.5 (IP-), U18.6 (IP-), U18.7 (IP-), U18.8 (IP-)
- new net: R53.2, R54.1
- new net: J11.1 (Pin_1), U18.1 (IP+), U18.2 (IP+), U18.3 (IP+), U18.4 (IP+)
Other:
- moved on the sheet: R50
