File: hardware/kicad/sheets/amp_current.kicad_sch (KiCad schematic)
At the start: 22 parts, among them J11 AMP OUT (+ / -), J12 CRYOCOOLER (+ / -), U17 ISO7741DW, U18 ACS37800KMACTR-030B3-SPI

Commit message: Replace the ±15 V LDOs with one LT3097 and add a power-good interlock
- rails_15v: ADP7142 + ADP7182 replaced by one LT3097 (±14.7 V, 147 k SET
  resistors); the ADP5071 output caps are now 22 uF / 50 V and double as the
  LT3097 inputs. PGP / PGN make the PG_15V node (fed from +15 V, so it reads
  0 V if a rail is missing).
- amp_control: a series BSS138 (Q9) gated by PG_15V blocks AMP_REM unless
  both rails are good. New power_good sheet: LED (D23) and the active-low
  PG_15V_N flag on GPIO43 (PG_15V_N_PIN).
- Tooling: LT3097 symbol, footprint and 3D envelope; datasheet rules (191),
  GPIO check, BOM tables, floor plan, PAD_BRIDGES and pre-placed GND vias in
  gen_pcb.py, new fix_route.py for post-route clean-up.
- Board regenerated and routed with Freerouting 2.5.0: DRC 0 unconnected,
  0 schematic-parity issues, no copper violations. Gerbers, JLCPCB zip,
  renders, BOM, CPL and schematic PDF regenerated.

Co-Authored-By: Claude Sonnet 5.5 <noreply@anthropic.com>
Parts:
- removed C51: 1uF, Capacitor_SMD:C_0805_2012Metric, symbol Device:C
- removed R47: 10k, Resistor_SMD:R_0603_1608Metric, symbol Device:R_US
- removed R50: 1M, Resistor_SMD:R_1206_3216Metric, symbol Device:R_US
- added C52: 100nF, Capacitor_SMD:C_0603_1608Metric, symbol Device:C
- added J12: CRYOCOOLER (+ / -), TerminalBlock_Phoenix:TerminalBlock_Phoenix_MKDS-1,5-2-5.08_1x02_P5.08mm_Horizontal, symbol Connector:Screw_Terminal_01x02
- added PS1: MIE1W0505BGLVH-3R-Z, cryocooler:CONV_MIE1W0505BGLVH-3R-Z, symbol cryocooler:MIE1W0505BGLVH-3R-Z
- C51: renamed from C52; value 100nF -> 1uF; footprint Capacitor_SMD:C_0603_1608Metric -> Capacitor_SMD:C_0805_2012Metric
- J11: renamed from J12; value CRYOCOOLER (+ / -) -> AMP OUT (+ / -)
- R47: renamed from PS1; value MIE1W0505BGLVH-3R-Z -> 10k; footprint cryocooler:CONV_MIE1W0505BGLVH-3R-Z -> Resistor_SMD:R_0603_1608Metric; symbol cryocooler:MIE1W0505BGLVH-3R-Z -> Device:R_US
- R53: renamed from J11; value AMP OUT (+ / -) -> 1M; footprint TerminalBlock_Phoenix:TerminalBlock_Phoenix_MKDS-1,5-2-5.08_1x02_P5.08mm_Horizontal -> Resistor_SMD:R_1206_3216Metric; symbol Connector:Screw_Terminal_01x02 -> Device:R_US
- renumbered R51 to R50, R52 to R51, R53 to R52
Connections:
- net +3V3: now also R47.1
- net +5V_ISO: now also PS1.9_10 (VIN); no longer R47.9_10 (VIN)
- net ACS_MOSI: now also R47.2
- net GND: now also PS1.1 (GND1), PS1.11_12 (GND1); no longer R47.1 (GND1), R47.11_12 (GND1)
- net ISO_3V3: now also C52.1, PS1.5_6 (VOUT); no longer R47.5_6 (VOUT)
- net ISO_GND: now also C52.2, J12.2 (Pin_2), PS1.2 (GND2), PS1.3_4 (GND2), PS1.7 (VSEL); no longer R47.2 (GND2), R47.3_4 (GND2), R47.7 (VSEL), R53.2 (Pin_2)
- net at U18.1 (IP+), U18.2 (IP+), U18.3 (IP+)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: now also J11.1 (Pin_1); no longer R53.1 (Pin_1)
- net at R49.1, U18.16 (VINP): now also R50.1
- net at U18.5 (IP-), U18.6 (IP-), U18.7 (IP-)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: now also R53.2, J12.1 (Pin_1); no longer J11.1 (Pin_1), R52.2
- net at R48.2: now also PS1.8 (EN); no longer R47.8 (EN)
- new net: R52.2, R53.1
Other:
- moved on the sheet: C51, J11, R50, R51, R52
