File: hardware/kicad/sheets/amp_current.kicad_sch (KiCad schematic)
At the start: 22 parts, among them J11 AMP OUT (+ / -), J12 CRYOCOOLER (+ / -), U17 ISO7741DW, U18 ACS37800KMACTR-030B3-SPI

Commit message: WIP: restructure PCB for the Phoenix UCS 125-87 housing
Work in progress, layout not finished: about 90 parts still do not fit
their sections and the board is not routed.

- Right-angle connectors: Phoenix MSTBA 2,5 / MC 1,5, JST XH side entry,
  Hirose DF13, Molex 505448-0871 (new footprint from the Molex drawing)
- Datasheet and product links on every symbol (tools/part_links.py)
- Test points so every IC has one on its own nets
- gen_pcb.py: 100 x 62 mm two-sided board, housing holes and restricted
  corners, ESP32 antenna notch, one section per sheet, board ID block,
  ESP32 pin names, pin-1 marks, blue mask
- Housing drawings in hardware/housing/

Co-Authored-By: Claude Opus 5.5 <noreply@anthropic.com>
Parts:
- removed C49: 100nF, Capacitor_SMD:C_0603_1608Metric, symbol Device:C
- removed R46, R47: 10k, Resistor_SMD:R_0603_1608Metric, symbol Device:R_US
- removed R49: 4.02k, Resistor_SMD:R_0603_1608Metric, symbol Device:R_US
- removed R50, R52: 1M, Resistor_SMD:R_1206_3216Metric, symbol Device:R_US
- added C45: 10uF, Capacitor_SMD:C_0805_2012Metric, symbol Device:C
- added C51: 1uF, Capacitor_SMD:C_0805_2012Metric, symbol Device:C
- added J11: AMP OUT (+ / -), Connector_Phoenix_MSTB:PhoenixContact_MSTBA_2,5_2-G-5,08_1x02_P5.08mm_Horizontal, symbol Connector:Screw_Terminal_01x02
- added J12: CRYOCOOLER (+ / -), Connector_Phoenix_MSTB:PhoenixContact_MSTBA_2,5_2-G-5,08_1x02_P5.08mm_Horizontal, symbol Connector:Screw_Terminal_01x02
- added PS1: MIE1W0505BGLVH-3R-Z, cryocooler:CONV_MIE1W0505BGLVH-3R-Z, symbol cryocooler:MIE1W0505BGLVH-3R-Z
- added R53: 1M, Resistor_SMD:R_1206_3216Metric, symbol Device:R_US
- C46, C48, C52: Product (none) -> https://www.digikey.com/en/products/result?keywords=C0603C1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
- C47: Product (none) -> https://www.digikey.com/en/products/result?keywords=CL31A22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
- C49: renamed from C50; Product (none) -> https://www.digikey.com/en/products/result?keywords=C0603C1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
- C50: renamed from C51; value 1uF -> 100nF; footprint Capacitor_SMD:C_0805_2012Metric -> Capacitor_SMD:C_0603_1608Metric; Product (none) -> https://www.digikey.com/en/products/result?keywords=C0603C1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
- R45, R48: Product (none) -> https://www.digikey.com/en/products/result?keywords=AR0603F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
- R46: renamed from PS1; value MIE1W0505BGLVH-3R-Z -> 10k; footprint cryocooler:CONV_MIE1W0505BGLVH-3R-Z -> Resistor_SMD:R_0603_1608Metric; symbol cryocooler:MIE1W0505BGLVH-3R-Z -> Device:R_US; Product (none) -> https://www.digikey.com/en/products/result?keywords=AR0603F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
- R47: renamed from C45; value 10uF -> 10k; footprint Capacitor_SMD:C_0805_2012Metric -> Resistor_SMD:R_0603_1608Metric; symbol Device:C -> Device:R_US; Product (none) -> https://www.digikey.com/en/products/result?keywords=AR0603F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
- R49: renamed from R51; value 1M -> 4.02k; footprint Resistor_SMD:R_1206_3216Metric -> Resistor_SMD:R_0603_1608Metric; Product (none) -> https://www.digikey.com/en/products/result?keywords=RC0603F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
- R50: renamed from R53; Product (none) -> https://www.digikey.com/en/products/result?keywords=RC1206F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
- R51: renamed from J11; value AMP OUT (+ / -) -> 1M; footprint TerminalBlock_Phoenix:TerminalBlock_Phoenix_MKDS-1,5-2-5.08_1x02_P5.08mm_Horizontal -> Resistor_SMD:R_1206_3216Metric; symbol Connector:Screw_Terminal_01x02 -> Device:R_US; Product (none) -> https://www.digikey.com/en/products/result?keywords=RC1206F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
- R52: renamed from J12; value CRYOCOOLER (+ / -) -> 1M; footprint TerminalBlock_Phoenix:TerminalBlock_Phoenix_MKDS-1,5-2-5.08_1x02_P5.08mm_Horizontal -> Resistor_SMD:R_1206_3216Metric; symbol Connector:Screw_Terminal_01x02 -> Device:R_US; Product (none) -> https://www.digikey.com/en/products/result?keywords=RC1206F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
- U17: Product (none) -> https://www.digikey.com/en/products/result?keywords=ISO7741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
- U18: Product (none) -> https://www.digikey.com/en/products/result?keywords=ACS3780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
Connections:
- net +3V3: now also C49.1, R46.1, R47.1
- net +5V_ISO: now also C45.1, PS1.9_10 (VIN); no longer R46.9_10 (VIN), R47.1
- net ACS_MOSI: now also R47.2
- net ACS_SCK: now also R46.2
- net GND: now also C49.2, C45.2, PS1.1 (GND1), PS1.11_12 (GND1); no longer R46.1 (GND1), R46.11_12 (GND1), R47.2
- net ISO_3V3: now also C51.1, PS1.5_6 (VOUT); no longer C49.1, R46.5_6 (VOUT)
- net ISO_GND: now also R49.2, C51.2, J11.2 (Pin_2), J12.2 (Pin_2), PS1.2 (GND2), PS1.3_4 (GND2), PS1.7 (VSEL); no longer C49.2, R46.2 (GND2), R46.3_4 (GND2), R46.7 (VSEL), R51.2 (Pin_2), R52.2 (Pin_2)
- net at U18.5 (IP-), U18.6 (IP-), U18.7 (IP-)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: now also J12.1 (Pin_1), R53.2; no longer R50.2, R52.1 (Pin_1)
- net at R48.2: now also PS1.8 (EN); no longer R46.8 (EN)
- net at R50.1: now also R49.1, U18.16 (VINP)
- net at U18.1 (IP+), U18.2 (IP+), U18.3 (IP+)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: now also J11.1 (Pin_1); no longer R51.1 (Pin_1)
- new net: R51.2, R52.1
- new net: R52.2, R53.1
- new net: R50.2, R51.1
Other:
- moved on the sheet: C49, C50, R49, R50

Commit message: Ground the M12 shield, order the ground loops, name the J14 cable parts
- J10: shielded symbol (Conn_01x04_Shielded); the M12 shield pin and its
  four shell legs are pad SH, tied to GND
- TP22-TP25: Keystone 5001 black miniature PC test points (KiCad
  TestPoint_Keystone_5000-5004 footprint, 1.02 mm hole per Keystone's
  drawing); now in the BOM, the bare pad test points stay out
- J14 BOM note: cable housing Molex 5054320801 with 505431 terminals, or
  tin pre-crimped leads 797581148 / 797581149 (from molex.com)

Only netlist change: GND gains J10 SH. DRC 0 errors, 0 unconnected, 0
schematic-parity issues; ERC 0; 193/193 datasheet rules.

Co-Authored-By: Claude Opus 5.5 <noreply@anthropic.com>
Parts:
- removed C51: 1uF, Capacitor_SMD:C_0805_2012Metric, symbol Device:C
- removed R47: 10k, Resistor_SMD:R_0603_1608Metric, symbol Device:R_US
- removed R50: 1M, Resistor_SMD:R_1206_3216Metric, symbol Device:R_US
- added C52: 100nF, Capacitor_SMD:C_0603_1608Metric, symbol Device:C
- added J12: CRYOCOOLER (+ / -), Connector_Phoenix_MSTB:PhoenixContact_MSTBA_2,5_2-G-5,08_1x02_P5.08mm_Horizontal, symbol Connector:Screw_Terminal_01x02
- added PS1: MIE1W0505BGLVH-3R-Z, cryocooler:CONV_MIE1W0505BGLVH-3R-Z, symbol cryocooler:MIE1W0505BGLVH-3R-Z
- C51: renamed from C52; value 100nF -> 1uF; footprint Capacitor_SMD:C_0603_1608Metric -> Capacitor_SMD:C_0805_2012Metric; Product https://www.digikey.com/en/products/result?keywords=C0603C1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 -> https://www.digikey.com/en/products/result?keywords=08055C1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
- J11: renamed from J12; value CRYOCOOLER (+ / -) -> AMP OUT (+ / -)
- R47: renamed from PS1; value MIE1W0505BGLVH-3R-Z -> 10k; footprint cryocooler:CONV_MIE1W0505BGLVH-3R-Z -> Resistor_SMD:R_0603_1608Metric; symbol cryocooler:MIE1W0505BGLVH-3R-Z -> Device:R_US; Product https://www.digikey.com/en/products/result?keywords=MIE1W05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 -> https://www.digikey.com/en/products/result?keywords=AR0603F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
- R53: renamed from J11; value AMP OUT (+ / -) -> 1M; footprint Connector_Phoenix_MSTB:PhoenixContact_MSTBA_2,5_2-G-5,08_1x02_P5.08mm_Horizontal -> Resistor_SMD:R_1206_3216Metric; symbol Connector:Screw_Terminal_01x02 -> Device:R_US; Product https://www.phoenixcontact.com/en-us/products/pcb-header-ms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 -> https://www.digikey.com/en/products/result?keywords=RC1206F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
- renumbered R51 to R50, R52 to R51, R53 to R52
Connections:
- net +3V3: now also R47.1
- net +5V_ISO: now also PS1.9_10 (VIN); no longer R47.9_10 (VIN)
- net ACS_MOSI: now also R47.2
- net GND: now also PS1.1 (GND1), PS1.11_12 (GND1); no longer R47.1 (GND1), R47.11_12 (GND1)
- net ISO_3V3: now also C52.1, PS1.5_6 (VOUT); no longer R47.5_6 (VOUT)
- net ISO_GND: now also C52.2, J12.2 (Pin_2), PS1.2 (GND2), PS1.3_4 (GND2), PS1.7 (VSEL); no longer R47.2 (GND2), R47.3_4 (GND2), R47.7 (VSEL), R53.2 (Pin_2)
- net at U18.1 (IP+), U18.2 (IP+), U18.3 (IP+)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: now also J11.1 (Pin_1); no longer R53.1 (Pin_1)
- net at R49.1, U18.16 (VINP): now also R50.1
- net at U18.5 (IP-), U18.6 (IP-), U18.7 (IP-)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: now also R53.2, J12.1 (Pin_1); no longer J11.1 (Pin_1), R52.2
- net at R48.2: now also PS1.8 (EN); no longer R47.8 (EN)
- new net: R52.2, R53.1
Other:
- moved on the sheet: C51, J11, R50, R51, R52
