File: hardware/kicad/sheets/cooling.kicad_sch (KiCad schematic)
At the start: 22 parts, among them J10 ALPHACOOL ES FLOW (3-pin), J11 ALPHACOOL ES NTC 10k, J8 FAN (4-pin PWM), J9 PUMP (4-pin PWM), U21 EMC2303-x-KP

Commit message: KiCad: cleaner layout, decoupling blocks, label directions, KiCad format fixes
- move IC decoupling caps into labelled blocks at the side of each sheet
- global labels show input/output direction per net
- no 4-way junctions (generator now checks and fails)
- generator output matches KiCad's saved format (hide property, junction
  and wire normalisation, lib symbol embedded fonts, multi-unit pins)
- hand-laid USB ESD protection as a pass-through

Co-Authored-By: Claude Sonnet 5.5 <noreply@anthropic.com>
Other:
- note added: "EMC2303 DECOUPLING CAPACITORS"
