File: hardware/kicad/sheets/cooling.kicad_sch (KiCad schematic)
At the start: 22 parts, among them J3 FAN (4-pin PWM), J4 PUMP (4-pin PWM), J5 ALPHACOOL ES FLOW (3-pin), J6 ALPHACOOL ES NTC 10k, U10 EMC2303-x-KP

Commit message: Split cooling into Water Cooling and Cold Head Temp sections, each with a supply jumper and LED
Water Cooling (EMC2303, SC18IS604 bridge, NTC, fan/pump/flow) sits behind JP4
on +3V3_COOL together with its pull-ups. Cold Head Temp (ADS1220, PT1000) gets
a new jumper JP5 and LED D22 on +3V3_CH. JP2 is relabelled for the +-15V rails
and moved into the RAILS +-15V box. PCB regenerated with two silk boxes, routed,
leftovers finished with a grid router; board render added to the main README.

Co-Authored-By: Claude Sonnet 5.5 <noreply@anthropic.com>
Connections:
- net +3V3 is gone; now on net +3V3_COOL: R14.1, R15.1, R16.1, R17.1, R18.1, R19.1, R20.1, R21.1, R23.1, R24.1
Other:
- title: Cooling -> Water Cooling

Commit message: WIP: restructure PCB for the Phoenix UCS 125-87 housing
Work in progress, layout not finished: about 90 parts still do not fit
their sections and the board is not routed.

- Right-angle connectors: Phoenix MSTBA 2,5 / MC 1,5, JST XH side entry,
  Hirose DF13, Molex 505448-0871 (new footprint from the Molex drawing)
- Datasheet and product links on every symbol (tools/part_links.py)
- Test points so every IC has one on its own nets
- gen_pcb.py: 100 x 62 mm two-sided board, housing holes and restricted
  corners, ESP32 antenna notch, one section per sheet, board ID block,
  ESP32 pin names, pin-1 marks, blue mask
- Housing drawings in hardware/housing/

Co-Authored-By: Claude Opus 5.5 <noreply@anthropic.com>
Parts:
- removed C25: 100nF, Capacitor_SMD:C_0603_1608Metric, symbol Device:C
- removed J5: ALPHACOOL ES FLOW (3-pin), Connector_Molex:Molex_KK-254_AE-6410-03A_1x03_P2.54mm_Vertical, symbol Connector_Generic:Conn_01x03
- removed R17: 1k, Resistor_SMD:R_0603_1608Metric, symbol Device:R_US
- removed R18, R20, R24: 10k, Resistor_SMD:R_0603_1608Metric, symbol Device:R_US
- added C28: 100nF, Capacitor_SMD:C_0603_1608Metric, symbol Device:C
- added D2: FAN FAULT, LED_SMD:LED_0603_1608Metric, symbol Device:LED
- added J3: FAN (4-pin PWM), Connector_JST:JST_XH_S4B-XH-A_1x04_P2.50mm_Horizontal, symbol Connector_Generic:Conn_01x04
- added R19, R21: 4.7k, Resistor_SMD:R_0603_1608Metric, symbol Device:R_US
- added R23: 10k, Resistor_SMD:R_0603_1608Metric, symbol Device:R_US
- C24: Product (none) -> https://www.digikey.com/en/products/result?keywords=08055C1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
- C25: renamed from R14; value 33k -> 100nF; footprint Resistor_SMD:R_0603_1608Metric -> Capacitor_SMD:C_0603_1608Metric; symbol Device:R_US -> Device:C; Product (none) -> https://www.digikey.com/en/products/result?keywords=C0603C1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
- C26, C27: Product (none) -> https://www.digikey.com/en/products/result?keywords=C1210C2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
- J4: footprint Connector_Molex:Molex_KK-254_AE-6410-04A_1x04_P2.54mm_Vertical -> Connector_JST:JST_XH_S4B-XH-A_1x04_P2.50mm_Horizontal; Product (none) -> https://www.digikey.com/en/products/result?keywords=S4B-XH-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
- J5: renamed from R23; value 10k -> ALPHACOOL ES FLOW (3-pin); footprint Resistor_SMD:R_0603_1608Metric -> Connector_JST:JST_XH_S3B-XH-A_1x03_P2.50mm_Horizontal; symbol Device:R_US -> Connector_Generic:Conn_01x03; Product (none) -> https://www.digikey.com/en/products/result?keywords=S3B-XH-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
- J6: footprint Connector_JST:JST_XH_B2B-XH-A_1x02_P2.50mm_Vertical -> Connector_Hirose:Hirose_DF13-02P-1.25DS_1x02_P1.25mm_Horizontal; Product (none) -> https://www.digikey.com/en/products/result?keywords=DF13-2P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
- R14: renamed from R15; value 4.7k -> 33k; Product (none) -> https://www.digikey.com/en/products/result?keywords=RC0603F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
- R15: renamed from R16; value 10k -> 4.7k; Product (none) -> https://www.digikey.com/en/products/result?keywords=RC0603F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
- R16: renamed from D2; value FAN FAULT -> 10k; footprint LED_SMD:LED_0603_1608Metric -> Resistor_SMD:R_0603_1608Metric; symbol Device:LED -> Device:R_US; Product (none) -> https://www.digikey.com/en/products/result?keywords=AR0603F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
- R17: renamed from J3; value FAN (4-pin PWM) -> 1k; footprint Connector_Molex:Molex_KK-254_AE-6410-04A_1x04_P2.54mm_Vertical -> Resistor_SMD:R_0603_1608Metric; symbol Connector_Generic:Conn_01x04 -> Device:R_US; Product (none) -> https://www.digikey.com/en/products/result?keywords=RC0603F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
- R18: renamed from R19; value 4.7k -> 10k; Product (none) -> https://www.digikey.com/en/products/result?keywords=AR0603F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
- R20: renamed from R21; value 4.7k -> 10k; Product (none) -> https://www.digikey.com/en/products/result?keywords=AR0603F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
- R22: Product (none) -> https://www.digikey.com/en/products/result?keywords=RC0603F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
- R24: renamed from C28; value 100nF -> 10k; footprint Capacitor_SMD:C_0603_1608Metric -> Resistor_SMD:R_0603_1608Metric; symbol Device:C -> Device:R_US; Product (none) -> https://www.digikey.com/en/products/result?keywords=AR0603F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
- U10: Product (none) -> https://www.digikey.com/en/products/result?keywords=EMC2303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
Connections:
- net +12V: now also J5.2 (Pin_2), J3.2 (Pin_2); no longer R17.2 (Pin_2)
- net +3V3_COOL: now also R16.1, R17.1, R24.1, R19.1, R21.1, R23.1; no longer J5.1
- net FAN_ALERT: now also R16.2, D2.1 (K); no longer R15.2, R16.1 (K)
- net FLOW_TACH: now also R23.2; no longer J5.2
- net GND: now also C25.2, J5.1 (Pin_1), C28.2, J3.1 (Pin_1); no longer R17.1 (Pin_1), R24.2
- net NTC_ADC: now also R24.2, C28.1; no longer R24.1
- net at J4.3 (Pin_3), U10.8 (TACH2): now also R21.2; no longer R20.2
- net at J4.4 (Pin_4), U10.7 (PWM2): now also R20.2
- net at U10.5 (PWM1): now also R18.2, J3.4 (Pin_4); no longer R17.4 (Pin_4)
- net at R22.2: now also J5.3 (Pin_3)
- net at U10.4 (ADDR_SEL): now also R14.2; no longer C25.2
- net at U10.9 (CLK): now also R15.2; no longer R14.2
- new net: D2.2 (A), R17.2
- new net: J3.3 (Pin_3), R19.2, U10.6 (TACH1)
Other:
- moved on the sheet: R14, R15, R16, R18, R20

Commit message: Use an M12 receptacle for the PT1000 and JST PH headers for the 2-pin I/O
- J10 (cold head PT1000): TE T4145035041-001, M12 A-coded 4-pin female,
  right angle, shielded, panel and PCB mount through the right side wall;
  footprint from TE drawing T41450350X1001 rev B
- J6, J7, J13 (NTC, panel button, relay out): Adafruit 1769 (4UCON 17311),
  JST PH compatible 2-pin right-angle SMT; footprint from its drawing
- BOM, part links and 3D envelopes for both; schematic nets unchanged
- gen_pcb: ground fan-out before routing (a locked via and short track per
  small ground pad, clear of other holes) so no ground pad is left on a
  pour island; fallback labels must sit inside a section box
- fix_route: skip paste apertures (not non-plated holes) as foreign copper,
  nudge tracks off crowded pads, remove GND vias that crowd another hole

DRC 0 errors, 0 unconnected, 0 schematic-parity issues; ERC 0; 193/193
datasheet rules.

Co-Authored-By: Claude Opus 5.5 <noreply@anthropic.com>
Parts:
- J6: footprint Connector_Hirose:Hirose_DF13-02P-1.25DS_1x02_P1.25mm_Horizontal -> cryocooler:Adafruit_1769_JST-PH_1x02_P2.00mm_Horizontal_SMD; Product https://www.digikey.com/en/products/result?keywords=DF13-2P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 -> https://www.adafruit.com/product/1769
Changed lines of the file:
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@@
 			)
 		)
-		(property "Footprint" "Connector_Hirose:Hirose_DF13-02P-1.25DS_1x02_P1.25mm_Horizontal"
+		(property "Footprint" "cryocooler:Adafruit_1769_JST-PH_1x02_P2.00mm_Horizontal_SMD"
 			(at 139.7 190.5 0)
 			(hide yes)
@@
 			)
 		)
-		(property "Datasheet" "https://www.hirose.com/api/v1/series/DF13/documents/product_series_catalog/content?lang=EN"
+		(property "Datasheet" "https://cdn-shop.adafruit.com/datasheets/17311.pdf"
 			(at 139.7 190.5 0)
 			(hide yes)
@@
 			)
 		)
-		(property "Product" "https://www.digikey.com/en/products/result?keywords=DF13-2P-1.25DS%2825%29"
+		(property "Product" "https://www.adafruit.com/product/1769"
 			(at 139.7 190.5 0)
 			(hide yes)
