File: hardware/kicad/sheets/indicators.kicad_sch (KiCad schematic)
At the start: 10 parts, among them U24 74AHCT1G125

Commit message: KiCad: cleaner layout, decoupling blocks, label directions, KiCad format fixes
- move IC decoupling caps into labelled blocks at the side of each sheet
- global labels show input/output direction per net
- no 4-way junctions (generator now checks and fails)
- generator output matches KiCad's saved format (hide property, junction
  and wire normalisation, lib symbol embedded fonts, multi-unit pins)
- hand-laid USB ESD protection as a pass-through

Co-Authored-By: Claude Sonnet 5.5 <noreply@anthropic.com>
Other:
- note added: "74AHCT1G125 DECOUPLING CAPACITORS"
- note added: "WS2812B DECOUPLING CAPACITORS"
