File: hardware/kicad/sheets/indicators.kicad_sch (KiCad schematic)
At the start: 10 parts, among them U24 74AHCT1G125

Commit message: Put supply pins on top and grounds on the bottom of IC symbols; flake8-clean Python
Schematic: re-laid out pins on U2, U3, U6, U7, U11, U14, U17-U20, U22-U24
and PS1 (supply on top, ground/strap pins on the bottom edge) via custom
`cryocooler:` symbols (make_lib.from_stock) and a gnd_bus helper; U18/U2
use mirroring instead of a 180 degree rotation. Nets are unchanged (ERC 0,
117/117 datasheet rules, PCB nets still match). Text placement now shows
every power-symbol name, avoids wires, and uses a realistic character width.

Python: black -l 79 -S plus manual wrapping so hardware/kicad and scripts/
pass flake8; add .flake8.

Co-Authored-By: Claude Sonnet 5.5 <noreply@anthropic.com>
Parts:
- removed C74: 100nF, Capacitor_SMD:C_0603_1608Metric, symbol Device:C
- removed D9: WS2812B, LED_SMD:LED_WS2812B_PLCC4_5.0x5.0mm_P3.2mm, symbol LED:WS2812B
- removed R70: 10k, Resistor_SMD:R_0603_1608Metric, symbol Device:R_US
- added D7: READY (green), LED_SMD:LED_0603_1608Metric, symbol Device:LED
- added D8: FAULT (red), LED_SMD:LED_0603_1608Metric, symbol Device:LED
- added R68: 470, Resistor_SMD:R_0603_1608Metric, symbol Device:R_US
- C74: renamed from R71; value 330 -> 100nF; footprint Resistor_SMD:R_0603_1608Metric -> Capacitor_SMD:C_0603_1608Metric; symbol Device:R_US -> Device:C
- D9: renamed from D7; value READY (green) -> WS2812B; footprint LED_SMD:LED_0603_1608Metric -> LED_SMD:LED_WS2812B_PLCC4_5.0x5.0mm_P3.2mm; symbol Device:LED -> LED:WS2812B
- R70: renamed from D8; value FAULT (red) -> 10k; footprint LED_SMD:LED_0603_1608Metric -> Resistor_SMD:R_0603_1608Metric; symbol Device:LED -> Device:R_US
- R71: renamed from U24; value 74AHCT1G125 -> 330; footprint Package_TO_SOT_SMD:SOT-23-5 -> Resistor_SMD:R_0603_1608Metric; symbol 74xGxx:74AHCT1G125 -> Device:R_US
- U24: renamed from R68; value 470 -> 74AHCT1G125; footprint Resistor_SMD:R_0603_1608Metric -> Package_TO_SOT_SMD:SOT-23-5; symbol Device:R_US -> cryocooler:74AHCT1G125
Connections:
- net +5V: now also C74.1, D9.1 (VDD), U24.5 (VCC); no longer R71.5 (VCC)
- net GND: now also C74.2, D9.3 (VSS), R70.2, U24.1, U24.3 (GND), D7.1 (K), D8.1 (K); no longer D9.1 (K), R70.1 (K), R71.1, R71.3 (GND)
- net LED_READY: now also R68.1; no longer U24.1
- net STATUS_RGB: now also R70.1, U24.2; no longer R71.2
- net at D9.2 (DOUT): no longer U24.2
- net at R69.2: now also D8.2 (A); no longer R70.2 (A)
- new net: R71.1, U24.4
- new net: D9.4 (DIN), R71.2
- new net: D7.2 (A), R68.2
Other:
- moved on the sheet: R70

Commit message: KiCad schematic: INA239, ADS1220, SC18IS604 bridge, relay driver, test points
- system_current: INA237 -> INA239 (SPI, CS GPIO3) with the 49.9 ohm / 470 nF
  input filter, power LED and ALERT LED; VBUS shares the filtered IN- node.
- cold_head: ADS122C04 -> ADS1220 (SPI, CS GPIO44).
- i2c_bridge (new): SC18IS604 SPI-to-I2C bridge for the EMC2303, with a
  74LVC1G125 gating its MISO onto the shared bus.
- compressor_relay (new): GPIO16 high-side switch sharing one generator
  function with the amplifier REM switch.
- debug (new): about 40 test points and rail LEDs (the isolated rail LED
  returns to ISO_GND).
- ISO7741 -> ACS37800 SPI lines are straight wires (pins reordered on the
  symbol); USB_VBUS is one wire plus a naming label.
- Custom symbols for INA239, ADS1220, SC18IS604; datasheet rules 117 -> 162;
  GPIO map checks updated. ERC 0.

Co-Authored-By: Claude Sonnet 5.5 <noreply@anthropic.com>
Parts:
- removed D7: READY (green), LED_SMD:LED_0603_1608Metric, symbol Device:LED
- removed D8: FAULT (red), LED_SMD:LED_0603_1608Metric, symbol Device:LED
- removed D9: WS2812B, LED_SMD:LED_WS2812B_PLCC4_5.0x5.0mm_P3.2mm, symbol LED:WS2812B
- removed R68, R69: 470, Resistor_SMD:R_0603_1608Metric, symbol Device:R_US
- removed R70: 10k, Resistor_SMD:R_0603_1608Metric, symbol Device:R_US
- added C75, C76: 100nF, Capacitor_SMD:C_0603_1608Metric, symbol Device:C
- added D9: READY (green), LED_SMD:LED_0603_1608Metric, symbol Device:LED
- added R73: 470, Resistor_SMD:R_0603_1608Metric, symbol Device:R_US
- added R74: 10k, Resistor_SMD:R_0603_1608Metric, symbol Device:R_US
- added R75: 330, Resistor_SMD:R_0603_1608Metric, symbol Device:R_US
- D10: renamed from C73; value 100nF -> FAULT (red); footprint Capacitor_SMD:C_0603_1608Metric -> LED_SMD:LED_0603_1608Metric; symbol Device:C -> Device:LED
- D11: renamed from C74; value 100nF -> WS2812B; footprint Capacitor_SMD:C_0603_1608Metric -> LED_SMD:LED_WS2812B_PLCC4_5.0x5.0mm_P3.2mm; symbol Device:C -> LED:WS2812B
- R72: renamed from R71; value 330 -> 470
Connections:
- net +5V: now also C75.1, C76.1; no longer D10.1
- net GND: now also D10.1 (K), D11.3 (VSS), C75.2, C76.2, D9.1 (K), R74.2; no longer D10.2, D11.2
- net LED_FAULT: now also R73.1
- net LED_READY: now also R72.1
- net STATUS_RGB: now also R74.1
- net at U24.4: now also R75.1; no longer R72.1
- net at R72.2: now also D9.2 (A)
- new net: D11.4 (DIN), R75.2
- new net: D10.2 (A), R73.2
Other:
- moved on the sheet: R72

Commit message: Move the IMU off-board (J14) and add labelled module boxes to the PCB
The LSM6DSOX is now the Adafruit breakout (product 4438) mounted on the
cryocooler and cabled to a 10-pin JST XH header (J14) over the shared SPI
bus. U19 and its capacitors are gone; J14 and six 100 R series resistors
are added, and every other reference number is unchanged.

PCB (130 x 110 mm, was 130 x 100):
- one outlined, labelled silkscreen box per module (pcbfloorplan.py); the
  placer keeps parts inside their box and reserves a label pocket beside
  every part so each label sits next to its own part
- box 3D models for U3, L2, L3, F1 and PS1, whose library models are missing
- re-routed; DRC 0 errors, 0 unconnected; back logo recentred
- gen_pcb.py texts redoes the silkscreen on a routed board

Firmware: SPI clock constant for the module, comments updated; ambient
temperature now reads the cooler-body IMU temperature.

Docs, BOM and fabrication files regenerated.

Co-Authored-By: Claude Sonnet 5.5 <noreply@anthropic.com>
Parts:
- removed C75: 100nF, Capacitor_SMD:C_0603_1608Metric, symbol Device:C
- removed D9: READY (green), LED_SMD:LED_0603_1608Metric, symbol Device:LED
- removed R72: 470, Resistor_SMD:R_0603_1608Metric, symbol Device:R_US
- added C76: 100nF, Capacitor_SMD:C_0603_1608Metric, symbol Device:C
- added R74: 10k, Resistor_SMD:R_0603_1608Metric, symbol Device:R_US
- added U24: 74AHCT1G125, Package_TO_SOT_SMD:SOT-23-5, symbol cryocooler:74AHCT1G125
- D10: renamed from D11; value WS2812B -> FAULT (red); footprint LED_SMD:LED_WS2812B_PLCC4_5.0x5.0mm_P3.2mm -> LED_SMD:LED_0603_1608Metric; symbol LED:WS2812B -> Device:LED
- D11: renamed from R74; value 10k -> WS2812B; footprint Resistor_SMD:R_0603_1608Metric -> LED_SMD:LED_WS2812B_PLCC4_5.0x5.0mm_P3.2mm; symbol Device:R_US -> LED:WS2812B
- D9: renamed from D10; value FAULT (red) -> READY (green)
- R73: renamed from U24; value 74AHCT1G125 -> 470; footprint Package_TO_SOT_SMD:SOT-23-5 -> Resistor_SMD:R_0603_1608Metric; symbol cryocooler:74AHCT1G125 -> Device:R_US
- renumbered C76 to C75, R73 to R72
Connections:
- net +5V: now also D11.1 (VDD), C76.1, U24.5 (VCC); no longer D10.1 (VDD), R73.5 (VCC)
- net GND: now also D10.1 (K), D11.3 (VSS), C76.2, R74.2, U24.1, U24.3 (GND); no longer D10.3 (VSS), D11.2, R73.1, R73.3 (GND)
- net LED_FAULT: now also R73.1; no longer R72.1
- net LED_READY: now also R72.1
- net STATUS_RGB: now also R74.1, U24.2; no longer D11.1, R73.2
- net at R75.1: now also U24.4; no longer R73.4
- net at R75.2: now also D11.4 (DIN); no longer D10.4 (DIN)
- net at D10.2 (A): now also R73.2
Other:
- moved on the sheet: C75, D9, R72

Commit message: Add per-section supply jumpers, 8-pin IMU header and connector pin labels
- Four 1.27 mm 2-pin jumpers (JP1-JP4), each with a rail-on LED, cut the
  supply of one section for debugging: signal generator +3V3, +-15V
  generator +5V in, isolated amp-current supply +5V in, and a shared
  +3V3 net for the cooling chips (EMC2303, RTD ADC, I2C bridge).
- J14 is now an 8-pin JST XH in the Adafruit LSM6DSOX pad order
  (VIN, GND, SCL, SDA, DO, CS, I1, I2); firmware pin comments updated.
- Pin-function labels beside every connector, "RAILS ±15V" box title.
- Board re-placed and re-routed (130 x 110 mm); DRC 0 errors, 0 unconnected,
  ERC 0, 173 datasheet rules pass. BOM, READMEs, Gerbers and renders
  regenerated; link_usb_vbus.py now adapts to the routed layout.

Co-Authored-By: Claude Sonnet 5.5 <noreply@anthropic.com>
Parts:
- removed R73: 470, Resistor_SMD:R_0603_1608Metric, symbol Device:R_US
- removed R75: 330, Resistor_SMD:R_0603_1608Metric, symbol Device:R_US
- removed U24: 74AHCT1G125, Package_TO_SOT_SMD:SOT-23-5, symbol cryocooler:74AHCT1G125
- added D10: FAULT (red), LED_SMD:LED_0603_1608Metric, symbol Device:LED
- added D9: READY (green), LED_SMD:LED_0603_1608Metric, symbol Device:LED
- added R74: 10k, Resistor_SMD:R_0603_1608Metric, symbol Device:R_US
- R73: renamed from D9; value READY (green) -> 470; footprint LED_SMD:LED_0603_1608Metric -> Resistor_SMD:R_0603_1608Metric; symbol Device:LED -> Device:R_US
- R75: renamed from R74; value 10k -> 330
- U24: renamed from D10; value FAULT (red) -> 74AHCT1G125; footprint LED_SMD:LED_0603_1608Metric -> Package_TO_SOT_SMD:SOT-23-5; symbol Device:LED -> cryocooler:74AHCT1G125
Connections:
- net +5V: now also U24.5 (VCC)
- net GND: now also U24.3 (GND), D10.1 (K), D9.1 (K), R74.2; no longer R73.1 (K), R75.2
- net LED_FAULT: now also R73.1
- net STATUS_RGB: now also U24.2, R74.1; no longer R75.1
- net at D11.4 (DIN): now also R75.2
- net at R72.2: now also D9.2 (A); no longer R73.2 (A)
- new net: D10.2 (A), R73.2
- new net: R75.1, U24.4
Other:
- moved on the sheet: R73, R75
