File: hardware/kicad/sheets/indicators.kicad_sch (KiCad schematic)
At the start: 10 parts, among them U24 74AHCT1G125

Commit message: Replace the ±15 V LDOs with one LT3097 and add a power-good interlock
- rails_15v: ADP7142 + ADP7182 replaced by one LT3097 (±14.7 V, 147 k SET
  resistors); the ADP5071 output caps are now 22 uF / 50 V and double as the
  LT3097 inputs. PGP / PGN make the PG_15V node (fed from +15 V, so it reads
  0 V if a rail is missing).
- amp_control: a series BSS138 (Q9) gated by PG_15V blocks AMP_REM unless
  both rails are good. New power_good sheet: LED (D23) and the active-low
  PG_15V_N flag on GPIO43 (PG_15V_N_PIN).
- Tooling: LT3097 symbol, footprint and 3D envelope; datasheet rules (191),
  GPIO check, BOM tables, floor plan, PAD_BRIDGES and pre-placed GND vias in
  gen_pcb.py, new fix_route.py for post-route clean-up.
- Board regenerated and routed with Freerouting 2.5.0: DRC 0 unconnected,
  0 schematic-parity issues, no copper violations. Gerbers, JLCPCB zip,
  renders, BOM, CPL and schematic PDF regenerated.

Co-Authored-By: Claude Sonnet 5.5 <noreply@anthropic.com>
Parts:
- removed R73: 470, Resistor_SMD:R_0603_1608Metric, symbol Device:R_US
- removed U24: 74AHCT1G125, Package_TO_SOT_SMD:SOT-23-5, symbol cryocooler:74AHCT1G125
- added C75, C76: 100nF, Capacitor_SMD:C_0603_1608Metric, symbol Device:C
- R73: renamed from C75; value 100nF -> 470; footprint Capacitor_SMD:C_0603_1608Metric -> Resistor_SMD:R_0603_1608Metric; symbol Device:C -> Device:R_US
- U24: renamed from C76; value 100nF -> 74AHCT1G125; footprint Capacitor_SMD:C_0603_1608Metric -> Package_TO_SOT_SMD:SOT-23-5; symbol Device:C -> cryocooler:74AHCT1G125
Connections:
- net +5V: now also U24.5 (VCC), C75.1, C76.1; no longer R73.1, U24.1
- net GND: now also U24.1, U24.3 (GND), C75.2, C76.2; no longer R73.2, U24.2
- net LED_FAULT: now also R73.1
- net STATUS_RGB: now also U24.2
- net at D10.2 (A): now also R73.2
- net at R75.1: now also U24.4

Commit message: Log +-15 V power-good changes and add one LED per LT3097 PG pin
Firmware
- amplifier: configure PG_15V_N_PIN (GPIO43, active LOW), log the starting
  state and every debounced change (PowerGoodMonitor in power_good.h);
  amplifier::isPowerGood() reports the level. The lines reach the dashboard
  console through the logger ring buffer.
- dashboard: console colours for "power lost" (red), "power restored" and
  "power good: yes" (green), "power good: no" (yellow).
- native tests for the debounce logic and the amplifier stub.

Hardware
- power_good sheet: PGP and PGN each drive their own node (220k/62k from
  +15 V) and a green LED (D24 +15 V, D25 -15 V) through a BSS138W; a BAT54AW
  with a 10k pull-up ANDs the nodes into PG_15V, so the REM interlock and the
  PG_15V_N flag are unchanged.
- 0402 resistors, SOT-323 FETs and one BAT54AW so the stage fits the power
  box; Power Good parts are placed last in gen_pcb.py.
- Board re-routed with Freerouting 2.5.0 and cleaned with fix_route.py: DRC
  0 unconnected, no copper violations. Gerbers, JLCPCB zip, renders, BOM, CPL
  and schematic PDF regenerated; datasheet rules 193/193.

Co-Authored-By: Claude Sonnet 5.5 <noreply@anthropic.com>
Parts:
- removed D10: FAULT (red), LED_SMD:LED_0603_1608Metric, symbol Device:LED
- removed D9: READY (green), LED_SMD:LED_0603_1608Metric, symbol Device:LED
- added C75, C76: 100nF, Capacitor_SMD:C_0603_1608Metric, symbol Device:C
- D10: renamed from C76; value 100nF -> FAULT (red); footprint Capacitor_SMD:C_0603_1608Metric -> LED_SMD:LED_0603_1608Metric; symbol Device:C -> Device:LED
- D9: renamed from C75; value 100nF -> READY (green); footprint Capacitor_SMD:C_0603_1608Metric -> LED_SMD:LED_0603_1608Metric; symbol Device:C -> Device:LED
Connections:
- net +5V: now also C75.1, C76.1; no longer D10.1, D9.1
- net GND: now also D10.1 (K), D9.1 (K), C75.2, C76.2; no longer D10.2, D9.2
- net at R72.2: now also D9.2 (A)
- net at R73.2: now also D10.2 (A)

Commit message: WIP: restructure PCB for the Phoenix UCS 125-87 housing
Work in progress, layout not finished: about 90 parts still do not fit
their sections and the board is not routed.

- Right-angle connectors: Phoenix MSTBA 2,5 / MC 1,5, JST XH side entry,
  Hirose DF13, Molex 505448-0871 (new footprint from the Molex drawing)
- Datasheet and product links on every symbol (tools/part_links.py)
- Test points so every IC has one on its own nets
- gen_pcb.py: 100 x 62 mm two-sided board, housing holes and restricted
  corners, ESP32 antenna notch, one section per sheet, board ID block,
  ESP32 pin names, pin-1 marks, blue mask
- Housing drawings in hardware/housing/

Co-Authored-By: Claude Opus 5.5 <noreply@anthropic.com>
Parts:
- removed C75: 100nF, Capacitor_SMD:C_0603_1608Metric, symbol Device:C
- removed D9: READY (green), LED_SMD:LED_0603_1608Metric, symbol Device:LED
- removed R72: 470, Resistor_SMD:R_0603_1608Metric, symbol Device:R_US
- added C76: 100nF, Capacitor_SMD:C_0603_1608Metric, symbol Device:C
- added R74: 10k, Resistor_SMD:R_0603_1608Metric, symbol Device:R_US
- added U24: 74AHCT1G125, Package_TO_SOT_SMD:SOT-23-5, symbol cryocooler:74AHCT1G125
- C75: renamed from C76; Product (none) -> https://www.digikey.com/en/products/result?keywords=C0603C1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
- D10: renamed from D11; value WS2812B -> FAULT (red); footprint LED_SMD:LED_WS2812B_PLCC4_5.0x5.0mm_P3.2mm -> LED_SMD:LED_0603_1608Metric; symbol LED:WS2812B -> Device:LED; Product (none) -> https://www.digikey.com/en/products/result?keywords=LTST-C1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
- D11: renamed from R74; value 10k -> WS2812B; footprint Resistor_SMD:R_0603_1608Metric -> LED_SMD:LED_WS2812B_PLCC4_5.0x5.0mm_P3.2mm; symbol Device:R_US -> LED:WS2812B; Product (none) -> https://www.digikey.com/en/products/result?keywords=1655
- D9: renamed from D10; value FAULT (red) -> READY (green); Product (none) -> https://www.digikey.com/en/products/result?keywords=LTST-C1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
- R72: renamed from R73; Product (none) -> https://www.digikey.com/en/products/result?keywords=RC0603F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
- R73: renamed from U24; value 74AHCT1G125 -> 470; footprint Package_TO_SOT_SMD:SOT-23-5 -> Resistor_SMD:R_0603_1608Metric; symbol cryocooler:74AHCT1G125 -> Device:R_US; Product (none) -> https://www.digikey.com/en/products/result?keywords=RC0603F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
- R75: Product (none) -> https://www.digikey.com/en/products/result?keywords=RC0603F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
Connections:
- net +5V: now also D11.1 (VDD), C76.1, U24.5 (VCC); no longer D10.1 (VDD), R73.5 (VCC)
- net GND: now also D10.1 (K), D11.3 (VSS), C76.2, R74.2, U24.1, U24.3 (GND); no longer D10.3 (VSS), D11.2, R73.1, R73.3 (GND)
- net LED_FAULT: now also R73.1; no longer R72.1
- net LED_READY: now also R72.1
- net STATUS_RGB: now also R74.1, U24.2; no longer D11.1, R73.2
- net at R75.1: now also U24.4; no longer R73.4
- net at R75.2: now also D11.4 (DIN); no longer D10.4 (DIN)
- net at D10.2 (A): now also R73.2
Other:
- moved on the sheet: C75, D9, R72

Commit message: Ground the M12 shield, order the ground loops, name the J14 cable parts
- J10: shielded symbol (Conn_01x04_Shielded); the M12 shield pin and its
  four shell legs are pad SH, tied to GND
- TP22-TP25: Keystone 5001 black miniature PC test points (KiCad
  TestPoint_Keystone_5000-5004 footprint, 1.02 mm hole per Keystone's
  drawing); now in the BOM, the bare pad test points stay out
- J14 BOM note: cable housing Molex 5054320801 with 505431 terminals, or
  tin pre-crimped leads 797581148 / 797581149 (from molex.com)

Only netlist change: GND gains J10 SH. DRC 0 errors, 0 unconnected, 0
schematic-parity issues; ERC 0; 193/193 datasheet rules.

Co-Authored-By: Claude Opus 5.5 <noreply@anthropic.com>
Parts:
- removed R72, R73: 470, Resistor_SMD:R_0603_1608Metric, symbol Device:R_US
- removed U24: 74AHCT1G125, Package_TO_SOT_SMD:SOT-23-5, symbol cryocooler:74AHCT1G125
- added D10: FAULT (red), LED_SMD:LED_0603_1608Metric, symbol Device:LED
- added D11: WS2812B, LED_SMD:LED_WS2812B_PLCC4_5.0x5.0mm_P3.2mm, symbol LED:WS2812B
- added D9: READY (green), LED_SMD:LED_0603_1608Metric, symbol Device:LED
- R72: renamed from D9; value READY (green) -> 470; footprint LED_SMD:LED_0603_1608Metric -> Resistor_SMD:R_0603_1608Metric; symbol Device:LED -> Device:R_US; Product https://www.digikey.com/en/products/result?keywords=LTST-C1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 -> https://www.digikey.com/en/products/result?keywords=RC0603F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
- R73: renamed from D10; value FAULT (red) -> 470; footprint LED_SMD:LED_0603_1608Metric -> Resistor_SMD:R_0603_1608Metric; symbol Device:LED -> Device:R_US; Product https://www.digikey.com/en/products/result?keywords=LTST-C1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 -> https://www.digikey.com/en/products/result?keywords=RC0603F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
- U24: renamed from D11; value WS2812B -> 74AHCT1G125; footprint LED_SMD:LED_WS2812B_PLCC4_5.0x5.0mm_P3.2mm -> Package_TO_SOT_SMD:SOT-23-5; symbol LED:WS2812B -> cryocooler:74AHCT1G125; Product https://www.digikey.com/en/products/result?keywords=1655 -> https://www.digikey.com/en/products/result?keywords=SN74AHC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
Connections:
- net +5V: now also U24.5 (VCC), D11.1 (VDD); no longer U24.1 (VDD)
- net GND: now also U24.1, D10.1 (K), D11.3 (VSS), D9.1 (K); no longer R72.1 (K), R73.1 (K)
- net LED_FAULT: now also R73.1
- net LED_READY: now also R72.1
- net STATUS_RGB: now also U24.2
- net at R73.2: now also D10.2 (A)
- net at R72.2: now also D9.2 (A)
- net at R75.1: now also U24.4
- net at R75.2: now also D11.4 (DIN); no longer U24.4 (DIN)
Other:
- moved on the sheet: R72, R73
