File: hardware/kicad/sheets/power_button.kicad_sch (KiCad schematic)
At the start: 22 parts, among them J3 PANEL BUTTON, Q1 IRF4905S, Q2 BSS138, Q3 BSS138, Q4 BSS138, SW3 POWER, U3 LTC2954CTS8-2, U4 LM4040DBZ-5, U5 CL25N8-G

Commit message: KiCad: cleaner layout, decoupling blocks, label directions, KiCad format fixes
- move IC decoupling caps into labelled blocks at the side of each sheet
- global labels show input/output direction per net
- no 4-way junctions (generator now checks and fails)
- generator output matches KiCad's saved format (hide property, junction
  and wire normalisation, lib symbol embedded fonts, multi-unit pins)
- hand-laid USB ESD protection as a pass-through

Co-Authored-By: Claude Sonnet 5.5 <noreply@anthropic.com>
Parts:
- C8: footprint Capacitor_SMD:C_0805_2012Metric -> Capacitor_SMD:C_0603_1608Metric
Other:
- note added: "LTC2954 DECOUPLING CAPACITORS"
