File: hardware/kicad/sheets/power_button.kicad_sch (KiCad schematic)
At the start: 22 parts, among them J3 PANEL BUTTON, Q1 IRF4905S, Q2 BSS138, Q3 BSS138, Q4 BSS138, SW3 POWER, U3 LTC2954CTS8-2, U4 LM4040DBZ-5, U5 CL25N8-G

Commit message: Fixing the UUID issues
Parts:
- removed C8, C9: 100nF, Capacitor_SMD:C_0603_1608Metric, symbol Device:C
- removed D2: RED/GREEN, LED_SMD:LED_1206_3216Metric, symbol Device:LED_Dual_Bidirectional
- removed J3: PANEL BUTTON, Connector_JST:JST_XH_B2B-XH-A_1x02_P2.50mm_Vertical, symbol Connector_Generic:Conn_01x02
- removed R10, R14, R8: 10k, Resistor_SMD:R_0603_1608Metric, symbol Device:R_US
- removed R11, R15, R16: 100k, Resistor_SMD:R_0603_1608Metric, symbol Device:R_US
- removed R12, R13: 330, Resistor_SMD:R_0603_1608Metric, symbol Device:R_US
- removed R7: 220k, Resistor_SMD:R_0603_1608Metric, symbol Device:R_US
- removed R9: 82k, Resistor_SMD:R_0603_1608Metric, symbol Device:R_US
- removed U3: LTC2954CTS8-2, Package_TO_SOT_SMD:SOT-23-8, symbol cryocooler:LTC2954CTS8-2
- removed U4: LM4040DBZ-5, Package_TO_SOT_SMD:SOT-23, symbol Reference_Voltage:LM4040DBZ-5
- removed U5: CL25N8-G, Package_TO_SOT_SMD:SOT-89-3, symbol cryocooler:CL25N8-G
- added C29, C30: 100nF, Capacitor_SMD:C_0603_1608Metric, symbol Device:C
- added D3: RED/GREEN, LED_SMD:LED_1206_3216Metric, symbol Device:LED_Dual_Bidirectional
- added J7: PANEL BUTTON, Connector_JST:JST_XH_B2B-XH-A_1x02_P2.50mm_Vertical, symbol Connector_Generic:Conn_01x02
- added R27: 220k, Resistor_SMD:R_0603_1608Metric, symbol Device:R_US
- added R28, R30, R34: 10k, Resistor_SMD:R_0603_1608Metric, symbol Device:R_US
- added R29: 82k, Resistor_SMD:R_0603_1608Metric, symbol Device:R_US
- added R31, R35, R36: 100k, Resistor_SMD:R_0603_1608Metric, symbol Device:R_US
- added R32, R33: 330, Resistor_SMD:R_0603_1608Metric, symbol Device:R_US
- added U11: LTC2954CTS8-2, Package_TO_SOT_SMD:SOT-23-8, symbol cryocooler:LTC2954CTS8-2
- added U12: LM4040DBZ-5, Package_TO_SOT_SMD:SOT-23, symbol Reference_Voltage:LM4040DBZ-5
- added U13: CL25N8-G, Package_TO_SOT_SMD:SOT-89-3, symbol cryocooler:CL25N8-G
Connections:
- net +3V3: now also R30.2, R34.1
- net GND: now also C29.2, C30.2, J7.2 (Pin_2), R35.2, U11.4 (GND), U12.2 (A)
- net PWR_INT: now also R30.1, U11.5 (~{INT})
- net PWR_KILL: now also R28.2
- net VIN: now also C29.1, R29.1, R31.1, R36.1, U11.1 (VIN), U13.1 (VA)
- net at Q1.1 (G): now also R31.2, U11.6 (~{EN})
- net at Q2.1 (G), Q4.1 (G): now also R34.2, R35.1
- net at Q3.1 (G), Q4.3 (D): now also R36.2
- net at Q2.3 (D): now also D3.2 (AK), R32.2
- net at SW3.1: now also J7.1 (Pin_1), U11.2 (PB)
- net at Q3.3 (D): now also D3.1 (KA), R33.2
- new net: R32.1, R33.1, U13.2 (VB)
- new net: C30.1, U11.7 (PDT)
- new net: R27.2, R28.1, U11.8 (~{KILL})
- new net: R27.1, R29.2, U12.1 (K)
