File: hardware/kicad/sheets/signal_gen.kicad_sch (KiCad schematic)
At the start: 32 parts, among them U11 SG-8002CA-PH 25MHz, U12 AD9833BRMZ, U13 OPA1656ID, U14 AD633JRZ-R7, U15 MCP4921-E/SN, U16 LM4040DBZ-2.5, U17 OPA188ID

Commit message: KiCad: cleaner layout, decoupling blocks, label directions, KiCad format fixes
- move IC decoupling caps into labelled blocks at the side of each sheet
- global labels show input/output direction per net
- no 4-way junctions (generator now checks and fails)
- generator output matches KiCad's saved format (hide property, junction
  and wire normalisation, lib symbol embedded fonts, multi-unit pins)
- hand-laid USB ESD protection as a pass-through

Co-Authored-By: Claude Sonnet 5.5 <noreply@anthropic.com>
Parts:
- C32: value 100nF -> 10nF
- C34: value 10uF -> 1uF
- C35: value 10nF -> 10uF; footprint Capacitor_SMD:C_0603_1608Metric -> Capacitor_SMD:C_0805_2012Metric
- C37: value 1uF -> 100nF; footprint Capacitor_SMD:C_0805_2012Metric -> Capacitor_SMD:C_0603_1608Metric
- C39, C45: value 100nF -> 10uF; footprint Capacitor_SMD:C_0603_1608Metric -> Capacitor_SMD:C_0805_2012Metric
- C42, C44: value 10uF -> 100nF; footprint Capacitor_SMD:C_0805_2012Metric -> Capacitor_SMD:C_0603_1608Metric
Connections:
- net +15V: now also C42.1; no longer C38.1
- net +3V3: now also C45.1; no longer C43.1
- net +5V: now also C37.1, C38.1, C39.1; no longer C33.1, C34.1, C35.1
- net -15V: now also C43.1; no longer C39.1
- net GND: now also C37.2, C42.2; no longer C32.2, C34.2
- net SIG_SINE: now also C35.2; no longer C42.2
- net at U12.1 (COMP): now also C32.2; no longer C35.2
- net at U12.10 (VOUT): now also C34.1; no longer C37.1
- net at C36.1: now also R33.2, U15.6 (Vref), U16.1 (K); no longer U12.3 (CAP/2.5V)
- net at R27.1, U13.3 (+): now also C34.2; no longer C37.2
- net at R31.2: now also C35.1; no longer C42.1
- new net: C33.1, U12.3 (CAP/2.5V)
Other:
- note added: "AD633 +15V DECOUPLING CAPACITORS"
- note added: "AD633 -15V DECOUPLING CAPACITORS"
- note added: "AD9833 DECOUPLING CAPACITORS"
- note added: "MCP4921 DECOUPLING CAPACITORS"
- note added: "OPA1656 +15V DECOUPLING CAPACITORS"
- note added: "OPA1656 -15V DECOUPLING CAPACITORS"
- note added: "OPA188 +15V DECOUPLING CAPACITORS"
- note added: "OPA188 -15V DECOUPLING CAPACITORS"
- note added: "SG-8002CA DECOUPLING CAPACITORS"
