File: hardware/kicad/sheets/signal_gen.kicad_sch (KiCad schematic)
At the start: 32 parts, among them U3 SG-8002CA-PH 25MHz, U4 AD9833BRMZ, U5 OPA1656ID, U6 AD633JRZ-R7, U7 MCP4921-E/SN, U8 LM4040DBZ-2.5, U9 OPA188ID

Commit message: WIP: restructure PCB for the Phoenix UCS 125-87 housing
Work in progress, layout not finished: about 90 parts still do not fit
their sections and the board is not routed.

- Right-angle connectors: Phoenix MSTBA 2,5 / MC 1,5, JST XH side entry,
  Hirose DF13, Molex 505448-0871 (new footprint from the Molex drawing)
- Datasheet and product links on every symbol (tools/part_links.py)
- Test points so every IC has one on its own nets
- gen_pcb.py: 100 x 62 mm two-sided board, housing holes and restricted
  corners, ESP32 antenna notch, one section per sheet, board ID block,
  ESP32 pin names, pin-1 marks, blue mask
- Housing drawings in hardware/housing/

Co-Authored-By: Claude Opus 5.5 <noreply@anthropic.com>
Parts:
- removed C10: 1uF, Capacitor_SMD:C_0805_2012Metric, symbol Device:C
- removed C8: 10nF, Capacitor_SMD:C_0603_1608Metric, symbol Device:C
- removed R11: 6.8k, Resistor_SMD:R_0603_1608Metric, symbol Device:R_US
- removed R8, R9: 100, Resistor_SMD:R_0603_1608Metric, symbol Device:R_US
- removed unit 1 of U5
- added C9: 100nF, Capacitor_SMD:C_0603_1608Metric, symbol Device:C
- added R10, R5: 100k, Resistor_SMD:R_0603_1608Metric, symbol Device:R_US
- added R13: 10k, Resistor_SMD:R_0603_1608Metric, symbol Device:R_US
- added R7: 3.3k, Resistor_SMD:R_0603_1608Metric, symbol Device:R_US
- added unit 2 of U5
- added U8: LM4040DBZ-2.5, Package_TO_SOT_SMD:SOT-23, symbol Reference_Voltage:LM4040DBZ-2.5
- C10: renamed from R5; value 100k -> 1uF; footprint Resistor_SMD:R_0603_1608Metric -> Capacitor_SMD:C_0805_2012Metric; symbol Device:R_US -> Device:C; Product (none) -> https://www.digikey.com/en/products/result?keywords=08055C1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
- C11: renamed from R10; value 100k -> 10uF; footprint Resistor_SMD:R_0603_1608Metric -> Capacitor_SMD:C_0805_2012Metric; symbol Device:R_US -> Device:C; Product (none) -> https://www.digikey.com/en/products/result?keywords=CL21A10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
- C12, C13, C14, C16, C17, C18, C19, C20, C22, C23: Product (none) -> https://www.digikey.com/en/products/result?keywords=C0603C1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
- C15, C21: Product (none) -> https://www.digikey.com/en/products/result?keywords=CL21A10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
- C8: renamed from C9; value 100nF -> 10nF; Product (none) -> https://www.digikey.com/en/products/result?keywords=CL10B10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
- R11: renamed from U8; value LM4040DBZ-2.5 -> 6.8k; footprint Package_TO_SOT_SMD:SOT-23 -> Resistor_SMD:R_0603_1608Metric; symbol Reference_Voltage:LM4040DBZ-2.5 -> Device:R_US; Product (none) -> https://www.digikey.com/en/products/result?keywords=RC0603F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
- R12: Product (none) -> https://www.digikey.com/en/products/result?keywords=RC0603F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
- R6: renamed from R7; value 3.3k -> 51k; Product (none) -> https://www.digikey.com/en/products/result?keywords=CR0603-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
- R8: renamed from U5; value OPA1656ID -> 100; footprint Package_SO:SOIC-8_3.9x4.9mm_P1.27mm -> Resistor_SMD:R_0603_1608Metric; symbol Amplifier_Operational:OPA1656ID -> Device:R_US; Product (none) -> https://www.digikey.com/en/products/result?keywords=AR0603F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
- R9: renamed from C11; value 10uF -> 100; footprint Capacitor_SMD:C_0805_2012Metric -> Resistor_SMD:R_0603_1608Metric; symbol Device:C -> Device:R_US; Product (none) -> https://www.digikey.com/en/products/result?keywords=AR0603F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
- TP2: renamed from U9; value OPA188ID -> MCP4921_VREF; footprint Package_SO:SOIC-8_3.9x4.9mm_P1.27mm -> TestPoint:TestPoint_Pad_D1.5mm; symbol Amplifier_Operational:OPA188xxD -> Connector:TestPoint
- U3: Product (none) -> https://www.digikey.com/en/products/result?keywords=SG-8002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
- U4: Product (none) -> https://www.digikey.com/en/products/result?keywords=AD9833B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
- U5: renamed from R6; value 51k -> OPA1656ID; footprint Resistor_SMD:R_0603_1608Metric -> Package_SO:SOIC-8_3.9x4.9mm_P1.27mm; symbol Device:R_US -> Amplifier_Operational:OPA1656ID; Product (none) -> https://www.digikey.com/en/products/result?keywords=OPA1656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
- U5: Product (none) -> https://www.digikey.com/en/products/result?keywords=OPA1656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
- U6: Product (none) -> https://www.digikey.com/en/products/result?keywords=AD633JR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
- U7: Product (none) -> https://www.digikey.com/en/products/result?keywords=MCP4921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
- U9: renamed from R13; value 10k -> OPA188ID; footprint Resistor_SMD:R_0603_1608Metric -> Package_SO:SOIC-8_3.9x4.9mm_P1.27mm; symbol Device:R_US -> Amplifier_Operational:OPA188xxD; Product (none) -> https://www.digikey.com/en/products/result?keywords=OPA188A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
Connections:
- net +15V: now also U9.7 (V+); no longer TP2.7 (V+)
- net +3V3_SG: now also R11.1
- net +5V: now also C8.1
- net -15V: now also U9.4 (V-); no longer TP2.4 (V-)
- net GND: now also C9.2, R10.2, R13.2, R5.2, R7.2, U5.5 (+), U8.2 (A); no longer C10.2, C11.2, C8.2, R11.2 (A), R6.2, R8.5 (+), U9.2
- net SIG_SINE: now also C11.2, R10.1; no longer C11.1, R9.2
- net at R6.1: now also U5.2 (-), R7.1; no longer U5.1
- net at U4.1 (COMP): now also C8.2
- net at U4.10 (VOUT): now also C10.1
- net at U4.3 (CAP/2.5V): now also C9.1; no longer C8.1
- net at U6.7 (X1): now also R8.2
- net at R12.2, U6.1 (Y1): now also U9.6; no longer TP2.6
- net at R9.1: now also U6.5 (W)
- net at C12.1, U7.6 (Vref): now also R11.2, TP2.1, U8.1 (K); no longer R11.1 (K)
- net at U7.8 (Vout): now also U9.3 (+); no longer TP2.3 (+)
- new net: R6.2, R8.1, U5.1
- new net: R12.1, R13.1, U9.2 (-)
- new net: C10.2, R5.1, U5.3 (+)
- new net: C11.1, R9.2
- new net: U5.6 (-), U5.7
- now unconnected: U9.1
Other:
- moved on the sheet: C8, R11, R6

Commit message: Lay out the board for the Phoenix UCS 145-125 housing
Move to a 120 x 100 mm, 4-layer, blue-mask board for the UCS 145-125-F-CCD
7035 housing: housing mounting holes and restricted corners, ESP32 antenna
over a routed notch, one labelled section per schematic sheet with almost
every part on top. Placed, routed and cleaned up: DRC 0 errors, 0
unconnected, 0 schematic-parity issues; ERC 0; 193/193 datasheet rules.

- AGENTS.md: test points go on the same side as the part they test, close
  to it
- gen_pcb: test points held to their IC's side and within 8 mm; silkscreen
  check measures text by ink and also fails on pads, part outlines, section
  lines and pin-1 dots; titles along or up a border; connector labels and
  ESP32 pin names reserved before the passives; pin-1 dots only where the
  footprint has no mark; footprints carry the schematic's library links and
  fields; mounting holes are board-only H1-H4
- fix_route: generic clean-up (no old-board coordinate edits); removes GND
  vias in keep-outs or on foreign pads, links stranded ground pads, nudges
  squeezed tracks, handles back-side pour islands
- kicad_dru: fix the rule file (an invalid USB-C rule made KiCad ignore it);
  housing-corner and antenna keep-out part rules
- schematic: pad test points excluded from the BOM
- README / fabrication README updated for the new board

Co-Authored-By: Claude Opus 5.5 <noreply@anthropic.com>
Parts:
- TP2: now left out of the parts list
Changed lines of the file:
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@@
 		(body_style 1)
 		(exclude_from_sim no)
-		(in_bom yes)
+		(in_bom no)
 		(on_board yes)
 		(in_pos_files yes)
