File: hardware/kicad/sheets/amp_control.kicad_sch (KiCad schematic)
At the start: 10 parts, among them J4 AMP REM / GND, J5 AMP SIGNAL IN / GND, Q5 BSS138, Q6 BSS84

Commit message: Fixing the UUID issues
Parts:
- removed D5: RED/GREEN, LED_SMD:LED_1206_3216Metric, symbol Device:LED_Dual_Bidirectional
- removed J4: AMP REM / GND, TerminalBlock_Phoenix:TerminalBlock_Phoenix_MKDS-1,5-2-5.08_1x02_P5.08mm_Horizontal, symbol Connector:Screw_Terminal_01x02
- removed J5: AMP SIGNAL IN / GND, TerminalBlock_Phoenix:TerminalBlock_Phoenix_MKDS-1,5-2-5.08_1x02_P5.08mm_Horizontal, symbol Connector:Screw_Terminal_01x02
- removed R36: 1k, Resistor_SMD:R_0603_1608Metric, symbol Device:R_US
- added D4: RED/GREEN, LED_SMD:LED_1206_3216Metric, symbol Device:LED_Dual_Bidirectional
- added J8: AMP REM / GND, TerminalBlock_Phoenix:TerminalBlock_Phoenix_MKDS-1,5-2-5.08_1x02_P5.08mm_Horizontal, symbol Connector:Screw_Terminal_01x02
- added J9: AMP SIGNAL IN / GND, TerminalBlock_Phoenix:TerminalBlock_Phoenix_MKDS-1,5-2-5.08_1x02_P5.08mm_Horizontal, symbol Connector:Screw_Terminal_01x02
- added R41: 2.2k, Resistor_SMD:R_0603_1608Metric, symbol Device:R_US
- R37: value 100k -> 1k
- R39: value 1k -> 100k
- R40: value 2.2k -> 1k
Connections:
- net +12V: now also R39.1; no longer R38.1
- net +5V: now also R41.1; no longer R40.1
- net AMP_REM: now also R40.1, D4.2 (AK), J8.1 (Pin_1); no longer R39.1
- net AMP_REM_EN: now also R37.1
- net GND: now also R38.2, R40.2, J8.2 (Pin_2), J9.2 (Pin_2); no longer R37.2, R39.2
- net SIG_SINE: now also J9.1 (Pin_1)
- net at Q5.1 (G): now also R37.2, R38.1; no longer R37.1
- net at Q5.3 (D), Q6.1 (G): now also R39.2; no longer R38.2
- new net: D4.1 (KA), R41.2
