File: hardware/kicad/sheets/cold_head.kicad_sch (KiCad schematic)
At the start: 13 parts, among them J12 RTD PT1000 4-wire, U22 ADS122C04IPWR

Commit message: Fixing the UUID issues
Parts:
- removed C64, C67, C69: 100nF, Capacitor_SMD:C_0603_1608Metric, symbol Device:C
- removed C65: 1uF, Capacitor_SMD:C_0805_2012Metric, symbol Device:C
- removed C66, C68: 10nF, Capacitor_SMD:C_0603_1608Metric, symbol Device:C
- removed J12: RTD PT1000 4-wire, Connector_JST:JST_XH_B4B-XH-A_1x04_P2.50mm_Vertical, symbol Connector_Generic:Conn_01x04
- removed R62, R63: 10k, Resistor_SMD:R_0603_1608Metric, symbol Device:R_US
- removed R64, R65: 1k, Resistor_SMD:R_0603_1608Metric, symbol Device:R_US
- removed R66: 3.9k, Resistor_SMD:R_0603_1608Metric, symbol Device:R_US
- removed U22: ADS122C04IPWR, Package_SO:TSSOP-16_4.4x5mm_P0.65mm, symbol cryocooler:ADS122C04IPWR
- added C31, C34, C36: 100nF, Capacitor_SMD:C_0603_1608Metric, symbol Device:C
- added C32: 1uF, Capacitor_SMD:C_0805_2012Metric, symbol Device:C
- added C33, C35: 10nF, Capacitor_SMD:C_0603_1608Metric, symbol Device:C
- added J10: RTD PT1000 4-wire, Connector_JST:JST_XH_B4B-XH-A_1x04_P2.50mm_Vertical, symbol Connector_Generic:Conn_01x04
- added R42, R43: 10k, Resistor_SMD:R_0603_1608Metric, symbol Device:R_US
- added R44, R45: 1k, Resistor_SMD:R_0603_1608Metric, symbol Device:R_US
- added R46: 3.9k, Resistor_SMD:R_0603_1608Metric, symbol Device:R_US
- added U14: ADS122C04IPWR, Package_SO:TSSOP-16_4.4x5mm_P0.65mm, symbol cryocooler:ADS122C04IPWR
Connections:
- net +3V3: now also C31.1, C32.1, R42.1, R43.1, U14.1 (A0), U14.12 (AVDD), U14.13 (DVDD), U14.2 (A1)
- net GND: now also C31.2, C32.2, C33.2, C35.2, C36.2, R46.2, U14.4 (DGND), U14.5 (AVSS), U14.8 (REFN)
- net SCL: now also U14.16 (SCL)
- net SDA: now also U14.15 (SDA)
- new net: C33.1, C34.1, R44.1, U14.10 (AIN1)
- new net: C34.2, C35.1, R45.1, U14.11 (AIN0)
- new net: R43.2, U14.14 (~{DRDY})
- new net: R42.2, U14.3 (~{RESET})
- new net: J10.1 (Pin_1), U14.6 (AIN3)
- new net: C36.1, J10.4 (Pin_4), R46.1, U14.9 (REFP)
- new net: J10.2 (Pin_2), R44.2
- new net: J10.3 (Pin_3), R45.2
