File: hardware/kicad/sheets/cold_head.kicad_sch (KiCad schematic)
At the start: 13 parts, among them J10 RTD PT1000 4-wire, U14 ADS122C04IPWR

Commit message: Put supply pins on top and grounds on the bottom of IC symbols; flake8-clean Python
Schematic: re-laid out pins on U2, U3, U6, U7, U11, U14, U17-U20, U22-U24
and PS1 (supply on top, ground/strap pins on the bottom edge) via custom
`cryocooler:` symbols (make_lib.from_stock) and a gnd_bus helper; U18/U2
use mirroring instead of a 180 degree rotation. Nets are unchanged (ERC 0,
117/117 datasheet rules, PCB nets still match). Text placement now shows
every power-symbol name, avoids wires, and uses a realistic character width.

Python: black -l 79 -S plus manual wrapping so hardware/kicad and scripts/
pass flake8; add .flake8.

Co-Authored-By: Claude Sonnet 5.5 <noreply@anthropic.com>
Parts:
- removed C34: 100nF, Capacitor_SMD:C_0603_1608Metric, symbol Device:C
- removed J10: RTD PT1000 4-wire, Connector_JST:JST_XH_B4B-XH-A_1x04_P2.50mm_Vertical, symbol Connector_Generic:Conn_01x04
- removed R46: 3.9k, Resistor_SMD:R_0603_1608Metric, symbol Device:R_US
- added C33: 10nF, Capacitor_SMD:C_0603_1608Metric, symbol Device:C
- added R42: 10k, Resistor_SMD:R_0603_1608Metric, symbol Device:R_US
- added R44: 1k, Resistor_SMD:R_0603_1608Metric, symbol Device:R_US
- C34: renamed from R44; value 1k -> 100nF; footprint Resistor_SMD:R_0603_1608Metric -> Capacitor_SMD:C_0603_1608Metric; symbol Device:R_US -> Device:C
- J10: renamed from R43; value 10k -> RTD PT1000 4-wire; footprint Resistor_SMD:R_0603_1608Metric -> Connector_JST:JST_XH_B4B-XH-A_1x04_P2.50mm_Vertical; symbol Device:R_US -> Connector_Generic:Conn_01x04
- R45: renamed from C33; value 10nF -> 1k; footprint Capacitor_SMD:C_0603_1608Metric -> Resistor_SMD:R_0603_1608Metric; symbol Device:C -> Device:R_US
- R46: renamed from R45; value 1k -> 3.9k
- renumbered R42 to R43
Connections:
- net +3V3: now also R42.1; no longer J10.1
- net GND: now also R46.2, C33.2; no longer R45.2
- net at C34.1, U14.10 (AIN1): now also C33.1, R44.1; no longer R45.1
- net at C35.1, U14.11 (AIN0): now also C34.2, R45.1; no longer R46.1
- net at U14.14 (~{DRDY}): now also R43.2; no longer J10.2
- net at U14.3 (~{RESET}): now also R42.2; no longer R43.2
- net at U14.6 (AIN3): now also J10.1 (Pin_1)
- net at C36.1, U14.9 (REFP): now also J10.4 (Pin_4), R46.1
- new net: J10.2 (Pin_2), R44.2
- new net: J10.3 (Pin_3), R45.2
Other:
- moved on the sheet: R43, R46

Commit message: KiCad schematic: INA239, ADS1220, SC18IS604 bridge, relay driver, test points
- system_current: INA237 -> INA239 (SPI, CS GPIO3) with the 49.9 ohm / 470 nF
  input filter, power LED and ALERT LED; VBUS shares the filtered IN- node.
- cold_head: ADS122C04 -> ADS1220 (SPI, CS GPIO44).
- i2c_bridge (new): SC18IS604 SPI-to-I2C bridge for the EMC2303, with a
  74LVC1G125 gating its MISO onto the shared bus.
- compressor_relay (new): GPIO16 high-side switch sharing one generator
  function with the amplifier REM switch.
- debug (new): about 40 test points and rail LEDs (the isolated rail LED
  returns to ISO_GND).
- ISO7741 -> ACS37800 SPI lines are straight wires (pins reordered on the
  symbol); USB_VBUS is one wire plus a naming label.
- Custom symbols for INA239, ADS1220, SC18IS604; datasheet rules 117 -> 162;
  GPIO map checks updated. ERC 0.

Co-Authored-By: Claude Sonnet 5.5 <noreply@anthropic.com>
Parts:
- removed C34: 100nF, Capacitor_SMD:C_0603_1608Metric, symbol Device:C
- removed R46: 3.9k, Resistor_SMD:R_0603_1608Metric, symbol Device:R_US
- removed U14: ADS122C04IPWR, Package_SO:TSSOP-16_4.4x5mm_P0.65mm, symbol cryocooler:ADS122C04IPWR
- added C31: 100nF, Capacitor_SMD:C_0603_1608Metric, symbol Device:C
- added C33: 10nF, Capacitor_SMD:C_0603_1608Metric, symbol Device:C
- added R41: 10k, Resistor_SMD:R_0603_1608Metric, symbol Device:R_US
- added U14: ADS1220IPW, Package_SO:TSSOP-16_4.4x5mm_P0.65mm, symbol cryocooler:ADS1220IPW
- C34: renamed from R44; value 1k -> 100nF; footprint Resistor_SMD:R_0603_1608Metric -> Capacitor_SMD:C_0603_1608Metric; symbol Device:R_US -> Device:C
- R40: renamed from C31; value 100nF -> 10k; footprint Capacitor_SMD:C_0603_1608Metric -> Resistor_SMD:R_0603_1608Metric; symbol Device:C -> Device:R_US
- R42: renamed from R43; value 10k -> 1k
- R43: renamed from C33; value 10nF -> 1k; footprint Capacitor_SMD:C_0603_1608Metric -> Resistor_SMD:R_0603_1608Metric; symbol Device:C -> Device:R_US
- R44: renamed from R45; value 1k -> 3.9k
- TP2: renamed from R42; value 10k -> ADS1220_DRDY; footprint Resistor_SMD:R_0603_1608Metric -> TestPoint:TestPoint_Pad_D1.5mm; symbol Device:R_US -> Connector:TestPoint
Connections:
- net +3V3: now also C31.1, R41.1, U14.12 (AVDD), U14.13 (DVDD); no longer R42.1, TP2.1
- net GND: now also R44.2, C31.2, C33.2, U14.3 (CLK), U14.4 (DGND), U14.5 (AVSS), U14.8 (REFN0); no longer R40.2, R43.2
- net at R43.1: now also C34.2, C35.1, U14.11 (AIN0/REFP1); no longer C34.1
- net at R44.1: now also C36.1, J10.4 (Pin_4), U14.9 (REFP0); no longer C35.1
- net at R42.2: now also J10.2 (Pin_2)
- net at J10.1 (Pin_1): now also U14.6 (AIN3/REFN1)
- net at J10.3 (Pin_3): now also R43.2; no longer R44.2
- new net: R41.2, TP2.1, U14.14 (~{DRDY})
- new net: C33.1, C34.1, R42.1, U14.10 (AIN1)
- new net ADS1220_CS: R40.2, U14.2 (~{CS})
- new net SPI_MISO: U14.15 (DOUT/~{DRDY})
- new net SPI_MOSI: U14.16 (DIN)
- new net SPI_SCK: U14.1 (SCLK)
Other:
- note added: "ADS1220 DECOUPLING CAPACITORS"
- note added: "PT1000 4-wire ratiometric: IDAC1 (AIN3) excites, AIN1/AIN0 sense, Rref (3.9k) on REFP0/REFN0. SPI mode 1 on the main bus (CS GPIO44), internal oscillator (CLK tied low). DRDY is not wired to the MCU."
- note removed: "ADS122C04 DECOUPLING CAPACITORS"
- note removed: "PT1000 4-wire ratiometric: IDAC1 (AIN3) excites, AIN1/AIN0 sense, Rref (3.9k) on REFP/REFN. I2C 0x45 (A0=A1=DVDD)."
- moved on the sheet: R42, R44

Commit message: Add per-section supply jumpers, 8-pin IMU header and connector pin labels
- Four 1.27 mm 2-pin jumpers (JP1-JP4), each with a rail-on LED, cut the
  supply of one section for debugging: signal generator +3V3, +-15V
  generator +5V in, isolated amp-current supply +5V in, and a shared
  +3V3 net for the cooling chips (EMC2303, RTD ADC, I2C bridge).
- J14 is now an 8-pin JST XH in the Adafruit LSM6DSOX pad order
  (VIN, GND, SCL, SDA, DO, CS, I1, I2); firmware pin comments updated.
- Pin-function labels beside every connector, "RAILS ±15V" box title.
- Board re-placed and re-routed (130 x 110 mm); DRC 0 errors, 0 unconnected,
  ERC 0, 173 datasheet rules pass. BOM, READMEs, Gerbers and renders
  regenerated; link_usb_vbus.py now adapts to the routed layout.

Co-Authored-By: Claude Sonnet 5.5 <noreply@anthropic.com>
Connections:
- net +3V3: no longer C31.1, C32.1, U14.12 (AVDD), U14.13 (DVDD)
- new net +3V3_COOL: C31.1, C32.1, U14.12 (AVDD), U14.13 (DVDD)

Commit message: Split cooling into Water Cooling and Cold Head Temp sections, each with a supply jumper and LED
Water Cooling (EMC2303, SC18IS604 bridge, NTC, fan/pump/flow) sits behind JP4
on +3V3_COOL together with its pull-ups. Cold Head Temp (ADS1220, PT1000) gets
a new jumper JP5 and LED D22 on +3V3_CH. JP2 is relabelled for the +-15V rails
and moved into the RAILS +-15V box. PCB regenerated with two silk boxes, routed,
leftovers finished with a grid router; board render added to the main README.

Co-Authored-By: Claude Sonnet 5.5 <noreply@anthropic.com>
Connections:
- net +3V3: no longer R41.1
- net +3V3_COOL renamed +3V3_CH
- net +3V3_CH: now also R41.1
Other:
- title: Cold Head -> Cold Head Temp

Commit message: Replace the ±15 V LDOs with one LT3097 and add a power-good interlock
- rails_15v: ADP7142 + ADP7182 replaced by one LT3097 (±14.7 V, 147 k SET
  resistors); the ADP5071 output caps are now 22 uF / 50 V and double as the
  LT3097 inputs. PGP / PGN make the PG_15V node (fed from +15 V, so it reads
  0 V if a rail is missing).
- amp_control: a series BSS138 (Q9) gated by PG_15V blocks AMP_REM unless
  both rails are good. New power_good sheet: LED (D23) and the active-low
  PG_15V_N flag on GPIO43 (PG_15V_N_PIN).
- Tooling: LT3097 symbol, footprint and 3D envelope; datasheet rules (191),
  GPIO check, BOM tables, floor plan, PAD_BRIDGES and pre-placed GND vias in
  gen_pcb.py, new fix_route.py for post-route clean-up.
- Board regenerated and routed with Freerouting 2.5.0: DRC 0 unconnected,
  0 schematic-parity issues, no copper violations. Gerbers, JLCPCB zip,
  renders, BOM, CPL and schematic PDF regenerated.

Co-Authored-By: Claude Sonnet 5.5 <noreply@anthropic.com>
Parts:
- removed C31, C34: 100nF, Capacitor_SMD:C_0603_1608Metric, symbol Device:C
- removed TP2: ADS1220_DRDY, TestPoint:TestPoint_Pad_D1.5mm, symbol Connector:TestPoint
- added C32: 1uF, Capacitor_SMD:C_0805_2012Metric, symbol Device:C
- added C33, C35: 10nF, Capacitor_SMD:C_0603_1608Metric, symbol Device:C
- C31: renamed from C32; value 1uF -> 100nF; footprint Capacitor_SMD:C_0805_2012Metric -> Capacitor_SMD:C_0603_1608Metric
- C34: renamed from R43; value 1k -> 100nF; footprint Resistor_SMD:R_0603_1608Metric -> Capacitor_SMD:C_0603_1608Metric; symbol Device:R_US -> Device:C
- J10: renamed from R42; value 1k -> RTD PT1000 4-wire; footprint Resistor_SMD:R_0603_1608Metric -> Connector_JST:JST_XH_B4B-XH-A_1x04_P2.50mm_Vertical; symbol Device:R_US -> Connector_Generic:Conn_01x04
- R42: renamed from C33; value 10nF -> 1k; footprint Capacitor_SMD:C_0603_1608Metric -> Resistor_SMD:R_0603_1608Metric; symbol Device:C -> Device:R_US
- R43: renamed from C35; value 10nF -> 1k; footprint Capacitor_SMD:C_0603_1608Metric -> Resistor_SMD:R_0603_1608Metric; symbol Device:C -> Device:R_US
- TP2: renamed from J10; value RTD PT1000 4-wire -> ADS1220_DRDY; footprint Connector_JST:JST_XH_B4B-XH-A_1x04_P2.50mm_Vertical -> TestPoint:TestPoint_Pad_D1.5mm; symbol Connector_Generic:Conn_01x04 -> Connector:TestPoint
Connections:
- net +3V3_CH: now also C32.1
- net GND: now also C32.2, C33.2, C35.2; no longer R42.2, R43.2
- net at R43.1, U14.11 (AIN0/REFP1): now also C34.2, C35.1; no longer C34.1
- net at C36.1, R44.1, U14.9 (REFP0): now also J10.4 (Pin_4); no longer TP2.4 (Pin_4)
- net at R41.2, U14.14 (~{DRDY}): now also TP2.1
- net at R42.1, U14.10 (AIN1): now also C34.1, C33.1; no longer J10.1
- net at U14.6 (AIN3/REFN1): now also J10.1 (Pin_1); no longer TP2.1 (Pin_1)
- net at J10.2 (Pin_2): now also R42.2; no longer TP2.2 (Pin_2)
- new net: J10.3 (Pin_3), R43.2
Other:
- moved on the sheet: C31
