File: hardware/kicad/sheets/imu.kicad_sch (KiCad schematic)
At the start: 5 parts, among them U23 LSM6DSOXTR

Commit message: Fixing the UUID issues
Parts:
- removed C70, C72: 100nF, Capacitor_SMD:C_0603_1608Metric, symbol Device:C
- removed C71: 10uF, Capacitor_SMD:C_0805_2012Metric, symbol Device:C
- removed R67: 10k, Resistor_SMD:R_0603_1608Metric, symbol Device:R_US
- removed U23: LSM6DSOXTR, Package_LGA:LGA-14_3x2.5mm_P0.5mm_LayoutBorder3x4y, symbol cryocooler:LSM6DSOXTR
- added C53, C55: 100nF, Capacitor_SMD:C_0603_1608Metric, symbol Device:C
- added C54: 10uF, Capacitor_SMD:C_0805_2012Metric, symbol Device:C
- added R56: 10k, Resistor_SMD:R_0603_1608Metric, symbol Device:R_US
- added U19: LSM6DSOXTR, Package_LGA:LGA-14_3x2.5mm_P0.5mm_LayoutBorder3x4y, symbol cryocooler:LSM6DSOXTR
Connections:
- net +3V3: now also C53.1, C54.1, C55.1, R56.1, U19.5 (VDDIO), U19.8 (VDD)
- net GND: now also C53.2, C54.2, C55.2, U19.2 (SDx), U19.3 (SCx), U19.6 (GND), U19.7 (GND)
- net IMU_CS: now also R56.2, U19.12 (~{CS})
- net IMU_INT1: now also U19.4 (INT1)
- net IMU_INT2: now also U19.9 (INT2)
- net SPI_MISO: now also U19.1 (SDO)
- net SPI_MOSI: now also U19.14 (SDI)
- net SPI_SCK: now also U19.13 (SPC)
