File: hardware/kicad/sheets/imu.kicad_sch (KiCad schematic)
At the start: 8 parts, among them J14 IMU LSM6DSOX module

Commit message: WIP: restructure PCB for the Phoenix UCS 125-87 housing
Work in progress, layout not finished: about 90 parts still do not fit
their sections and the board is not routed.

- Right-angle connectors: Phoenix MSTBA 2,5 / MC 1,5, JST XH side entry,
  Hirose DF13, Molex 505448-0871 (new footprint from the Molex drawing)
- Datasheet and product links on every symbol (tools/part_links.py)
- Test points so every IC has one on its own nets
- gen_pcb.py: 100 x 62 mm two-sided board, housing holes and restricted
  corners, ESP32 antenna notch, one section per sheet, board ID block,
  ESP32 pin names, pin-1 marks, blue mask
- Housing drawings in hardware/housing/

Co-Authored-By: Claude Opus 5.5 <noreply@anthropic.com>
Parts:
- removed J14: IMU LSM6DSOX module, Connector_JST:JST_XH_B8B-XH-A_1x08_P2.50mm_Vertical, symbol Connector_Generic:Conn_01x08
- removed R91: 100, Resistor_SMD:R_0603_1608Metric, symbol Device:R_US
- added R94, R95: 100, Resistor_SMD:R_0603_1608Metric, symbol Device:R_US
- J14: renamed from R90; value 100 -> IMU LSM6DSOX module; footprint Resistor_SMD:R_0603_1608Metric -> cryocooler:Molex_Micro-Lock_Plus_505448-0871_2x04_P1.25mm_Horizontal; symbol Device:R_US -> Connector_Generic:Conn_01x08; Product (none) -> https://www.molex.com/en-us/products/part-detail/5054480871
- R54: renamed from R95; value 100 -> 10k; Product (none) -> https://www.digikey.com/en/products/result?keywords=AR0603F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
- R90: renamed from R93; Product (none) -> https://www.digikey.com/en/products/result?keywords=AR0603F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
- R91: renamed from R54; value 10k -> 100; Product (none) -> https://www.digikey.com/en/products/result?keywords=AR0603F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
- R92: Product (none) -> https://www.digikey.com/en/products/result?keywords=AR0603F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
- R93: renamed from R94; Product (none) -> https://www.digikey.com/en/products/result?keywords=AR0603F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
Connections:
- net +3V3: now also J14.1 (Pin_1), R54.1; no longer R91.1
- net GND: now also J14.2 (Pin_2)
- net IMU_CS: now also R54.2, R93.1; no longer R90.1, R91.2
- net IMU_INT1: now also R94.1; no longer R93.1
- net IMU_INT2: now also R95.1; no longer R54.1
- net SPI_MOSI: now also R91.1
- net SPI_SCK: now also R90.1; no longer J14.1
- net at R93.2: now also J14.6 (Pin_6)
- net at R92.2: now also J14.5 (Pin_5)
- net at R90.2: now also J14.3 (Pin_3)
- new net: J14.4 (Pin_4), R91.2
- new net: J14.7 (Pin_7), R94.2
- new net: J14.8 (Pin_8), R95.2
Other:
- moved on the sheet: R54, R90, R91, R93

Commit message: Ground the M12 shield, order the ground loops, name the J14 cable parts
- J10: shielded symbol (Conn_01x04_Shielded); the M12 shield pin and its
  four shell legs are pad SH, tied to GND
- TP22-TP25: Keystone 5001 black miniature PC test points (KiCad
  TestPoint_Keystone_5000-5004 footprint, 1.02 mm hole per Keystone's
  drawing); now in the BOM, the bare pad test points stay out
- J14 BOM note: cable housing Molex 5054320801 with 505431 terminals, or
  tin pre-crimped leads 797581148 / 797581149 (from molex.com)

Only netlist change: GND gains J10 SH. DRC 0 errors, 0 unconnected, 0
schematic-parity issues; ERC 0; 193/193 datasheet rules.

Co-Authored-By: Claude Opus 5.5 <noreply@anthropic.com>
Parts:
- removed R90, R94: 100, Resistor_SMD:R_0603_1608Metric, symbol Device:R_US
- added R54: 10k, Resistor_SMD:R_0603_1608Metric, symbol Device:R_US
- added R95: 100, Resistor_SMD:R_0603_1608Metric, symbol Device:R_US
- R93: renamed from R54; value 10k -> 100; Product https://www.digikey.com/en/products/result?keywords=AR0603FR-0710KL -> https://www.digikey.com/en/products/result?keywords=AR0603FR-07100RL
- renumbered R91 to R90, R92 to R91, R93 to R92, R95 to R94
Connections:
- net +3V3: now also R54.1; no longer R93.1
- net IMU_CS: now also R93.1, R54.2; no longer R92.1, R93.2
- net IMU_INT1: now also R94.1
- net IMU_INT2: now also R95.1; no longer R94.1
- net SPI_MISO: now also R92.1; no longer R91.1
- net SPI_MOSI: now also R91.1; no longer R90.1
- net SPI_SCK: now also R90.1
- net at R92.2: now also J14.5 (Pin_5); no longer J14.6 (Pin_6)
- net at R91.2: now also J14.4 (Pin_4); no longer J14.5 (Pin_5)
- net at R90.2: now also J14.3 (Pin_3); no longer J14.4 (Pin_4)
- net at J14.7 (Pin_7): now also R94.2
- net at J14.8 (Pin_8): now also R95.2; no longer R94.2
- new net: J14.6 (Pin_6), R93.2
Other:
- moved on the sheet: R90, R91, R92, R93, R94
