File: hardware/kicad/sheets/rails_logic.kicad_sch (KiCad schematic)
At the start: 11 parts, among them U6 AP63205WU-7, U7 LD1117S33TR

Commit message: Fixing the UUID issues
Parts:
- removed C10: 10uF/25V, Capacitor_SMD:C_1206_3216Metric, symbol Device:C
- removed C11, C12, C17: 100nF, Capacitor_SMD:C_0603_1608Metric, symbol Device:C
- removed C13, C14: 22uF/10V, Capacitor_SMD:C_1206_3216Metric, symbol Device:C
- removed C15: 10uF, Capacitor_SMD:C_0805_2012Metric, symbol Device:C
- removed C16: 22uF, Capacitor_Tantalum_SMD:CP_EIA-3528-21_Kemet-B, symbol Device:C_Polarized
- removed U6: AP63205WU-7, Package_TO_SOT_SMD:TSOT-23-6, symbol Regulator_Switching:AP63205WU
- removed U7: LD1117S33TR, Package_TO_SOT_SMD:SOT-223-3_TabPin2, symbol Regulator_Linear:LD1117S33TR_SOT223
- added C37: 10uF/25V, Capacitor_SMD:C_1206_3216Metric, symbol Device:C
- added C38, C39, C44: 100nF, Capacitor_SMD:C_0603_1608Metric, symbol Device:C
- added C40, C41: 22uF/10V, Capacitor_SMD:C_1206_3216Metric, symbol Device:C
- added C42: 10uF, Capacitor_SMD:C_0805_2012Metric, symbol Device:C
- added C43: 22uF, Capacitor_Tantalum_SMD:CP_EIA-3528-21_Kemet-B, symbol Device:C_Polarized
- added U15: AP63205WU-7, Package_TO_SOT_SMD:TSOT-23-6, symbol Regulator_Switching:AP63205WU
- added U16: LD1117S33TR, Package_TO_SOT_SMD:SOT-223-3_TabPin2, symbol Regulator_Linear:LD1117S33TR_SOT223
Connections:
- net +12V: now also C37.1, C38.1, U15.2 (EN), U15.3 (IN)
- net +3V3: now also C43.1, C44.1, U16.2 (VO)
- net +5V: now also C40.1, C41.1, C42.1, U15.1 (FB), U16.3 (VI)
- net GND: now also C37.2, C38.2, C40.2, C41.2, C42.2, C43.2, C44.2, U15.4 (GND), U16.1 (GND)
- net at L1.1: now also C39.1, U15.5 (SW)
- new net: C39.2, U15.6 (BST)
