File: hardware/kicad/sheets/rails_logic.kicad_sch (KiCad schematic)
At the start: 11 parts, among them U15 AP63205WU-7, U16 LD1117S33TR

Commit message: Put supply pins on top and grounds on the bottom of IC symbols; flake8-clean Python
Schematic: re-laid out pins on U2, U3, U6, U7, U11, U14, U17-U20, U22-U24
and PS1 (supply on top, ground/strap pins on the bottom edge) via custom
`cryocooler:` symbols (make_lib.from_stock) and a gnd_bus helper; U18/U2
use mirroring instead of a 180 degree rotation. Nets are unchanged (ERC 0,
117/117 datasheet rules, PCB nets still match). Text placement now shows
every power-symbol name, avoids wires, and uses a realistic character width.

Python: black -l 79 -S plus manual wrapping so hardware/kicad and scripts/
pass flake8; add .flake8.

Co-Authored-By: Claude Sonnet 5.5 <noreply@anthropic.com>
Parts:
- removed C38: 100nF, Capacitor_SMD:C_0603_1608Metric, symbol Device:C
- removed C40: 22uF/10V, Capacitor_SMD:C_1206_3216Metric, symbol Device:C
- removed C43: 22uF, Capacitor_Tantalum_SMD:CP_EIA-3528-21_Kemet-B, symbol Device:C_Polarized
- added C39: 100nF, Capacitor_SMD:C_0603_1608Metric, symbol Device:C
- added C41: 22uF/10V, Capacitor_SMD:C_1206_3216Metric, symbol Device:C
- added U15: AP63205WU-7, Package_TO_SOT_SMD:TSOT-23-6, symbol Regulator_Switching:AP63205WU
- C38: renamed from U15; value AP63205WU-7 -> 100nF; footprint Package_TO_SOT_SMD:TSOT-23-6 -> Capacitor_SMD:C_0603_1608Metric; symbol Regulator_Switching:AP63205WU -> Device:C
- C40: renamed from C39; value 100nF -> 22uF/10V; footprint Capacitor_SMD:C_0603_1608Metric -> Capacitor_SMD:C_1206_3216Metric
- C42: renamed from U16; value LD1117S33TR -> 10uF; footprint Package_TO_SOT_SMD:SOT-223-3_TabPin2 -> Capacitor_SMD:C_0805_2012Metric; symbol Regulator_Linear:LD1117S33TR_SOT223 -> Device:C
- C43: renamed from C42; value 10uF -> 22uF; footprint Capacitor_SMD:C_0805_2012Metric -> Capacitor_Tantalum_SMD:CP_EIA-3528-21_Kemet-B; symbol Device:C -> Device:C_Polarized
- U16: renamed from C41; value 22uF/10V -> LD1117S33TR; footprint Capacitor_SMD:C_1206_3216Metric -> Package_TO_SOT_SMD:SOT-223-3_TabPin2; symbol Device:C -> Regulator_Linear:LD1117S33TR_SOT223
Connections:
- net +12V: now also C38.1, U15.2 (EN), U15.3 (IN); no longer C38.2 (EN), C38.3 (IN)
- net +3V3: now also C43.1, U16.2 (VO); no longer C42.2 (VO)
- net +5V: now also C40.1, C42.1, U16.3 (VI), C41.1, U15.1 (FB); no longer C38.1 (FB), C42.3 (VI), C43.1, U16.1
- net GND: now also C38.2, C40.2, C42.2, U16.1 (GND), C41.2, U15.4 (GND); no longer C38.4 (GND), C42.1 (GND), U16.2
- new net: C39.1, L1.1, U15.5 (SW)
- new net: C39.2, U15.6 (BST)
Other:
- moved on the sheet: C40

Commit message: KiCad schematic: INA239, ADS1220, SC18IS604 bridge, relay driver, test points
- system_current: INA237 -> INA239 (SPI, CS GPIO3) with the 49.9 ohm / 470 nF
  input filter, power LED and ALERT LED; VBUS shares the filtered IN- node.
- cold_head: ADS122C04 -> ADS1220 (SPI, CS GPIO44).
- i2c_bridge (new): SC18IS604 SPI-to-I2C bridge for the EMC2303, with a
  74LVC1G125 gating its MISO onto the shared bus.
- compressor_relay (new): GPIO16 high-side switch sharing one generator
  function with the amplifier REM switch.
- debug (new): about 40 test points and rail LEDs (the isolated rail LED
  returns to ISO_GND).
- ISO7741 -> ACS37800 SPI lines are straight wires (pins reordered on the
  symbol); USB_VBUS is one wire plus a naming label.
- Custom symbols for INA239, ADS1220, SC18IS604; datasheet rules 117 -> 162;
  GPIO map checks updated. ERC 0.

Co-Authored-By: Claude Sonnet 5.5 <noreply@anthropic.com>
Parts:
- removed C38: 100nF, Capacitor_SMD:C_0603_1608Metric, symbol Device:C
- removed C40: 22uF/10V, Capacitor_SMD:C_1206_3216Metric, symbol Device:C
- removed C43: 22uF, Capacitor_Tantalum_SMD:CP_EIA-3528-21_Kemet-B, symbol Device:C_Polarized
- added C39: 100nF, Capacitor_SMD:C_0603_1608Metric, symbol Device:C
- added C41: 22uF/10V, Capacitor_SMD:C_1206_3216Metric, symbol Device:C
- added U15: AP63205WU-7, Package_TO_SOT_SMD:TSOT-23-6, symbol Regulator_Switching:AP63205WU
- C38: renamed from U15; value AP63205WU-7 -> 100nF; footprint Package_TO_SOT_SMD:TSOT-23-6 -> Capacitor_SMD:C_0603_1608Metric; symbol Regulator_Switching:AP63205WU -> Device:C
- C40: renamed from C39; value 100nF -> 22uF/10V; footprint Capacitor_SMD:C_0603_1608Metric -> Capacitor_SMD:C_1206_3216Metric
- C42: renamed from U16; value LD1117S33TR -> 10uF; footprint Package_TO_SOT_SMD:SOT-223-3_TabPin2 -> Capacitor_SMD:C_0805_2012Metric; symbol Regulator_Linear:LD1117S33TR_SOT223 -> Device:C
- C43: renamed from C42; value 10uF -> 22uF; footprint Capacitor_SMD:C_0805_2012Metric -> Capacitor_Tantalum_SMD:CP_EIA-3528-21_Kemet-B; symbol Device:C -> Device:C_Polarized
- U16: renamed from C41; value 22uF/10V -> LD1117S33TR; footprint Capacitor_SMD:C_1206_3216Metric -> Package_TO_SOT_SMD:SOT-223-3_TabPin2; symbol Device:C -> Regulator_Linear:LD1117S33TR_SOT223
Connections:
- net +12V: now also C38.1, U15.2 (EN), U15.3 (IN); no longer C38.2 (EN), C38.3 (IN)
- net +3V3: now also C43.1, U16.2 (VO); no longer C42.2 (VO)
- net +5V: now also C40.1, C42.1, U16.3 (VI), C41.1, U15.1 (FB); no longer C38.1 (FB), C42.3 (VI), C43.1, U16.1
- net GND: now also C38.2, C40.2, C42.2, U16.1 (GND), C41.2, U15.4 (GND); no longer C38.4 (GND), C42.1 (GND), U16.2
- new net: C39.1, L1.1, U15.5 (SW)
- new net: C39.2, U15.6 (BST)
Other:
- moved on the sheet: C40
