File: hardware/kicad/sheets/rails_logic.kicad_sch (KiCad schematic)
At the start: 11 parts, among them U15 AP63205WU-7, U16 LD1117S33TR

Commit message: Replace the ±15 V LDOs with one LT3097 and add a power-good interlock
- rails_15v: ADP7142 + ADP7182 replaced by one LT3097 (±14.7 V, 147 k SET
  resistors); the ADP5071 output caps are now 22 uF / 50 V and double as the
  LT3097 inputs. PGP / PGN make the PG_15V node (fed from +15 V, so it reads
  0 V if a rail is missing).
- amp_control: a series BSS138 (Q9) gated by PG_15V blocks AMP_REM unless
  both rails are good. New power_good sheet: LED (D23) and the active-low
  PG_15V_N flag on GPIO43 (PG_15V_N_PIN).
- Tooling: LT3097 symbol, footprint and 3D envelope; datasheet rules (191),
  GPIO check, BOM tables, floor plan, PAD_BRIDGES and pre-placed GND vias in
  gen_pcb.py, new fix_route.py for post-route clean-up.
- Board regenerated and routed with Freerouting 2.5.0: DRC 0 unconnected,
  0 schematic-parity issues, no copper violations. Gerbers, JLCPCB zip,
  renders, BOM, CPL and schematic PDF regenerated.

Co-Authored-By: Claude Sonnet 5.5 <noreply@anthropic.com>
Parts:
- removed C37: 10uF/25V, Capacitor_SMD:C_1206_3216Metric, symbol Device:C
- removed C39: 100nF, Capacitor_SMD:C_0603_1608Metric, symbol Device:C
- removed C43: 22uF, Capacitor_Tantalum_SMD:CP_EIA-3528-21_Kemet-B, symbol Device:C_Polarized
- added C38, C44: 100nF, Capacitor_SMD:C_0603_1608Metric, symbol Device:C
- added L1: SRN6045TA-4R7M, Inductor_SMD:L_Bourns_SRN6045TA, symbol Device:L
- C37: renamed from C38; value 100nF -> 10uF/25V; footprint Capacitor_SMD:C_0603_1608Metric -> Capacitor_SMD:C_1206_3216Metric
- C39: renamed from L1; value SRN6045TA-4R7M -> 100nF; footprint Inductor_SMD:L_Bourns_SRN6045TA -> Capacitor_SMD:C_0603_1608Metric; symbol Device:L -> Device:C
- C43: renamed from C44; value 100nF -> 22uF; footprint Capacitor_SMD:C_0603_1608Metric -> Capacitor_Tantalum_SMD:CP_EIA-3528-21_Kemet-B; symbol Device:C -> Device:C_Polarized
Connections:
- net +12V: now also C38.1
- net +3V3: now also C44.1
- net +5V: now also L1.2; no longer C39.2
- net GND: now also C38.2, C44.2
- net at C39.1, U15.5 (SW): now also L1.1
- net at U15.6 (BST): now also C39.2
Other:
- moved on the sheet: C37

Commit message: WIP: restructure PCB for the Phoenix UCS 125-87 housing
Work in progress, layout not finished: about 90 parts still do not fit
their sections and the board is not routed.

- Right-angle connectors: Phoenix MSTBA 2,5 / MC 1,5, JST XH side entry,
  Hirose DF13, Molex 505448-0871 (new footprint from the Molex drawing)
- Datasheet and product links on every symbol (tools/part_links.py)
- Test points so every IC has one on its own nets
- gen_pcb.py: 100 x 62 mm two-sided board, housing holes and restricted
  corners, ESP32 antenna notch, one section per sheet, board ID block,
  ESP32 pin names, pin-1 marks, blue mask
- Housing drawings in hardware/housing/

Co-Authored-By: Claude Opus 5.5 <noreply@anthropic.com>
Parts:
- removed C39: 100nF, Capacitor_SMD:C_0603_1608Metric, symbol Device:C
- removed C41: 22uF/10V, Capacitor_SMD:C_1206_3216Metric, symbol Device:C
- removed U15: AP63205WU-7, Package_TO_SOT_SMD:TSOT-23-6, symbol Regulator_Switching:AP63205WU
- added C38: 100nF, Capacitor_SMD:C_0603_1608Metric, symbol Device:C
- added C40: 22uF/10V, Capacitor_SMD:C_1206_3216Metric, symbol Device:C
- added C43: 22uF, Capacitor_Tantalum_SMD:CP_EIA-3528-21_Kemet-B, symbol Device:C_Polarized
- C37: Product (none) -> https://www.digikey.com/en/products/result?keywords=C3216X5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
- C39: renamed from C40; value 22uF/10V -> 100nF; footprint Capacitor_SMD:C_1206_3216Metric -> Capacitor_SMD:C_0603_1608Metric; Product (none) -> https://www.digikey.com/en/products/result?keywords=C0603C1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
- C41: renamed from U16; value LD1117S33TR -> 22uF/10V; footprint Package_TO_SOT_SMD:SOT-223-3_TabPin2 -> Capacitor_SMD:C_1206_3216Metric; symbol Regulator_Linear:LD1117S33TR_SOT223 -> Device:C; Product (none) -> https://www.digikey.com/en/products/result?keywords=CL31A22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
- C42: renamed from C43; value 22uF -> 10uF; footprint Capacitor_Tantalum_SMD:CP_EIA-3528-21_Kemet-B -> Capacitor_SMD:C_0805_2012Metric; symbol Device:C_Polarized -> Device:C; Product (none) -> https://www.digikey.com/en/products/result?keywords=CL21A10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
- C44: Product (none) -> https://www.digikey.com/en/products/result?keywords=C0603C1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
- L1: Product (none) -> https://www.digikey.com/en/products/result?keywords=SRP6050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
- U15: renamed from C38; value 100nF -> AP63205WU-7; footprint Capacitor_SMD:C_0603_1608Metric -> Package_TO_SOT_SMD:TSOT-23-6; symbol Device:C -> Regulator_Switching:AP63205WU; Product (none) -> https://www.digikey.com/en/products/result?keywords=AP63205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
- U16: renamed from C42; value 10uF -> LD1117S33TR; footprint Capacitor_SMD:C_0805_2012Metric -> Package_TO_SOT_SMD:SOT-223-3_TabPin2; symbol Device:C -> Regulator_Linear:LD1117S33TR_SOT223; Product (none) -> https://www.digikey.com/en/products/result?keywords=LD1117S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
Connections:
- net +12V: now also U15.2 (EN), U15.3 (IN), C38.1; no longer U15.1
- net +3V3: now also U16.2 (VO), C43.1; no longer C41.2 (VO), C42.1
- net +5V: now also C41.1, C42.1, U15.1 (FB), U16.3 (VI), C40.1; no longer C39.1, C41.3 (VI), U16.1
- net GND: now also C41.2, U15.4 (GND), U16.1 (GND), C38.2, C40.2, C43.2; no longer C39.2, C41.1 (GND), U15.2, U16.2
- net at L1.1: now also C39.1, U15.5 (SW)
- new net: C39.2, U15.6 (BST)
Other:
- moved on the sheet: C39

Commit message: Ground the M12 shield, order the ground loops, name the J14 cable parts
- J10: shielded symbol (Conn_01x04_Shielded); the M12 shield pin and its
  four shell legs are pad SH, tied to GND
- TP22-TP25: Keystone 5001 black miniature PC test points (KiCad
  TestPoint_Keystone_5000-5004 footprint, 1.02 mm hole per Keystone's
  drawing); now in the BOM, the bare pad test points stay out
- J14 BOM note: cable housing Molex 5054320801 with 505431 terminals, or
  tin pre-crimped leads 797581148 / 797581149 (from molex.com)

Only netlist change: GND gains J10 SH. DRC 0 errors, 0 unconnected, 0
schematic-parity issues; ERC 0; 193/193 datasheet rules.

Co-Authored-By: Claude Opus 5.5 <noreply@anthropic.com>
Parts:
- removed C37: 10uF/25V, Capacitor_SMD:C_1206_3216Metric, symbol Device:C
- removed C39: 100nF, Capacitor_SMD:C_0603_1608Metric, symbol Device:C
- removed C43: 22uF, Capacitor_Tantalum_SMD:CP_EIA-3528-21_Kemet-B, symbol Device:C_Polarized
- added C38, C44: 100nF, Capacitor_SMD:C_0603_1608Metric, symbol Device:C
- added L1: SRN6045TA-4R7M, Inductor_SMD:L_Bourns_SRN6045TA, symbol Device:L
- C37: renamed from C38; value 100nF -> 10uF/25V; footprint Capacitor_SMD:C_0603_1608Metric -> Capacitor_SMD:C_1206_3216Metric; Product https://www.digikey.com/en/products/result?keywords=C0603C1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 -> https://www.digikey.com/en/products/result?keywords=C3216X5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
- C39: renamed from L1; value SRN6045TA-4R7M -> 100nF; footprint Inductor_SMD:L_Bourns_SRN6045TA -> Capacitor_SMD:C_0603_1608Metric; symbol Device:L -> Device:C; Product https://www.digikey.com/en/products/result?keywords=SRP6050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 -> https://www.digikey.com/en/products/result?keywords=C0603C1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
- C43: renamed from C44; value 100nF -> 22uF; footprint Capacitor_SMD:C_0603_1608Metric -> Capacitor_Tantalum_SMD:CP_EIA-3528-21_Kemet-B; symbol Device:C -> Device:C_Polarized; Product https://www.digikey.com/en/products/result?keywords=C0603C1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 -> https://www.digikey.com/en/products/result?keywords=T491B22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
Connections:
- net +12V: now also C38.1
- net +3V3: now also C44.1
- net +5V: now also L1.2; no longer C39.2
- net GND: now also C38.2, C44.2
- net at C39.1, U15.5 (SW): now also L1.1
- net at U15.6 (BST): now also C39.2
Other:
- moved on the sheet: C37
