File: hardware/kicad/sheets/rails_15v.kicad_sch (KiCad schematic)
At the start: 31 parts, among them U20 ADP5071AREZ, U21 ADP7142AUJZ, U22 ADP7182AUJZ

Commit message: Move the IMU off-board (J14) and add labelled module boxes to the PCB
The LSM6DSOX is now the Adafruit breakout (product 4438) mounted on the
cryocooler and cabled to a 10-pin JST XH header (J14) over the shared SPI
bus. U19 and its capacitors are gone; J14 and six 100 R series resistors
are added, and every other reference number is unchanged.

PCB (130 x 110 mm, was 130 x 100):
- one outlined, labelled silkscreen box per module (pcbfloorplan.py); the
  placer keeps parts inside their box and reserves a label pocket beside
  every part so each label sits next to its own part
- box 3D models for U3, L2, L3, F1 and PS1, whose library models are missing
- re-routed; DRC 0 errors, 0 unconnected; back logo recentred
- gen_pcb.py texts redoes the silkscreen on a routed board

Firmware: SPI clock constant for the module, comments updated; ambient
temperature now reads the cooler-body IMU temperature.

Docs, BOM and fabrication files regenerated.

Co-Authored-By: Claude Sonnet 5.5 <noreply@anthropic.com>
Parts:
- removed C56, C57: 10uF, Capacitor_SMD:C_0805_2012Metric, symbol Device:C
- removed D5, D6: DFLS240, Diode_SMD:D_PowerDI-123, symbol Device:D_Schottky
- removed R60: 118k, Resistor_SMD:R_0603_1608Metric, symbol Device:R_US
- removed R61: 115k, Resistor_SMD:R_0603_1608Metric, symbol Device:R_US
- removed R63: 113k, Resistor_SMD:R_0603_1608Metric, symbol Device:R_US
- removed R64: 10k, Resistor_SMD:R_0603_1608Metric, symbol Device:R_US
- added C59: 47nF, Capacitor_SMD:C_1206_3216Metric, symbol Device:C
- added C62: 10uF/50V, Capacitor_SMD:C_1210_3225Metric, symbol Device:C
- added C64: 1uF, Capacitor_SMD:C_0805_2012Metric, symbol Device:C
- added C66, C69: 4.7uF/25V, Capacitor_SMD:C_1206_3216Metric, symbol Device:C
- added C68: 100pF, Capacitor_SMD:C_1206_3216Metric, symbol Device:C
- added L2: SRN8040TA-3R3M, Inductor_SMD:L_Bourns_SRN8040TA, symbol Device:L
- added R59: 2.55M, Resistor_SMD:R_0603_1608Metric, symbol Device:R_US
- C56: renamed from R55; value 5.6k -> 10uF; footprint Resistor_SMD:R_0603_1608Metric -> Capacitor_SMD:C_0805_2012Metric; symbol Device:R_US -> Device:C
- C57: renamed from C59; value 47nF -> 10uF; footprint Capacitor_SMD:C_1206_3216Metric -> Capacitor_SMD:C_0805_2012Metric
- C60: renamed from C61; value 68nF -> 1uF; footprint Capacitor_SMD:C_1206_3216Metric -> Capacitor_SMD:C_0805_2012Metric
- C61: renamed from L2; value SRN8040TA-3R3M -> 68nF; footprint Inductor_SMD:L_Bourns_SRN8040TA -> Capacitor_SMD:C_1206_3216Metric; symbol Device:L -> Device:C
- D5: renamed from R57; value 2.67M -> DFLS240; footprint Resistor_SMD:R_0603_1608Metric -> Diode_SMD:D_PowerDI-123; symbol Device:R_US -> Device:D_Schottky
- D6: renamed from R59; value 2.55M -> DFLS240; footprint Resistor_SMD:R_0603_1608Metric -> Diode_SMD:D_PowerDI-123; symbol Device:R_US -> Device:D_Schottky
- R55: renamed from C60; value 1uF -> 5.6k; footprint Capacitor_SMD:C_0805_2012Metric -> Resistor_SMD:R_0603_1608Metric; symbol Device:C -> Device:R_US
- R57: renamed from C62; value 10uF/50V -> 2.67M; footprint Capacitor_SMD:C_1210_3225Metric -> Resistor_SMD:R_0603_1608Metric; symbol Device:C -> Device:R_US
- R60: renamed from C64; value 1uF -> 118k; footprint Capacitor_SMD:C_0805_2012Metric -> Resistor_SMD:R_0603_1608Metric; symbol Device:C -> Device:R_US
- R61: renamed from C66; value 4.7uF/25V -> 115k; footprint Capacitor_SMD:C_1206_3216Metric -> Resistor_SMD:R_0603_1608Metric; symbol Device:C -> Device:R_US
- R63: renamed from C68; value 100pF -> 113k; footprint Capacitor_SMD:C_1206_3216Metric -> Resistor_SMD:R_0603_1608Metric; symbol Device:C -> Device:R_US
- R64: renamed from C69; value 4.7uF/25V -> 10k; footprint Capacitor_SMD:C_1206_3216Metric -> Resistor_SMD:R_0603_1608Metric; symbol Device:C -> Device:R_US
Connections:
- net +15V: now also C66.1
- net +16V5: now also C62.1
- net +5V: now also C56.1, C57.1
- net -15V: now also C68.1, C69.1; no longer R64.1
- net -16V5: now also D6.2 (A), R59.1; no longer D6.1
- net GND: now also C56.2, C61.2, C59.2, C62.2, C64.2, C66.2, C69.2; no longer R55.2, R57.2, R60.2, R61.2
- net at R60.1: now also U20.13 (FB2), R59.2; no longer U20.14 (VREF)
- net at R63.2, U22.4 (ADJ): now also R64.1, C68.2
- net at L3.1, U20.20 (SW2): now also D6.1 (K)
- net at U20.16 (VREG), U20.5 (SEQ): now also C60.1; no longer R55.1
- net at R56.1: now also C61.1; no longer C60.1
- net at U20.3 (INBK): now also L2.1; no longer C61.1
- net at U20.2 (SW1): now also D5.2 (A), L2.2; no longer C61.2
- net at R58.1, U20.7 (FB1): now also R57.2; no longer D5.2
- net at U20.8 (COMP1): now also R55.2; no longer C56.2
- net at R62.1, U21.4 (SENSE/ADJ): now also R61.2
- new net: C59.1, R55.1
- new net: C64.1, R60.2, U20.14 (VREF)
Other:
- moved on the sheet: C57, C60

Commit message: Add per-section supply jumpers, 8-pin IMU header and connector pin labels
- Four 1.27 mm 2-pin jumpers (JP1-JP4), each with a rail-on LED, cut the
  supply of one section for debugging: signal generator +3V3, +-15V
  generator +5V in, isolated amp-current supply +5V in, and a shared
  +3V3 net for the cooling chips (EMC2303, RTD ADC, I2C bridge).
- J14 is now an 8-pin JST XH in the Adafruit LSM6DSOX pad order
  (VIN, GND, SCL, SDA, DO, CS, I1, I2); firmware pin comments updated.
- Pin-function labels beside every connector, "RAILS ±15V" box title.
- Board re-placed and re-routed (130 x 110 mm); DRC 0 errors, 0 unconnected,
  ERC 0, 173 datasheet rules pass. BOM, READMEs, Gerbers and renders
  regenerated; link_usb_vbus.py now adapts to the routed layout.

Co-Authored-By: Claude Sonnet 5.5 <noreply@anthropic.com>
Parts:
- removed C65, C67: 4.7uF/25V, Capacitor_SMD:C_1206_3216Metric, symbol Device:C
- removed C68: 100pF, Capacitor_SMD:C_1206_3216Metric, symbol Device:C
- removed D6: DFLS240, Diode_SMD:D_PowerDI-123, symbol Device:D_Schottky
- removed R55: 5.6k, Resistor_SMD:R_0603_1608Metric, symbol Device:R_US
- removed R56: 12k, Resistor_SMD:R_0603_1608Metric, symbol Device:R_US
- added C56, C57: 10uF, Capacitor_SMD:C_0805_2012Metric, symbol Device:C
- added R58: 137k, Resistor_SMD:R_0603_1608Metric, symbol Device:R_US
- added R59: 2.55M, Resistor_SMD:R_0603_1608Metric, symbol Device:R_US
- added R62, R64: 10k, Resistor_SMD:R_0603_1608Metric, symbol Device:R_US
- C58: renamed from C56; value 10uF -> 100nF; footprint Capacitor_SMD:C_0805_2012Metric -> Capacitor_SMD:C_0603_1608Metric
- C59: renamed from C58; value 100nF -> 47nF; footprint Capacitor_SMD:C_0603_1608Metric -> Capacitor_SMD:C_1206_3216Metric
- C60: renamed from C59; value 47nF -> 1uF; footprint Capacitor_SMD:C_1206_3216Metric -> Capacitor_SMD:C_0805_2012Metric
- C62: renamed from R58; value 137k -> 10uF/50V; footprint Resistor_SMD:R_0603_1608Metric -> Capacitor_SMD:C_1210_3225Metric; symbol Device:R_US -> Device:C
- C63: renamed from R59; value 2.55M -> 10uF/50V; footprint Resistor_SMD:R_0603_1608Metric -> Capacitor_SMD:C_1210_3225Metric; symbol Device:R_US -> Device:C
- C64: renamed from C63; value 10uF/50V -> 1uF; footprint Capacitor_SMD:C_1210_3225Metric -> Capacitor_SMD:C_0805_2012Metric
- C65: renamed from U21; value ADP7142AUJZ -> 4.7uF/25V; footprint Package_TO_SOT_SMD:TSOT-23-5 -> Capacitor_SMD:C_1206_3216Metric; symbol Regulator_Linear:ADP7142AUJZ -> Device:C
- C66: renamed from R62; value 10k -> 4.7uF/25V; footprint Resistor_SMD:R_0603_1608Metric -> Capacitor_SMD:C_1206_3216Metric; symbol Device:R_US -> Device:C
- C67: renamed from U22; value ADP7182AUJZ -> 4.7uF/25V; footprint Package_TO_SOT_SMD:TSOT-23-5 -> Capacitor_SMD:C_1206_3216Metric; symbol cryocooler:ADP7182AUJZ -> Device:C
- C68: renamed from R64; value 10k -> 100pF; footprint Resistor_SMD:R_0603_1608Metric -> Capacitor_SMD:C_1206_3216Metric; symbol Device:R_US -> Device:C
- D6: renamed from L3; value SRN8040TA-6R8M -> DFLS240; footprint Inductor_SMD:L_Bourns_SRN8040TA -> Diode_SMD:D_PowerDI-123; symbol Device:L -> Device:D_Schottky
- L3: renamed from C62; value 10uF/50V -> SRN8040TA-6R8M; footprint Capacitor_SMD:C_1210_3225Metric -> Inductor_SMD:L_Bourns_SRN8040TA; symbol Device:C -> Device:L
- R55: renamed from C57; value 10uF -> 5.6k; footprint Capacitor_SMD:C_0805_2012Metric -> Resistor_SMD:R_0603_1608Metric; symbol Device:C -> Device:R_US
- R56: renamed from C60; value 1uF -> 12k; footprint Capacitor_SMD:C_0805_2012Metric -> Resistor_SMD:R_0603_1608Metric; symbol Device:C -> Device:R_US
- U21: renamed from C64; value 1uF -> ADP7142AUJZ; footprint Capacitor_SMD:C_0805_2012Metric -> Package_TO_SOT_SMD:TSOT-23-5; symbol Device:C -> Regulator_Linear:ADP7142AUJZ
- U22: renamed from C66; value 4.7uF/25V -> ADP7182AUJZ; footprint Capacitor_SMD:C_1206_3216Metric -> Package_TO_SOT_SMD:TSOT-23-5; symbol Device:C -> cryocooler:ADP7182AUJZ
Connections:
- net +15V: now also C66.1, U21.5 (VOUT); no longer C65.5 (VOUT), U22.1
- net +16V5: now also C62.1, U21.1 (VIN), U21.3 (EN); no longer C65.3 (EN), L3.1
- net -15V: now also C68.1, U22.5 (VOUT); no longer C67.5 (VOUT)
- net -16V5: now also C67.1, D6.2 (A), U22.2 (VIN), U22.3 (EN), R59.1; no longer C64.1, C67.2 (VIN), C67.3 (EN)
- net GND: now also C63.2, C67.2, U22.1 (GND), C56.2, C57.2, R58.2, R62.2, R64.2; no longer C67.1 (GND), C68.2, D6.2, R55.2, R56.2, U22.2
- net at C60.1: now also U20.16 (VREG), U20.5 (SEQ)
- net at R60.1, U20.13 (FB2): now also R59.2; no longer C63.2
- net at R60.2, U20.14 (VREF): now also C64.1; no longer U21.1
- net at R57.2, U20.7 (FB1): now also R58.1; no longer C62.1
- net at U20.8 (COMP1): now also R55.2
- net at C61.1: now also R56.1
- net at U20.12 (COMP2): now also R56.2
- net at D6.1 (K), U20.20 (SW2): now also L3.1
- net +5V renamed +5V_PS15
- net +5V_PS15: now also C56.1, C57.1; no longer C59.1, R55.1
- new net: C68.2, R63.2, R64.1, U22.4 (ADJ)
- new net: C59.1, R55.1
- new net: R61.2, R62.1, U21.4 (SENSE/ADJ)
Other:
- moved on the sheet: C58, C59, C60, C64
