File: hardware/kicad/sheets/rails_15v.kicad_sch (KiCad schematic)
At the start: 31 parts, among them U20 ADP5071AREZ, U21 LT3097ADJC

Commit message: WIP: restructure PCB for the Phoenix UCS 125-87 housing
Work in progress, layout not finished: about 90 parts still do not fit
their sections and the board is not routed.

- Right-angle connectors: Phoenix MSTBA 2,5 / MC 1,5, JST XH side entry,
  Hirose DF13, Molex 505448-0871 (new footprint from the Molex drawing)
- Datasheet and product links on every symbol (tools/part_links.py)
- Test points so every IC has one on its own nets
- gen_pcb.py: 100 x 62 mm two-sided board, housing holes and restricted
  corners, ESP32 antenna notch, one section per sheet, board ID block,
  ESP32 pin names, pin-1 marks, blue mask
- Housing drawings in hardware/housing/

Co-Authored-By: Claude Opus 5.5 <noreply@anthropic.com>
Parts:
- removed C56, C57: 10uF, Capacitor_SMD:C_0805_2012Metric, symbol Device:C
- removed C65: 22uF/50V, Capacitor_SMD:C_1210_3225Metric, symbol Device:C
- removed D5, D6: DFLS240, Diode_SMD:D_PowerDI-123, symbol Device:D_Schottky
- removed R60: 118k, Resistor_SMD:R_0603_1608Metric, symbol Device:R_US
- removed R61, R63: 432k, Resistor_SMD:R_0603_1608Metric, symbol Device:R_US
- added C59: 47nF, Capacitor_SMD:C_1206_3216Metric, symbol Device:C
- added C62: 22uF/50V, Capacitor_SMD:C_1210_3225Metric, symbol Device:C
- added C64: 1uF, Capacitor_SMD:C_0805_2012Metric, symbol Device:C
- added C68: 1uF/50V, Capacitor_SMD:C_1206_3216Metric, symbol Device:C
- added L2: SRP7050TA-3R3M, cryocooler:L_Bourns_SRP7050TA, symbol Device:L
- added R59: 2.55M, Resistor_SMD:R_0603_1608Metric, symbol Device:R_US
- added R62, R64: 147k, Resistor_SMD:R_0603_1608Metric, symbol Device:R_US
- C56: renamed from R55; value 5.6k -> 10uF; footprint Resistor_SMD:R_0603_1608Metric -> Capacitor_SMD:C_0805_2012Metric; symbol Device:R_US -> Device:C; Product (none) -> https://www.digikey.com/en/products/result?keywords=CL21A10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
- C57: renamed from C59; value 47nF -> 10uF; footprint Capacitor_SMD:C_1206_3216Metric -> Capacitor_SMD:C_0805_2012Metric; Product (none) -> https://www.digikey.com/en/products/result?keywords=CL21A10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
- C58: Product (none) -> https://www.digikey.com/en/products/result?keywords=C0603C1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
- C60: renamed from C61; value 68nF -> 1uF; footprint Capacitor_SMD:C_1206_3216Metric -> Capacitor_SMD:C_0805_2012Metric; Product (none) -> https://www.digikey.com/en/products/result?keywords=08055C1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
- C61: renamed from L2; value SRP7050TA-3R3M -> 68nF; footprint cryocooler:L_Bourns_SRP7050TA -> Capacitor_SMD:C_1206_3216Metric; symbol Device:L -> Device:C; Product (none) -> https://www.digikey.com/en/products/result?keywords=CC1206K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
- C63: Product (none) -> https://www.digikey.com/en/products/result?keywords=CL32B22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
- C65: renamed from R101; value 10k -> 22uF/50V; footprint Resistor_SMD:R_0603_1608Metric -> Capacitor_SMD:C_1210_3225Metric; symbol Device:R_US -> Device:C; Product (none) -> https://www.digikey.com/en/products/result?keywords=CL32B22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
- C66: renamed from C67; value 22uF/50V -> 1uF/50V; footprint Capacitor_SMD:C_1210_3225Metric -> Capacitor_SMD:C_1206_3216Metric; Product (none) -> https://www.digikey.com/en/products/result?keywords=CL31B10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
- C67: renamed from R102; value 10k -> 22uF/50V; footprint Resistor_SMD:R_0603_1608Metric -> Capacitor_SMD:C_1210_3225Metric; symbol Device:R_US -> Device:C; Product (none) -> https://www.digikey.com/en/products/result?keywords=CL32B22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
- D5: renamed from R57; value 2.67M -> DFLS240; footprint Resistor_SMD:R_0603_1608Metric -> Diode_SMD:D_PowerDI-123; symbol Device:R_US -> Device:D_Schottky; Product (none) -> https://www.digikey.com/en/products/result?keywords=DFLS240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
- D6: renamed from R59; value 2.55M -> DFLS240; footprint Resistor_SMD:R_0603_1608Metric -> Diode_SMD:D_PowerDI-123; symbol Device:R_US -> Device:D_Schottky; Product (none) -> https://www.digikey.com/en/products/result?keywords=DFLS240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
- L3: Product (none) -> https://www.digikey.com/en/products/result?keywords=SRP7050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
- R101: renamed from C66; value 1uF/50V -> 10k; footprint Capacitor_SMD:C_1206_3216Metric -> Resistor_SMD:R_0603_1608Metric; symbol Device:C -> Device:R_US; Product (none) -> https://www.digikey.com/en/products/result?keywords=AR0603F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
- R102: renamed from C68; value 1uF/50V -> 10k; footprint Capacitor_SMD:C_1206_3216Metric -> Resistor_SMD:R_0603_1608Metric; symbol Device:C -> Device:R_US; Product (none) -> https://www.digikey.com/en/products/result?keywords=AR0603F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
- R55: renamed from C60; value 1uF -> 5.6k; footprint Capacitor_SMD:C_0805_2012Metric -> Resistor_SMD:R_0603_1608Metric; symbol Device:C -> Device:R_US; Product (none) -> https://www.digikey.com/en/products/result?keywords=RC0603F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
- R56, R58: Product (none) -> https://www.digikey.com/en/products/result?keywords=RC0603F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
- R57: renamed from C62; value 22uF/50V -> 2.67M; footprint Capacitor_SMD:C_1210_3225Metric -> Resistor_SMD:R_0603_1608Metric; symbol Device:C -> Device:R_US; Product (none) -> https://www.digikey.com/en/products/result?keywords=CRCW060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
- R60: renamed from C64; value 1uF -> 118k; footprint Capacitor_SMD:C_0805_2012Metric -> Resistor_SMD:R_0603_1608Metric; symbol Device:C -> Device:R_US; Product (none) -> https://www.digikey.com/en/products/result?keywords=RC0603F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
- R61: renamed from R62; value 147k -> 432k; Product (none) -> https://www.digikey.com/en/products/result?keywords=RC0603F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
- R63: renamed from R64; value 147k -> 432k; Product (none) -> https://www.digikey.com/en/products/result?keywords=RC0603F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
- U20: Product (none) -> https://www.digikey.com/en/products/result?keywords=ADP5071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
- U21: Product (none) -> https://www.digikey.com/en/products/result?keywords=LT3097A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
Connections:
- net +15V: now also C65.1, R61.1
- net +16V5: now also C62.1
- net +5V_PS15: now also C56.1, C57.1
- net -15V: now also C67.1, R63.1; no longer C66.1
- net -16V5: now also D6.2 (A), R59.1; no longer D6.1
- net GND: now also C56.2, C61.2, C59.2, C62.2, C64.2, C68.2, R62.2, R64.2; no longer R55.2, R57.2, R60.2, R61.2, R63.2
- net at U20.2 (SW1): now also D5.2 (A), L2.2; no longer C61.2
- net at U21.10 (PGFBN): now also R102.1, R63.2; no longer C67.1
- net at L3.1, U20.20 (SW2): now also D6.1 (K)
- net at R58.1, U20.7 (FB1): now also R57.2; no longer D5.2
- net at U20.13 (FB2): now also R60.1, R59.2; no longer D6.2
- net at U20.16 (VREG), U20.5 (SEQ): now also C60.1; no longer R55.1
- net at R56.1: now also C61.1; no longer C60.1
- net at U20.14 (VREF): now also R60.2, C64.1; no longer R60.1
- net at U20.3 (INBK): now also L2.1; no longer C61.1
- net at U20.8 (COMP1): now also R55.2; no longer C56.2
- net at U21.17 (PGFBP): now also R101.1, R61.2; no longer C65.1
- new net: C68.1, R64.1, U21.12 (SETN)
- new net: C59.1, R55.1
- new net: C66.1, R62.1, U21.18 (SETP)
Other:
- moved on the sheet: C57, C60, C66, R61, R63

Commit message: Ground the M12 shield, order the ground loops, name the J14 cable parts
- J10: shielded symbol (Conn_01x04_Shielded); the M12 shield pin and its
  four shell legs are pad SH, tied to GND
- TP22-TP25: Keystone 5001 black miniature PC test points (KiCad
  TestPoint_Keystone_5000-5004 footprint, 1.02 mm hole per Keystone's
  drawing); now in the BOM, the bare pad test points stay out
- J14 BOM note: cable housing Molex 5054320801 with 505431 terminals, or
  tin pre-crimped leads 797581148 / 797581149 (from molex.com)

Only netlist change: GND gains J10 SH. DRC 0 errors, 0 unconnected, 0
schematic-parity issues; ERC 0; 193/193 datasheet rules.

Co-Authored-By: Claude Opus 5.5 <noreply@anthropic.com>
Parts:
- removed C56: 10uF, Capacitor_SMD:C_0805_2012Metric, symbol Device:C
- removed L2: SRP7050TA-3R3M, cryocooler:L_Bourns_SRP7050TA, symbol Device:L
- removed R56: 12k, Resistor_SMD:R_0603_1608Metric, symbol Device:R_US
- removed R57: 2.67M, Resistor_SMD:R_0603_1608Metric, symbol Device:R_US
- removed R59: 2.55M, Resistor_SMD:R_0603_1608Metric, symbol Device:R_US
- removed R61, R63: 432k, Resistor_SMD:R_0603_1608Metric, symbol Device:R_US
- removed R62, R64: 147k, Resistor_SMD:R_0603_1608Metric, symbol Device:R_US
- added C59: 47nF, Capacitor_SMD:C_1206_3216Metric, symbol Device:C
- added C61: 68nF, Capacitor_SMD:C_1206_3216Metric, symbol Device:C
- added C63: 22uF/50V, Capacitor_SMD:C_1210_3225Metric, symbol Device:C
- added C66, C68: 1uF/50V, Capacitor_SMD:C_1206_3216Metric, symbol Device:C
- added D5: DFLS240, Diode_SMD:D_PowerDI-123, symbol Device:D_Schottky
- added R101, R102: 10k, Resistor_SMD:R_0603_1608Metric, symbol Device:R_US
- added R58: 137k, Resistor_SMD:R_0603_1608Metric, symbol Device:R_US
- C57: renamed from C58; value 100nF -> 10uF; footprint Capacitor_SMD:C_0603_1608Metric -> Capacitor_SMD:C_0805_2012Metric; Product https://www.digikey.com/en/products/result?keywords=C0603C1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 -> https://www.digikey.com/en/products/result?keywords=CL21A10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
- C58: renamed from R55; value 5.6k -> 100nF; footprint Resistor_SMD:R_0603_1608Metric -> Capacitor_SMD:C_0603_1608Metric; symbol Device:R_US -> Device:C; Product https://www.digikey.com/en/products/result?keywords=RC0603F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 -> https://www.digikey.com/en/products/result?keywords=C0603C1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
- L2: renamed from D5; value DFLS240 -> SRP7050TA-3R3M; footprint Diode_SMD:D_PowerDI-123 -> cryocooler:L_Bourns_SRP7050TA; symbol Device:D_Schottky -> Device:L; Product https://www.digikey.com/en/products/result?keywords=DFLS240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 -> https://www.digikey.com/en/products/result?keywords=SRP7050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
- R55: renamed from C59; value 47nF -> 5.6k; footprint Capacitor_SMD:C_1206_3216Metric -> Resistor_SMD:R_0603_1608Metric; symbol Device:C -> Device:R_US; Product https://www.digikey.com/en/products/result?keywords=C1206C4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 -> https://www.digikey.com/en/products/result?keywords=RC0603F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
- R56: renamed from C61; value 68nF -> 12k; footprint Capacitor_SMD:C_1206_3216Metric -> Resistor_SMD:R_0603_1608Metric; symbol Device:C -> Device:R_US; Product https://www.digikey.com/en/products/result?keywords=CC1206K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 -> https://www.digikey.com/en/products/result?keywords=RC0603F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
- R57: renamed from R58; value 137k -> 2.67M; Product https://www.digikey.com/en/products/result?keywords=RC0603F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 -> https://www.digikey.com/en/products/result?keywords=CRCW060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
- R59: renamed from R60; value 118k -> 2.55M; Product https://www.digikey.com/en/products/result?keywords=RC0603FR-07118KL -> https://www.digikey.com/en/products/result?keywords=RC0603FR-072M55L
- R60: renamed from C63; value 22uF/50V -> 118k; footprint Capacitor_SMD:C_1210_3225Metric -> Resistor_SMD:R_0603_1608Metric; symbol Device:C -> Device:R_US; Product https://www.digikey.com/en/products/result?keywords=CL32B22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 -> https://www.digikey.com/en/products/result?keywords=RC0603F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
- R61: renamed from R101; value 10k -> 432k; Product https://www.digikey.com/en/products/result?keywords=AR0603F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 -> https://www.digikey.com/en/products/result?keywords=RC0603F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
- R62: renamed from C66; value 1uF/50V -> 147k; footprint Capacitor_SMD:C_1206_3216Metric -> Resistor_SMD:R_0603_1608Metric; symbol Device:C -> Device:R_US; Product https://www.digikey.com/en/products/result?keywords=CL31B10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 -> https://www.digikey.com/en/products/result?keywords=RC0603F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
- R63: renamed from R102; value 10k -> 432k; Product https://www.digikey.com/en/products/result?keywords=AR0603F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 -> https://www.digikey.com/en/products/result?keywords=RC0603F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
- R64: renamed from C68; value 1uF/50V -> 147k; footprint Capacitor_SMD:C_1206_3216Metric -> Resistor_SMD:R_0603_1608Metric; symbol Device:C -> Device:R_US; Product https://www.digikey.com/en/products/result?keywords=CL31B10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 -> https://www.digikey.com/en/products/result?keywords=RC0603F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
- renumbered C57 to C56
Connections:
- net +15V: now also R61.1
- net +16V5: now also R57.1, D5.1 (K); no longer L2.1 (K)
- net +5V_PS15: now also C58.1
- net -15V: now also R63.1
- net -16V5: now also R59.1, C63.1; no longer R60.1
- net GND: now also C58.2, C59.2, C61.2, C63.2, C66.2, C68.2, R101.2, R102.2, R58.2; no longer R55.2, R56.2, R57.2, R60.2, R61.2, R63.2
- net at U20.12 (COMP2): now also R56.2
- net at U20.13 (FB2): now also R59.2, R60.1; no longer R59.1
- net at C64.1, U20.14 (VREF): now also R60.2; no longer R59.2
- net at L2.2, U20.2 (SW1): now also D5.2 (A)
- net at U20.3 (INBK): now also L2.1
- net at U20.7 (FB1): now also R57.2, R58.1; no longer R57.1
- net at U20.8 (COMP1): now also R55.2; no longer C58.2
- net at R64.1, U21.12 (SETN): now also C68.1
- net at R55.1: now also C59.1; no longer C58.1
- net at R62.1, U21.18 (SETP): now also C66.1
- net at U21.10 (PGFBN): now also R63.2, R102.1; no longer R63.1
- net at R56.1: now also C61.1
- net at U21.17 (PGFBP): now also R61.2, R101.1; no longer R61.1
Other:
- moved on the sheet: C56, C57, R57, R59, R61, R63
