File: hardware/kicad/sheets/compressor_relay.kicad_sch (KiCad schematic)
At the start: 10 parts, among them J13 COMPRESSOR RELAY / GND, Q7 BSS138, Q8 BSS84

Commit message: Move the IMU off-board (J14) and add labelled module boxes to the PCB
The LSM6DSOX is now the Adafruit breakout (product 4438) mounted on the
cryocooler and cabled to a 10-pin JST XH header (J14) over the shared SPI
bus. U19 and its capacitors are gone; J14 and six 100 R series resistors
are added, and every other reference number is unchanged.

PCB (130 x 110 mm, was 130 x 100):
- one outlined, labelled silkscreen box per module (pcbfloorplan.py); the
  placer keeps parts inside their box and reserves a label pocket beside
  every part so each label sits next to its own part
- box 3D models for U3, L2, L3, F1 and PS1, whose library models are missing
- re-routed; DRC 0 errors, 0 unconnected; back logo recentred
- gen_pcb.py texts redoes the silkscreen on a routed board

Firmware: SPI clock constant for the module, comments updated; ambient
temperature now reads the cooler-body IMU temperature.

Docs, BOM and fabrication files regenerated.

Co-Authored-By: Claude Sonnet 5.5 <noreply@anthropic.com>
Parts:
- removed D12: RED/GREEN, LED_SMD:LED_1206_3216Metric, symbol Device:LED_Dual_Bidirectional
- removed R76: 1k, Resistor_SMD:R_0603_1608Metric, symbol Device:R_US
- removed R80: 2.2k, Resistor_SMD:R_0603_1608Metric, symbol Device:R_US
- added D13: 1N4148W, Diode_SMD:D_SOD-123, symbol Device:D
- added J13: COMPRESSOR RELAY / GND, Connector_JST:JST_XH_B2B-XH-A_1x02_P2.50mm_Vertical, symbol Connector:Screw_Terminal_01x02
- added Q7: BSS138, Package_TO_SOT_SMD:SOT-23, symbol Transistor_FET:BSS138
- D12: renamed from D13; value 1N4148W -> RED/GREEN; footprint Diode_SMD:D_SOD-123 -> LED_SMD:LED_1206_3216Metric; symbol Device:D -> Device:LED_Dual_Bidirectional
- R76: renamed from Q7; value BSS138 -> 1k; footprint Package_TO_SOT_SMD:SOT-23 -> Resistor_SMD:R_0603_1608Metric; symbol Transistor_FET:BSS138 -> Device:R_US
- R80: renamed from J13; value COMPRESSOR RELAY / GND -> 2.2k; footprint Connector_JST:JST_XH_B2B-XH-A_1x02_P2.50mm_Vertical -> Resistor_SMD:R_0603_1608Metric; symbol Connector:Screw_Terminal_01x02 -> Device:R_US
Connections:
- net +5V: now also R80.1
- net COMP_RELAY: now also D12.2 (AK), D13.1 (K), J13.1 (Pin_1); no longer D12.1 (K), R80.1 (Pin_1)
- net COMP_RELAY_EN: now also R76.1
- net GND: now also D13.2 (A), J13.2 (Pin_2), Q7.2 (S); no longer D12.2 (A), R76.2 (S), R80.2 (Pin_2)
- net at R77.1: now also R76.2, Q7.1 (G); no longer R76.1 (G)
- net at Q8.1 (G), R78.2: now also Q7.3 (D); no longer R76.3 (D)
- new net: D12.1 (KA), R80.2

Commit message: Add per-section supply jumpers, 8-pin IMU header and connector pin labels
- Four 1.27 mm 2-pin jumpers (JP1-JP4), each with a rail-on LED, cut the
  supply of one section for debugging: signal generator +3V3, +-15V
  generator +5V in, isolated amp-current supply +5V in, and a shared
  +3V3 net for the cooling chips (EMC2303, RTD ADC, I2C bridge).
- J14 is now an 8-pin JST XH in the Adafruit LSM6DSOX pad order
  (VIN, GND, SCL, SDA, DO, CS, I1, I2); firmware pin comments updated.
- Pin-function labels beside every connector, "RAILS ±15V" box title.
- Board re-placed and re-routed (130 x 110 mm); DRC 0 errors, 0 unconnected,
  ERC 0, 173 datasheet rules pass. BOM, READMEs, Gerbers and renders
  regenerated; link_usb_vbus.py now adapts to the routed layout.

Co-Authored-By: Claude Sonnet 5.5 <noreply@anthropic.com>
Parts:
- removed D12: RED/GREEN, LED_SMD:LED_1206_3216Metric, symbol Device:LED_Dual_Bidirectional
- removed D13: 1N4148W, Diode_SMD:D_SOD-123, symbol Device:D
- added J13: COMPRESSOR RELAY / GND, Connector_JST:JST_XH_B2B-XH-A_1x02_P2.50mm_Vertical, symbol Connector:Screw_Terminal_01x02
- added R77: 100k, Resistor_SMD:R_0603_1608Metric, symbol Device:R_US
- D12: renamed from R80; value 2.2k -> RED/GREEN; footprint Resistor_SMD:R_0603_1608Metric -> LED_SMD:LED_1206_3216Metric; symbol Device:R_US -> Device:LED_Dual_Bidirectional
- D13: renamed from J13; value COMPRESSOR RELAY / GND -> 1N4148W; footprint Connector_JST:JST_XH_B2B-XH-A_1x02_P2.50mm_Vertical -> Diode_SMD:D_SOD-123; symbol Connector:Screw_Terminal_01x02 -> Device:D
- Q7: renamed from R77; value 100k -> BSS138; footprint Resistor_SMD:R_0603_1608Metric -> Package_TO_SOT_SMD:SOT-23; symbol Device:R_US -> Transistor_FET:BSS138
- Q8: renamed from R78; value 100k -> BSS84; footprint Resistor_SMD:R_0603_1608Metric -> Package_TO_SOT_SMD:SOT-23; symbol Device:R_US -> Transistor_FET:BSS84
- R78: renamed from Q7; value BSS138 -> 100k; footprint Package_TO_SOT_SMD:SOT-23 -> Resistor_SMD:R_0603_1608Metric; symbol Transistor_FET:BSS138 -> Device:R_US
- R79: renamed from Q8; value BSS84 -> 1k; footprint Package_TO_SOT_SMD:SOT-23 -> Resistor_SMD:R_0603_1608Metric; symbol Transistor_FET:BSS84 -> Device:R_US
- R80: renamed from R79; value 1k -> 2.2k
Connections:
- net +12V: now also Q8.2 (S), R78.1; no longer Q8.1, R79.2 (S)
- net +5V: now also R80.1; no longer D12.1
- net COMP_RELAY: now also D12.2 (AK), Q8.3 (D), R79.1, J13.1 (Pin_1); no longer R79.3 (D), R80.1
- net GND: now also R79.2, J13.2 (Pin_2), R77.2; no longer R78.2 (S), R80.2
- net at Q7.1 (G), R76.2: now also R77.1; no longer R78.1 (G)
- new net: D12.1 (KA), R80.2
- new net: Q7.3 (D), Q8.1 (G), R78.2
Other:
- moved on the sheet: R80

Commit message: Replace the ±15 V LDOs with one LT3097 and add a power-good interlock
- rails_15v: ADP7142 + ADP7182 replaced by one LT3097 (±14.7 V, 147 k SET
  resistors); the ADP5071 output caps are now 22 uF / 50 V and double as the
  LT3097 inputs. PGP / PGN make the PG_15V node (fed from +15 V, so it reads
  0 V if a rail is missing).
- amp_control: a series BSS138 (Q9) gated by PG_15V blocks AMP_REM unless
  both rails are good. New power_good sheet: LED (D23) and the active-low
  PG_15V_N flag on GPIO43 (PG_15V_N_PIN).
- Tooling: LT3097 symbol, footprint and 3D envelope; datasheet rules (191),
  GPIO check, BOM tables, floor plan, PAD_BRIDGES and pre-placed GND vias in
  gen_pcb.py, new fix_route.py for post-route clean-up.
- Board regenerated and routed with Freerouting 2.5.0: DRC 0 unconnected,
  0 schematic-parity issues, no copper violations. Gerbers, JLCPCB zip,
  renders, BOM, CPL and schematic PDF regenerated.

Co-Authored-By: Claude Sonnet 5.5 <noreply@anthropic.com>
Parts:
- removed Q7: BSS138, Package_TO_SOT_SMD:SOT-23, symbol Transistor_FET:BSS138
- removed R76: 1k, Resistor_SMD:R_0603_1608Metric, symbol Device:R_US
- removed R77: 100k, Resistor_SMD:R_0603_1608Metric, symbol Device:R_US
- added D12: RED/GREEN, LED_SMD:LED_1206_3216Metric, symbol Device:LED_Dual_Bidirectional
- added D13: 1N4148W, Diode_SMD:D_SOD-123, symbol Device:D
- added J13: COMPRESSOR RELAY / GND, Connector_JST:JST_XH_B2B-XH-A_1x02_P2.50mm_Vertical, symbol Connector:Screw_Terminal_01x02
- Q7: renamed from D13; value 1N4148W -> BSS138; footprint Diode_SMD:D_SOD-123 -> Package_TO_SOT_SMD:SOT-23; symbol Device:D -> Transistor_FET:BSS138
- R76: renamed from D12; value RED/GREEN -> 1k; footprint LED_SMD:LED_1206_3216Metric -> Resistor_SMD:R_0603_1608Metric; symbol Device:LED_Dual_Bidirectional -> Device:R_US
- R77: renamed from J13; value COMPRESSOR RELAY / GND -> 100k; footprint Connector_JST:JST_XH_B2B-XH-A_1x02_P2.50mm_Vertical -> Resistor_SMD:R_0603_1608Metric; symbol Connector:Screw_Terminal_01x02 -> Device:R_US
Connections:
- net COMP_RELAY: now also D12.2 (AK), D13.1 (K), J13.1 (Pin_1); no longer Q7.1 (K), R76.2 (AK), R77.1 (Pin_1)
- net COMP_RELAY_EN: now also R76.1
- net GND: now also D13.2 (A), J13.2 (Pin_2)
- net at R80.2: now also D12.1 (KA); no longer R76.1 (KA)
- net at Q8.1 (G), R78.2: now also Q7.3 (D)
- new net: Q7.1 (G), R76.2, R77.1

Commit message: Log +-15 V power-good changes and add one LED per LT3097 PG pin
Firmware
- amplifier: configure PG_15V_N_PIN (GPIO43, active LOW), log the starting
  state and every debounced change (PowerGoodMonitor in power_good.h);
  amplifier::isPowerGood() reports the level. The lines reach the dashboard
  console through the logger ring buffer.
- dashboard: console colours for "power lost" (red), "power restored" and
  "power good: yes" (green), "power good: no" (yellow).
- native tests for the debounce logic and the amplifier stub.

Hardware
- power_good sheet: PGP and PGN each drive their own node (220k/62k from
  +15 V) and a green LED (D24 +15 V, D25 -15 V) through a BSS138W; a BAT54AW
  with a 10k pull-up ANDs the nodes into PG_15V, so the REM interlock and the
  PG_15V_N flag are unchanged.
- 0402 resistors, SOT-323 FETs and one BAT54AW so the stage fits the power
  box; Power Good parts are placed last in gen_pcb.py.
- Board re-routed with Freerouting 2.5.0 and cleaned with fix_route.py: DRC
  0 unconnected, no copper violations. Gerbers, JLCPCB zip, renders, BOM, CPL
  and schematic PDF regenerated; datasheet rules 193/193.

Co-Authored-By: Claude Sonnet 5.5 <noreply@anthropic.com>
Parts:
- removed R77: 100k, Resistor_SMD:R_0603_1608Metric, symbol Device:R_US
- added D13: 1N4148W, Diode_SMD:D_SOD-123, symbol Device:D
- R77: renamed from D13; value 1N4148W -> 100k; footprint Diode_SMD:D_SOD-123 -> Resistor_SMD:R_0603_1608Metric; symbol Device:D -> Device:R_US
Connections:
- net COMP_RELAY: now also D13.1 (K); no longer R77.1 (K)
- net GND: now also D13.2 (A)
- net at Q7.1 (G), R76.2: now also R77.1

Commit message: WIP: restructure PCB for the Phoenix UCS 125-87 housing
Work in progress, layout not finished: about 90 parts still do not fit
their sections and the board is not routed.

- Right-angle connectors: Phoenix MSTBA 2,5 / MC 1,5, JST XH side entry,
  Hirose DF13, Molex 505448-0871 (new footprint from the Molex drawing)
- Datasheet and product links on every symbol (tools/part_links.py)
- Test points so every IC has one on its own nets
- gen_pcb.py: 100 x 62 mm two-sided board, housing holes and restricted
  corners, ESP32 antenna notch, one section per sheet, board ID block,
  ESP32 pin names, pin-1 marks, blue mask
- Housing drawings in hardware/housing/

Co-Authored-By: Claude Opus 5.5 <noreply@anthropic.com>
Parts:
- removed D12: RED/GREEN, LED_SMD:LED_1206_3216Metric, symbol Device:LED_Dual_Bidirectional
- removed R76: 1k, Resistor_SMD:R_0603_1608Metric, symbol Device:R_US
- removed R80: 2.2k, Resistor_SMD:R_0603_1608Metric, symbol Device:R_US
- added D13: 1N4148W, Diode_SMD:D_SOD-123, symbol Device:D
- added J13: COMPRESSOR RELAY / GND, Connector_Hirose:Hirose_DF13-02P-1.25DS_1x02_P1.25mm_Horizontal, symbol Connector:Screw_Terminal_01x02
- added Q7: BSS138, Package_TO_SOT_SMD:SOT-23, symbol Transistor_FET:BSS138
- D12: renamed from D13; value 1N4148W -> RED/GREEN; footprint Diode_SMD:D_SOD-123 -> LED_SMD:LED_1206_3216Metric; symbol Device:D -> Device:LED_Dual_Bidirectional; Product (none) -> https://www.digikey.com/en/products/result?keywords=XZMDKVG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
- Q8: Product (none) -> https://www.digikey.com/en/products/result?keywords=BSS84
- R76: renamed from Q7; value BSS138 -> 1k; footprint Package_TO_SOT_SMD:SOT-23 -> Resistor_SMD:R_0603_1608Metric; symbol Transistor_FET:BSS138 -> Device:R_US; Product (none) -> https://www.digikey.com/en/products/result?keywords=RC0603F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
- R77, R78: Product (none) -> https://www.digikey.com/en/products/result?keywords=AR0603F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
- R79: Product (none) -> https://www.digikey.com/en/products/result?keywords=RC0603F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
- R80: renamed from J13; value COMPRESSOR RELAY / GND -> 2.2k; footprint Connector_JST:JST_XH_B2B-XH-A_1x02_P2.50mm_Vertical -> Resistor_SMD:R_0603_1608Metric; symbol Connector:Screw_Terminal_01x02 -> Device:R_US; Product (none) -> https://www.digikey.com/en/products/result?keywords=RC0603F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
Connections:
- net +5V: now also R80.1
- net COMP_RELAY: now also D12.2 (AK), D13.1 (K), J13.1 (Pin_1); no longer D12.1 (K), R80.1 (Pin_1)
- net COMP_RELAY_EN: now also R76.1
- net GND: now also D13.2 (A), J13.2 (Pin_2), Q7.2 (S); no longer D12.2 (A), R76.2 (S), R80.2 (Pin_2)
- net at R77.1: now also R76.2, Q7.1 (G); no longer R76.1 (G)
- net at Q8.1 (G), R78.2: now also Q7.3 (D); no longer R76.3 (D)
- new net: D12.1 (KA), R80.2

Commit message: Use an M12 receptacle for the PT1000 and JST PH headers for the 2-pin I/O
- J10 (cold head PT1000): TE T4145035041-001, M12 A-coded 4-pin female,
  right angle, shielded, panel and PCB mount through the right side wall;
  footprint from TE drawing T41450350X1001 rev B
- J6, J7, J13 (NTC, panel button, relay out): Adafruit 1769 (4UCON 17311),
  JST PH compatible 2-pin right-angle SMT; footprint from its drawing
- BOM, part links and 3D envelopes for both; schematic nets unchanged
- gen_pcb: ground fan-out before routing (a locked via and short track per
  small ground pad, clear of other holes) so no ground pad is left on a
  pour island; fallback labels must sit inside a section box
- fix_route: skip paste apertures (not non-plated holes) as foreign copper,
  nudge tracks off crowded pads, remove GND vias that crowd another hole

DRC 0 errors, 0 unconnected, 0 schematic-parity issues; ERC 0; 193/193
datasheet rules.

Co-Authored-By: Claude Opus 5.5 <noreply@anthropic.com>
Parts:
- J13: footprint Connector_Hirose:Hirose_DF13-02P-1.25DS_1x02_P1.25mm_Horizontal -> cryocooler:Adafruit_1769_JST-PH_1x02_P2.00mm_Horizontal_SMD; Product https://www.digikey.com/en/products/result?keywords=DF13-2P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 -> https://www.adafruit.com/product/1769
Changed lines of the file:
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@@
 			)
 		)
-		(property "Footprint" "Connector_Hirose:Hirose_DF13-02P-1.25DS_1x02_P1.25mm_Horizontal"
+		(property "Footprint" "cryocooler:Adafruit_1769_JST-PH_1x02_P2.00mm_Horizontal_SMD"
 			(at 177.8 73.66 0)
 			(hide yes)
@@
 			)
 		)
-		(property "Datasheet" "https://www.hirose.com/api/v1/series/DF13/documents/product_series_catalog/content?lang=EN"
+		(property "Datasheet" "https://cdn-shop.adafruit.com/datasheets/17311.pdf"
 			(at 177.8 73.66 0)
 			(hide yes)
@@
 			)
 		)
-		(property "Product" "https://www.digikey.com/en/products/result?keywords=DF13-2P-1.25DS%2825%29"
+		(property "Product" "https://www.adafruit.com/product/1769"
 			(at 177.8 73.66 0)
 			(hide yes)

Commit message: Ground the M12 shield, order the ground loops, name the J14 cable parts
- J10: shielded symbol (Conn_01x04_Shielded); the M12 shield pin and its
  four shell legs are pad SH, tied to GND
- TP22-TP25: Keystone 5001 black miniature PC test points (KiCad
  TestPoint_Keystone_5000-5004 footprint, 1.02 mm hole per Keystone's
  drawing); now in the BOM, the bare pad test points stay out
- J14 BOM note: cable housing Molex 5054320801 with 505431 terminals, or
  tin pre-crimped leads 797581148 / 797581149 (from molex.com)

Only netlist change: GND gains J10 SH. DRC 0 errors, 0 unconnected, 0
schematic-parity issues; ERC 0; 193/193 datasheet rules.

Co-Authored-By: Claude Opus 5.5 <noreply@anthropic.com>
Parts:
- removed D12: RED/GREEN, LED_SMD:LED_1206_3216Metric, symbol Device:LED_Dual_Bidirectional
- removed R76: 1k, Resistor_SMD:R_0603_1608Metric, symbol Device:R_US
- added J13: COMPRESSOR RELAY / GND, cryocooler:Adafruit_1769_JST-PH_1x02_P2.00mm_Horizontal_SMD, symbol Connector:Screw_Terminal_01x02
- added R77: 100k, Resistor_SMD:R_0603_1608Metric, symbol Device:R_US
- D12: renamed from J13; value COMPRESSOR RELAY / GND -> RED/GREEN; footprint cryocooler:Adafruit_1769_JST-PH_1x02_P2.00mm_Horizontal_SMD -> LED_SMD:LED_1206_3216Metric; symbol Connector:Screw_Terminal_01x02 -> Device:LED_Dual_Bidirectional; Product https://www.adafruit.com/product/1769 -> https://www.digikey.com/en/products/result?keywords=XZMDKVG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
- R76: renamed from R77; value 100k -> 1k; Product https://www.digikey.com/en/products/result?keywords=AR0603F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 -> https://www.digikey.com/en/products/result?keywords=RC0603F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
Connections:
- net COMP_RELAY: now also D12.2 (AK), J13.1 (Pin_1); no longer D12.1 (Pin_1)
- net COMP_RELAY_EN: now also R76.1
- net GND: now also J13.2 (Pin_2), R77.2; no longer D12.2 (Pin_2), R76.2
- net at Q7.1 (G): now also R76.2, R77.1; no longer R76.1
- net at R80.2: now also D12.1 (KA)
Other:
- moved on the sheet: R76
