File: hardware/kicad/sheets/debug.kicad_sch (KiCad schematic)
At the start: 49 parts

Commit message: Log +-15 V power-good changes and add one LED per LT3097 PG pin
Firmware
- amplifier: configure PG_15V_N_PIN (GPIO43, active LOW), log the starting
  state and every debounced change (PowerGoodMonitor in power_good.h);
  amplifier::isPowerGood() reports the level. The lines reach the dashboard
  console through the logger ring buffer.
- dashboard: console colours for "power lost" (red), "power restored" and
  "power good: yes" (green), "power good: no" (yellow).
- native tests for the debounce logic and the amplifier stub.

Hardware
- power_good sheet: PGP and PGN each drive their own node (220k/62k from
  +15 V) and a green LED (D24 +15 V, D25 -15 V) through a BSS138W; a BAT54AW
  with a 10k pull-up ANDs the nodes into PG_15V, so the REM interlock and the
  PG_15V_N flag are unchanged.
- 0402 resistors, SOT-323 FETs and one BAT54AW so the stage fits the power
  box; Power Good parts are placed last in gen_pcb.py.
- Board re-routed with Freerouting 2.5.0 and cleaned with fix_route.py: DRC
  0 unconnected, no copper violations. Gerbers, JLCPCB zip, renders, BOM, CPL
  and schematic PDF regenerated; datasheet rules 193/193.

Co-Authored-By: Claude Sonnet 5.5 <noreply@anthropic.com>
Parts:
- removed TP10: -15V, TestPoint:TestPoint_Pad_D1.5mm, symbol Connector:TestPoint
- removed TP11: +16V5, TestPoint:TestPoint_Pad_D1.5mm, symbol Connector:TestPoint
- removed TP12: -16V5, TestPoint:TestPoint_Pad_D1.5mm, symbol Connector:TestPoint
- removed TP13: ISO_3V3, TestPoint:TestPoint_Pad_D1.5mm, symbol Connector:TestPoint
- removed TP19: SPI_MOSI, TestPoint:TestPoint_Pad_D1.5mm, symbol Connector:TestPoint
- removed TP21: MCP4921_CS, TestPoint:TestPoint_Pad_D1.5mm, symbol Connector:TestPoint
- removed TP23: IMU_CS, TestPoint:TestPoint_Pad_D1.5mm, symbol Connector:TestPoint
- removed TP26: BRIDGE_CS, TestPoint:TestPoint_Pad_D1.5mm, symbol Connector:TestPoint
- removed TP28: ACS_MISO, TestPoint:TestPoint_Pad_D1.5mm, symbol Connector:TestPoint
- removed TP32: IMU_INT1, TestPoint:TestPoint_Pad_D1.5mm, symbol Connector:TestPoint
- removed TP6: VSW, TestPoint:TestPoint_Pad_D1.5mm, symbol Connector:TestPoint
- removed TP7: +5V, TestPoint:TestPoint_Pad_D1.5mm, symbol Connector:TestPoint
- removed TP8: +3V3, TestPoint:TestPoint_Pad_D1.5mm, symbol Connector:TestPoint
- removed TP9: +15V, TestPoint:TestPoint_Pad_D1.5mm, symbol Connector:TestPoint
- added D14: 5V (yellow), LED_SMD:LED_0603_1608Metric, symbol Device:LED
- added D15: +15V (white), LED_SMD:LED_0603_1608Metric, symbol Device:LED
- added D16: -15V (white), LED_SMD:LED_0603_1608Metric, symbol Device:LED
- added R86, R89: 1k, Resistor_SMD:R_0603_1608Metric, symbol Device:R_US
- added R87, R88: 4.7k, Resistor_SMD:R_0603_1608Metric, symbol Device:R_US
- added TP31: SCL, TestPoint:TestPoint_Pad_D1.5mm, symbol Connector:TestPoint
- added TP34: FAN_ALERT, TestPoint:TestPoint_Pad_D1.5mm, symbol Connector:TestPoint
- added TP35: PWR_KILL, TestPoint:TestPoint_Pad_D1.5mm, symbol Connector:TestPoint
- added TP38: PG_15V, TestPoint:TestPoint_Pad_D1.5mm, symbol Connector:TestPoint
- added TP39: ESP_EN, TestPoint:TestPoint_Pad_D1.5mm, symbol Connector:TestPoint
- added TP42: NTC_ADC, TestPoint:TestPoint_Pad_D1.5mm, symbol Connector:TestPoint
- added TP43: FLOW_TACH, TestPoint:TestPoint_Pad_D1.5mm, symbol Connector:TestPoint
- TP10: renamed from TP18; value SPI_SCK -> -15V
- TP11: renamed from TP20; value SPI_MISO -> +16V5
- TP12: renamed from TP22; value AD9833_FSYNC -> -16V5
- TP13: renamed from TP24; value INA239_CS -> ISO_3V3
- TP14: renamed from TP25; value ADS1220_CS -> GND; footprint TestPoint:TestPoint_Pad_D1.5mm -> TestPoint:TestPoint_Loop_D2.50mm_Drill1.0mm
- TP15: renamed from TP27; value ACS_CS -> GND; footprint TestPoint:TestPoint_Pad_D1.5mm -> TestPoint:TestPoint_Loop_D2.50mm_Drill1.0mm
- TP16: renamed from TP29; value BRIDGE_RESET -> GND; footprint TestPoint:TestPoint_Pad_D1.5mm -> TestPoint:TestPoint_Loop_D2.50mm_Drill1.0mm
- TP17: renamed from TP31; value SCL -> ISO_GND; footprint TestPoint:TestPoint_Pad_D1.5mm -> TestPoint:TestPoint_Loop_D2.50mm_Drill1.0mm
- TP18: renamed from TP33; value IMU_INT2 -> SPI_SCK
- TP19: renamed from TP34; value FAN_ALERT -> SPI_MOSI
- TP20: renamed from TP35; value PWR_KILL -> SPI_MISO
- TP21: renamed from TP36; value COMP_RELAY_EN -> MCP4921_CS
- TP22: renamed from TP37; value AMP_REM_EN -> AD9833_FSYNC
- TP23: renamed from TP38; value PG_15V -> IMU_CS
- TP24: renamed from TP39; value ESP_EN -> INA239_CS
- TP25: renamed from TP40; value ESP_BOOT -> ADS1220_CS
- TP26: renamed from TP41; value SIG_SINE -> BRIDGE_CS
- TP27: renamed from TP42; value NTC_ADC -> ACS_CS
- TP28: renamed from TP43; value FLOW_TACH -> ACS_MISO
- TP29: renamed from TP44; value STATUS_RGB -> BRIDGE_RESET
- TP32: renamed from R86; value 1k -> IMU_INT1; footprint Resistor_SMD:R_0603_1608Metric -> TestPoint:TestPoint_Pad_D1.5mm; symbol Device:R_US -> Connector:TestPoint
- TP33: renamed from D14; value 5V (yellow) -> IMU_INT2; footprint LED_SMD:LED_0603_1608Metric -> TestPoint:TestPoint_Pad_D1.5mm; symbol Device:LED -> Connector:TestPoint
- TP36: renamed from R87; value 4.7k -> COMP_RELAY_EN; footprint Resistor_SMD:R_0603_1608Metric -> TestPoint:TestPoint_Pad_D1.5mm; symbol Device:R_US -> Connector:TestPoint
- TP37: renamed from D15; value +15V (white) -> AMP_REM_EN; footprint LED_SMD:LED_0603_1608Metric -> TestPoint:TestPoint_Pad_D1.5mm; symbol Device:LED -> Connector:TestPoint
- TP40: renamed from R88; value 4.7k -> ESP_BOOT; footprint Resistor_SMD:R_0603_1608Metric -> TestPoint:TestPoint_Pad_D1.5mm; symbol Device:R_US -> Connector:TestPoint
- TP41: renamed from D16; value -15V (white) -> SIG_SINE; footprint LED_SMD:LED_0603_1608Metric -> TestPoint:TestPoint_Pad_D1.5mm; symbol Device:LED -> Connector:TestPoint
- TP44: renamed from R89; value 1k -> STATUS_RGB; footprint Resistor_SMD:R_0603_1608Metric -> TestPoint:TestPoint_Pad_D1.5mm; symbol Device:R_US -> Connector:TestPoint
- TP6: renamed from TP14; value GND -> VSW; footprint TestPoint:TestPoint_Loop_D2.50mm_Drill1.0mm -> TestPoint:TestPoint_Pad_D1.5mm
- TP7: renamed from TP15; value GND -> +5V; footprint TestPoint:TestPoint_Loop_D2.50mm_Drill1.0mm -> TestPoint:TestPoint_Pad_D1.5mm
- TP8: renamed from TP16; value GND -> +3V3; footprint TestPoint:TestPoint_Loop_D2.50mm_Drill1.0mm -> TestPoint:TestPoint_Pad_D1.5mm
- TP9: renamed from TP17; value ISO_GND -> +15V; footprint TestPoint:TestPoint_Loop_D2.50mm_Drill1.0mm -> TestPoint:TestPoint_Pad_D1.5mm
Connections:
- net +15V: now also TP9.1, R87.1; no longer TP36.1
- net +16V5: now also TP11.1
- net +3V3: now also TP8.1
- net +5V: now also TP7.1, R86.1; no longer TP32.1
- net -15V: now also TP10.1, R88.2; no longer TP40.2
- net -16V5: now also TP12.1
- net ACS_CS: now also TP27.1; no longer TP15.1
- net ACS_MISO: now also TP28.1
- net AD9833_FSYNC: now also TP22.1; no longer TP12.1
- net ADS1220_CS: now also TP25.1; no longer TP14.1
- net AMP_REM_EN: now also TP37.1; no longer TP22.1
- net BRIDGE_CS: now also TP26.1
- net BRIDGE_RESET: now also TP29.1; no longer TP16.1
- net COMP_RELAY_EN: now also TP36.1; no longer TP21.1
- net ESP_BOOT: now also TP40.1; no longer TP25.1
- net ESP_EN: now also TP39.1; no longer TP24.1
- net FAN_ALERT: now also TP34.1; no longer TP19.1
- net FLOW_TACH: now also TP43.1; no longer TP28.1
- net GND: now also TP14.1, TP15.1, TP16.1, D14.1 (K), D15.1 (K), D16.2 (A); no longer TP33.1 (K), TP37.1 (K), TP41.2 (A), TP6.1, TP7.1, TP8.1
- net IMU_CS: now also TP23.1
- net IMU_INT1: now also TP32.1
- net IMU_INT2: now also TP33.1; no longer TP18.1
- net INA239_CS: now also TP24.1; no longer TP13.1
- net ISO_3V3: now also TP13.1, R89.1; no longer TP44.1
- net ISO_GND: now also TP17.1; no longer TP9.1
- net MCP4921_CS: now also TP21.1
- net NTC_ADC: now also TP42.1; no longer TP27.1
- net PG_15V: now also TP38.1; no longer TP23.1
- net PWR_KILL: now also TP35.1; no longer TP20.1
- net SCL: now also TP31.1; no longer TP17.1
- net SIG_SINE: now also TP41.1; no longer TP26.1
- net SPI_MISO: now also TP20.1; no longer TP11.1
- net SPI_MOSI: now also TP19.1
- net SPI_SCK: now also TP18.1; no longer TP10.1
- net STATUS_RGB: now also TP44.1; no longer TP29.1
- net VSW: now also TP6.1
- net at D17.2 (A): now also R89.2; no longer TP44.2
- new net: D16.1 (K), R88.1
- new net: D15.2 (A), R87.2
- new net: D14.2 (A), R86.2
Other:
- moved on the sheet: TP10, TP11, TP12, TP13, TP14, TP15, TP16, TP17, TP18, TP19, TP20, TP21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

Commit message: WIP: restructure PCB for the Phoenix UCS 125-87 housing
Work in progress, layout not finished: about 90 parts still do not fit
their sections and the board is not routed.

- Right-angle connectors: Phoenix MSTBA 2,5 / MC 1,5, JST XH side entry,
  Hirose DF13, Molex 505448-0871 (new footprint from the Molex drawing)
- Datasheet and product links on every symbol (tools/part_links.py)
- Test points so every IC has one on its own nets
- gen_pcb.py: 100 x 62 mm two-sided board, housing holes and restricted
  corners, ESP32 antenna notch, one section per sheet, board ID block,
  ESP32 pin names, pin-1 marks, blue mask
- Housing drawings in hardware/housing/

Co-Authored-By: Claude Opus 5.5 <noreply@anthropic.com>
Parts:
- removed TP19: SPI_MOSI, TestPoint:TestPoint_Pad_D1.5mm, symbol Connector:TestPoint
- removed TP21: MCP4921_CS, TestPoint:TestPoint_Pad_D1.5mm, symbol Connector:TestPoint
- removed TP24: INA239_CS, TestPoint:TestPoint_Pad_D1.5mm, symbol Connector:TestPoint
- removed TP26: BRIDGE_CS, TestPoint:TestPoint_Pad_D1.5mm, symbol Connector:TestPoint
- removed TP28: ACS_MISO, TestPoint:TestPoint_Pad_D1.5mm, symbol Connector:TestPoint
- removed TP30: SDA, TestPoint:TestPoint_Pad_D1.5mm, symbol Connector:TestPoint
- removed TP4: VIN, TestPoint:TestPoint_Pad_D1.5mm, symbol Connector:TestPoint
- removed TP5: +12V, TestPoint:TestPoint_Pad_D1.5mm, symbol Connector:TestPoint
- removed TP6: VSW, TestPoint:TestPoint_Pad_D1.5mm, symbol Connector:TestPoint
- added D14: 5V (yellow), LED_SMD:LED_0603_1608Metric, symbol Device:LED
- added D15: +15V (white), LED_SMD:LED_0603_1608Metric, symbol Device:LED
- added D16: -15V (white), LED_SMD:LED_0603_1608Metric, symbol Device:LED
- added D17: ISO 3V3 (green), LED_SMD:LED_0603_1608Metric, symbol Device:LED
- added R87, R88: 4.7k, Resistor_SMD:R_0603_1608Metric, symbol Device:R_US
- added TP14: +16V5, TestPoint:TestPoint_Pad_D1.5mm, symbol Connector:TestPoint
- added TP40: IMU_INT1, TestPoint:TestPoint_Pad_D1.5mm, symbol Connector:TestPoint
- added TP41: IMU_INT2, TestPoint:TestPoint_Pad_D1.5mm, symbol Connector:TestPoint
- added TP44: COMP_RELAY_EN, TestPoint:TestPoint_Pad_D1.5mm, symbol Connector:TestPoint
- added TP45: AMP_REM_EN, TestPoint:TestPoint_Pad_D1.5mm, symbol Connector:TestPoint
- added TP48: ESP_BOOT, TestPoint:TestPoint_Pad_D1.5mm, symbol Connector:TestPoint
- added TP49: SIG_SINE, TestPoint:TestPoint_Pad_D1.5mm, symbol Connector:TestPoint
- added TP52: STATUS_RGB, TestPoint:TestPoint_Pad_D1.5mm, symbol Connector:TestPoint
- R86: renamed from D17; value ISO 3V3 (green) -> 1k; footprint LED_SMD:LED_0603_1608Metric -> Resistor_SMD:R_0603_1608Metric; symbol Device:LED -> Device:R_US; Product (none) -> https://www.digikey.com/en/products/result?keywords=RC0603F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
- R89: Product (none) -> https://www.digikey.com/en/products/result?keywords=RC0603F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
- TP10: value -15V -> +5V
- TP11: value +16V5 -> +3V3
- TP12: value -16V5 -> +15V
- TP13: value ISO_3V3 -> -15V
- TP15: renamed from TP14; value GND -> -16V5; footprint TestPoint:TestPoint_Loop_D2.50mm_Drill1.0mm -> TestPoint:TestPoint_Pad_D1.5mm
- TP16: renamed from TP15; value GND -> ISO_3V3; footprint TestPoint:TestPoint_Loop_D2.50mm_Drill1.0mm -> TestPoint:TestPoint_Pad_D1.5mm
- TP17: renamed from TP16; value GND -> +3V3_SG; footprint TestPoint:TestPoint_Loop_D2.50mm_Drill1.0mm -> TestPoint:TestPoint_Pad_D1.5mm
- TP18: renamed from TP17; value ISO_GND -> +3V3_COOL; footprint TestPoint:TestPoint_Loop_D2.50mm_Drill1.0mm -> TestPoint:TestPoint_Pad_D1.5mm
- TP19: renamed from TP18; value SPI_SCK -> +3V3_CH
- TP20: value SPI_MISO -> +5V_PS15
- TP21: renamed from TP22; value AD9833_FSYNC -> +5V_ISO
- TP22: renamed from TP23; value IMU_CS -> GND; footprint TestPoint:TestPoint_Pad_D1.5mm -> TestPoint:TestPoint_Loop_D2.50mm_Drill1.0mm
- TP23: renamed from TP25; value ADS1220_CS -> GND; footprint TestPoint:TestPoint_Pad_D1.5mm -> TestPoint:TestPoint_Loop_D2.50mm_Drill1.0mm
- TP24: renamed from TP27; value ACS_CS -> GND; footprint TestPoint:TestPoint_Pad_D1.5mm -> TestPoint:TestPoint_Loop_D2.50mm_Drill1.0mm
- TP25: renamed from TP29; value BRIDGE_RESET -> ISO_GND; footprint TestPoint:TestPoint_Pad_D1.5mm -> TestPoint:TestPoint_Loop_D2.50mm_Drill1.0mm
- TP26: renamed from TP31; value SCL -> SPI_SCK
- TP27: renamed from TP32; value IMU_INT1 -> SPI_MOSI
- TP28: renamed from TP33; value IMU_INT2 -> SPI_MISO
- TP29: renamed from TP34; value FAN_ALERT -> MCP4921_CS
- TP30: renamed from TP35; value PWR_KILL -> AD9833_FSYNC
- TP31: renamed from TP36; value COMP_RELAY_EN -> IMU_CS
- TP32: renamed from TP37; value AMP_REM_EN -> INA239_CS
- TP33: renamed from TP38; value PG_15V -> ADS1220_CS
- TP34: renamed from TP39; value ESP_EN -> BRIDGE_CS
- TP35: renamed from TP40; value ESP_BOOT -> ACS_CS
- TP36: renamed from TP41; value SIG_SINE -> ACS_MISO
- TP37: renamed from TP42; value NTC_ADC -> BRIDGE_RESET
- TP38: renamed from TP43; value FLOW_TACH -> SDA
- TP39: renamed from TP44; value STATUS_RGB -> SCL
- TP42: renamed from R86; value 1k -> FAN_ALERT; footprint Resistor_SMD:R_0603_1608Metric -> TestPoint:TestPoint_Pad_D1.5mm; symbol Device:R_US -> Connector:TestPoint
- TP43: renamed from D14; value 5V (yellow) -> PWR_KILL; footprint LED_SMD:LED_0603_1608Metric -> TestPoint:TestPoint_Pad_D1.5mm; symbol Device:LED -> Connector:TestPoint
- TP46: renamed from R87; value 4.7k -> PG_15V; footprint Resistor_SMD:R_0603_1608Metric -> TestPoint:TestPoint_Pad_D1.5mm; symbol Device:R_US -> Connector:TestPoint
- TP47: renamed from D15; value +15V (white) -> ESP_EN; footprint LED_SMD:LED_0603_1608Metric -> TestPoint:TestPoint_Pad_D1.5mm; symbol Device:LED -> Connector:TestPoint
- TP50: renamed from R88; value 4.7k -> NTC_ADC; footprint Resistor_SMD:R_0603_1608Metric -> TestPoint:TestPoint_Pad_D1.5mm; symbol Device:R_US -> Connector:TestPoint
- TP51: renamed from D16; value -15V (white) -> FLOW_TACH; footprint LED_SMD:LED_0603_1608Metric -> TestPoint:TestPoint_Pad_D1.5mm; symbol Device:LED -> Connector:TestPoint
- TP7: value +5V -> VIN
- TP8: value +3V3 -> +12V
- TP9: value +15V -> VSW
Connections:
- net +12V: now also TP8.1
- net +15V: now also TP12.1, R87.1; no longer TP46.1, TP9.1
- net +16V5: now also TP14.1; no longer TP11.1
- net +3V3: now also TP11.1; no longer TP8.1
- net +5V: now also R86.1, TP10.1; no longer TP42.1, TP7.1
- net -15V: now also TP13.1, R88.2; no longer TP10.1, TP50.2
- net -16V5: now also TP15.1; no longer TP12.1
- net ACS_CS: now also TP35.1; no longer TP24.1
- net ACS_MISO: now also TP36.1
- net AD9833_FSYNC: now also TP30.1; no longer TP21.1
- net ADS1220_CS: now also TP33.1; no longer TP23.1
- net AMP_REM_EN: now also TP45.1; no longer TP32.1
- net BRIDGE_CS: now also TP34.1
- net BRIDGE_RESET: now also TP37.1; no longer TP25.1
- net COMP_RELAY_EN: now also TP44.1; no longer TP31.1
- net ESP_BOOT: now also TP48.1; no longer TP35.1
- net ESP_EN: now also TP47.1; no longer TP34.1
- net FAN_ALERT: now also TP42.1; no longer TP29.1
- net FLOW_TACH: now also TP51.1; no longer TP38.1
- net GND: now also TP22.1, TP23.1, TP24.1, D14.1 (K), D15.1 (K), D16.2 (A); no longer TP15.1, TP16.1, TP17.1, TP43.1 (K), TP47.1 (K), TP51.2 (A)
- net IMU_CS: now also TP31.1; no longer TP22.1
- net IMU_INT1: now also TP40.1; no longer TP27.1
- net IMU_INT2: now also TP41.1; no longer TP28.1
- net INA239_CS: now also TP32.1
- net ISO_3V3: now also TP16.1; no longer TP13.1
- net ISO_GND: now also TP25.1, D17.1 (K); no longer R86.1 (K), TP18.1
- net MCP4921_CS: now also TP29.1
- net NTC_ADC: now also TP50.1; no longer TP37.1
- net PG_15V: now also TP46.1; no longer TP33.1
- net PWR_KILL: now also TP43.1; no longer TP30.1
- net SCL: now also TP39.1; no longer TP26.1
- net SDA: now also TP38.1
- net SIG_SINE: now also TP49.1; no longer TP36.1
- net SPI_MISO: now also TP28.1; no longer TP20.1
- net SPI_MOSI: now also TP27.1
- net SPI_SCK: now also TP26.1; no longer TP19.1
- net STATUS_RGB: now also TP52.1; no longer TP39.1
- net VIN: now also TP7.1
- net VSW: now also TP9.1
- net at R89.2: now also D17.2 (A); no longer R86.2 (A)
- new net: D16.1 (K), R88.1
- new net: D14.2 (A), R86.2
- new net: D15.2 (A), R87.2
- new net +3V3_CH: TP19.1
- new net +3V3_COOL: TP18.1
- new net +3V3_SG: TP17.1
- new net +5V_ISO: TP21.1
- new net +5V_PS15: TP20.1
Other:
- moved on the sheet: R86, TP15, TP16, TP17, TP18, TP19, TP20, TP21, TP22, TP23, TP24, TP25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

Commit message: Lay out the board for the Phoenix UCS 145-125 housing
Move to a 120 x 100 mm, 4-layer, blue-mask board for the UCS 145-125-F-CCD
7035 housing: housing mounting holes and restricted corners, ESP32 antenna
over a routed notch, one labelled section per schematic sheet with almost
every part on top. Placed, routed and cleaned up: DRC 0 errors, 0
unconnected, 0 schematic-parity issues; ERC 0; 193/193 datasheet rules.

- AGENTS.md: test points go on the same side as the part they test, close
  to it
- gen_pcb: test points held to their IC's side and within 8 mm; silkscreen
  check measures text by ink and also fails on pads, part outlines, section
  lines and pin-1 dots; titles along or up a border; connector labels and
  ESP32 pin names reserved before the passives; pin-1 dots only where the
  footprint has no mark; footprints carry the schematic's library links and
  fields; mounting holes are board-only H1-H4
- fix_route: generic clean-up (no old-board coordinate edits); removes GND
  vias in keep-outs or on foreign pads, links stranded ground pads, nudges
  squeezed tracks, handles back-side pour islands
- kicad_dru: fix the rule file (an invalid USB-C rule made KiCad ignore it);
  housing-corner and antenna keep-out part rules
- schematic: pad test points excluded from the BOM
- README / fabrication README updated for the new board

Co-Authored-By: Claude Opus 5.5 <noreply@anthropic.com>
Parts:
- TP10, TP11, TP12, TP13, TP14, TP15, TP16, TP17, TP18, TP19, TP20, TP21, TP26, TP27, TP28, TP29, TP30, TP31, TP32, TP33, TP34, TP35, TP36, TP37, TP38, TP39, TP40, TP41, TP42, TP43, TP44, TP45, TP46, TP47, TP48, TP49, TP50, TP51, TP52, TP7, TP8, TP9: now left out of the parts list
Changed lines of the file:
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@@
 		(body_style 1)
 		(exclude_from_sim no)
-		(in_bom yes)
+		(in_bom no)
 		(on_board yes)
 		(in_pos_files yes)
@@
 		(body_style 1)
 		(exclude_from_sim no)
-		(in_bom yes)
+		(in_bom no)
 		(on_board yes)
 		(in_pos_files yes)
@@
 		(body_style 1)
 		(exclude_from_sim no)
-		(in_bom yes)
+		(in_bom no)
 		(on_board yes)
 		(in_pos_files yes)
@@
 		(body_style 1)
 		(exclude_from_sim no)
-		(in_bom yes)
+		(in_bom no)
 		(on_board yes)
 		(in_pos_files yes)
@@
 		(body_style 1)
 		(exclude_from_sim no)
-		(in_bom yes)
+		(in_bom no)
 		(on_board yes)
 		(in_pos_files yes)
@@
 		(body_style 1)
 		(exclude_from_sim no)
-		(in_bom yes)
+		(in_bom no)
 		(on_board yes)
 		(in_pos_files yes)
@@
 		(body_style 1)
 		(exclude_from_sim no)
-		(in_bom yes)
+		(in_bom no)
 		(on_board yes)
 		(in_pos_files yes)
@@
 		(body_style 1)
 		(exclude_from_sim no)
-		(in_bom yes)
+		(in_bom no)
 		(on_board yes)
 		(in_pos_files yes)
@@
 		(body_style 1)
 		(exclude_from_sim no)
-		(in_bom yes)
+		(in_bom no)
 		(on_board yes)
 		(in_pos_files yes)
@@
 		(body_style 1)
 		(exclude_from_sim no)
-		(in_bom yes)
+		(in_bom no)
 		(on_board yes)
 		(in_pos_files yes)
@@
 		(body_style 1)
 		(exclude_from_sim no)
-		(in_bom yes)
+		(in_bom no)
 		(on_board yes)
 		(in_pos_files yes)
@@
 		(body_style 1)
 		(exclude_from_sim no)
-		(in_bom yes)
+		(in_bom no)
 		(on_board yes)
 		(in_pos_files yes)
@@
 		(body_style 1)
 		(exclude_from_sim no)
-		(in_bom yes)
+		(in_bom no)
 		(on_board yes)
 		(in_pos_files yes)
@@
 		(body_style 1)
 		(exclude_from_sim no)
-		(in_bom yes)
+		(in_bom no)
 		(on_board yes)
 		(in_pos_files yes)
@@
 		(body_style 1)
 		(exclude_from_sim no)
-		(in_bom yes)
+		(in_bom no)
 		(on_board yes)
 		(in_pos_files yes)
@@
 		(body_style 1)
 		(exclude_from_sim no)
-		(in_bom yes)
+		(in_bom no)
 		(on_board yes)
 		(in_pos_files yes)
@@
 		(body_style 1)
 		(exclude_from_sim no)
-		(in_bom yes)
+		(in_bom no)
 		(on_board yes)
 		(in_pos_files yes)
@@
 		(body_style 1)
 		(exclude_from_sim no)
-		(in_bom yes)
+		(in_bom no)
 		(on_board yes)
 		(in_pos_files yes)
@@
 		(body_style 1)
 		(exclude_from_sim no)
-		(in_bom yes)
+		(in_bom no)
 		(on_board yes)
 		(in_pos_files yes)
@@
 		(body_style 1)
 		(exclude_from_sim no)
-		(in_bom yes)
+		(in_bom no)
 		(on_board yes)
 		(in_pos_files yes)
@@
 		(body_style 1)
 		(exclude_from_sim no)
-		(in_bom yes)
+		(in_bom no)
 		(on_board yes)
 		(in_pos_files yes)
@@
 		(body_style 1)
 		(exclude_from_sim no)
-		(in_bom yes)
+		(in_bom no)
 		(on_board yes)
 		(in_pos_files yes)
@@
 		(body_style 1)
 		(exclude_from_sim no)
-		(in_bom yes)
+		(in_bom no)
 		(on_board yes)
 		(in_pos_files yes)
@@
 		(body_style 1)
 		(exclude_from_sim no)
-		(in_bom yes)
+		(in_bom no)
 		(on_board yes)
 		(in_pos_files yes)
@@
 		(body_style 1)
 		(exclude_from_sim no)
-		(in_bom yes)
+		(in_bom no)
 		(on_board yes)
 		(in_pos_files yes)
@@
 		(body_style 1)
 		(exclude_from_sim no)
-		(in_bom yes)
+		(in_bom no)
 		(on_board yes)
 		(in_pos_files yes)
@@
 		(body_style 1)
 		(exclude_from_sim no)
-		(in_bom yes)
+		(in_bom no)
 		(on_board yes)
 		(in_pos_files yes)
@@
 		(body_style 1)
 		(exclude_from_sim no)
-		(in_bom yes)
+		(in_bom no)
 		(on_board yes)
 		(in_pos_files yes)
@@
 		(body_style 1)
 		(exclude_from_sim no)
-		(in_bom yes)
+		(in_bom no)
 		(on_board yes)
 		(in_pos_files yes)
@@
 		(body_style 1)
 		(exclude_from_sim no)
-		(in_bom yes)
+		(in_bom no)
 		(on_board yes)
 		(in_pos_files yes)
@@
 		(body_style 1)
 		(exclude_from_sim no)
-		(in_bom yes)
+		(in_bom no)
 		(on_board yes)
 		(in_pos_files yes)
@@
 		(body_style 1)
 		(exclude_from_sim no)
-		(in_bom yes)
+		(in_bom no)
 		(on_board yes)
 		(in_pos_files yes)
@@
 		(body_style 1)
 		(exclude_from_sim no)
-		(in_bom yes)
+		(in_bom no)
 		(on_board yes)
 		(in_pos_files yes)
@@
 		(body_style 1)
 		(exclude_from_sim no)
-		(in_bom yes)
+		(in_bom no)
 		(on_board yes)
 		(in_pos_files yes)
@@
 		(body_style 1)
 		(exclude_from_sim no)
-		(in_bom yes)
+		(in_bom no)
 		(on_board yes)
 		(in_pos_files yes)
@@
 		(body_style 1)
 		(exclude_from_sim no)
-		(in_bom yes)
+		(in_bom no)
 		(on_board yes)
 		(in_pos_files yes)
@@
 		(body_style 1)
 		(exclude_from_sim no)
-		(in_bom yes)
+		(in_bom no)
 		(on_board yes)
 		(in_pos_files yes)
@@
 		(body_style 1)
 		(exclude_from_sim no)
-		(in_bom yes)
+		(in_bom no)
 		(on_board yes)
 		(in_pos_files yes)
@@
 		(body_style 1)
 		(exclude_from_sim no)
-		(in_bom yes)
+		(in_bom no)
 		(on_board yes)
 		(in_pos_files yes)
@@
 		(body_style 1)
 		(exclude_from_sim no)
-		(in_bom yes)
+		(in_bom no)
 		(on_board yes)
 		(in_pos_files yes)
@@
 		(body_style 1)
 		(exclude_from_sim no)
-		(in_bom yes)
+		(in_bom no)
 		(on_board yes)
 		(in_pos_files yes)
@@
 		(body_style 1)
 		(exclude_from_sim no)
-		(in_bom yes)
+		(in_bom no)
 		(on_board yes)
 		(in_pos_files yes)
