File: hardware/kicad/sheets/debug.kicad_sch (KiCad schematic)
At the start: 54 parts

Commit message: Ground the M12 shield, order the ground loops, name the J14 cable parts
- J10: shielded symbol (Conn_01x04_Shielded); the M12 shield pin and its
  four shell legs are pad SH, tied to GND
- TP22-TP25: Keystone 5001 black miniature PC test points (KiCad
  TestPoint_Keystone_5000-5004 footprint, 1.02 mm hole per Keystone's
  drawing); now in the BOM, the bare pad test points stay out
- J14 BOM note: cable housing Molex 5054320801 with 505431 terminals, or
  tin pre-crimped leads 797581148 / 797581149 (from molex.com)

Only netlist change: GND gains J10 SH. DRC 0 errors, 0 unconnected, 0
schematic-parity issues; ERC 0; 193/193 datasheet rules.

Co-Authored-By: Claude Opus 5.5 <noreply@anthropic.com>
Parts:
- removed R86, R89: 1k, Resistor_SMD:R_0603_1608Metric, symbol Device:R_US
- removed R87, R88: 4.7k, Resistor_SMD:R_0603_1608Metric, symbol Device:R_US
- removed TP21: +5V_ISO, TestPoint:TestPoint_Pad_D1.5mm, symbol Connector:TestPoint
- removed TP26: SPI_SCK, TestPoint:TestPoint_Pad_D1.5mm, symbol Connector:TestPoint
- added D14: 5V (yellow), LED_SMD:LED_0603_1608Metric, symbol Device:LED
- added D15: +15V (white), LED_SMD:LED_0603_1608Metric, symbol Device:LED
- added D16: -15V (white), LED_SMD:LED_0603_1608Metric, symbol Device:LED
- added D17: ISO 3V3 (green), LED_SMD:LED_0603_1608Metric, symbol Device:LED
- added TP22: GND, TestPoint:TestPoint_Keystone_5000-5004_Miniature, symbol Connector:TestPoint
- added TP52: STATUS_RGB, TestPoint:TestPoint_Pad_D1.5mm, symbol Connector:TestPoint
- R86: renamed from D14; value 5V (yellow) -> 1k; footprint LED_SMD:LED_0603_1608Metric -> Resistor_SMD:R_0603_1608Metric; symbol Device:LED -> Device:R_US; Product https://www.digikey.com/en/products/result?keywords=LTST-C1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 -> https://www.digikey.com/en/products/result?keywords=RC0603F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
- R87: renamed from D15; value +15V (white) -> 4.7k; footprint LED_SMD:LED_0603_1608Metric -> Resistor_SMD:R_0603_1608Metric; symbol Device:LED -> Device:R_US; Product https://www.digikey.com/en/products/result?keywords=LTW-C19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 -> https://www.digikey.com/en/products/result?keywords=RC0603F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
- R88: renamed from D16; value -15V (white) -> 4.7k; footprint LED_SMD:LED_0603_1608Metric -> Resistor_SMD:R_0603_1608Metric; symbol Device:LED -> Device:R_US; Product https://www.digikey.com/en/products/result?keywords=LTW-C19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 -> https://www.digikey.com/en/products/result?keywords=RC0603F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
- R89: renamed from D17; value ISO 3V3 (green) -> 1k; footprint LED_SMD:LED_0603_1608Metric -> Resistor_SMD:R_0603_1608Metric; symbol Device:LED -> Device:R_US; Product https://www.digikey.com/en/products/result?keywords=LTST-C1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 -> https://www.digikey.com/en/products/result?keywords=RC0603F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
- TP21: renamed from TP22; value GND -> +5V_ISO; footprint TestPoint:TestPoint_Loop_D2.50mm_Drill1.0mm -> TestPoint:TestPoint_Pad_D1.5mm; now left out of the parts list
- TP23, TP24, TP25: footprint TestPoint:TestPoint_Loop_D2.50mm_Drill1.0mm -> TestPoint:TestPoint_Keystone_5000-5004_Miniature; Product (none) -> https://www.keyelco.com/product.cfm/product_id/1310
- TP26: renamed from TP27; value SPI_MOSI -> SPI_SCK
- TP27: renamed from TP28; value SPI_MISO -> SPI_MOSI
- TP28: renamed from TP29; value MCP4921_CS -> SPI_MISO
- TP29: renamed from TP30; value AD9833_FSYNC -> MCP4921_CS
- TP30: renamed from TP31; value IMU_CS -> AD9833_FSYNC
- TP31: renamed from TP32; value INA239_CS -> IMU_CS
- TP32: renamed from TP33; value ADS1220_CS -> INA239_CS
- TP33: renamed from TP34; value BRIDGE_CS -> ADS1220_CS
- TP34: renamed from TP35; value ACS_CS -> BRIDGE_CS
- TP35: renamed from TP36; value ACS_MISO -> ACS_CS
- TP36: renamed from TP37; value BRIDGE_RESET -> ACS_MISO
- TP37: renamed from TP38; value SDA -> BRIDGE_RESET
- TP38: renamed from TP39; value SCL -> SDA
- TP39: renamed from TP40; value IMU_INT1 -> SCL
- TP40: renamed from TP41; value IMU_INT2 -> IMU_INT1
- TP41: renamed from TP42; value FAN_ALERT -> IMU_INT2
- TP42: renamed from TP43; value PWR_KILL -> FAN_ALERT
- TP43: renamed from TP44; value COMP_RELAY_EN -> PWR_KILL
- TP44: renamed from TP45; value AMP_REM_EN -> COMP_RELAY_EN
- TP45: renamed from TP46; value PG_15V -> AMP_REM_EN
- TP46: renamed from TP47; value ESP_EN -> PG_15V
- TP47: renamed from TP48; value ESP_BOOT -> ESP_EN
- TP48: renamed from TP49; value SIG_SINE -> ESP_BOOT
- TP49: renamed from TP50; value NTC_ADC -> SIG_SINE
- TP50: renamed from TP51; value FLOW_TACH -> NTC_ADC
- TP51: renamed from TP52; value STATUS_RGB -> FLOW_TACH
Connections:
- net +15V: now also R87.1
- net +5V: now also R86.1
- net +5V_ISO: now also TP21.1
- net -15V: now also R88.2
- net ACS_CS: now also TP35.1; no longer TP34.1
- net ACS_MISO: now also TP36.1; no longer TP35.1
- net AD9833_FSYNC: now also TP30.1; no longer TP29.1
- net ADS1220_CS: now also TP33.1; no longer TP32.1
- net AMP_REM_EN: now also TP45.1; no longer TP44.1
- net BRIDGE_CS: now also TP34.1; no longer TP33.1
- net BRIDGE_RESET: now also TP37.1; no longer TP36.1
- net COMP_RELAY_EN: now also TP44.1; no longer TP43.1
- net ESP_BOOT: now also TP48.1; no longer TP47.1
- net ESP_EN: now also TP47.1; no longer TP46.1
- net FAN_ALERT: now also TP42.1; no longer TP41.1
- net FLOW_TACH: now also TP51.1; no longer TP50.1
- net GND: now also D14.1 (K), D15.1 (K), D16.2 (A), TP22.1; no longer R86.1 (K), R87.1 (K), R88.2 (A), TP21.1
- net IMU_CS: now also TP31.1; no longer TP30.1
- net IMU_INT1: now also TP40.1; no longer TP39.1
- net IMU_INT2: now also TP41.1; no longer TP40.1
- net INA239_CS: now also TP32.1; no longer TP31.1
- net ISO_3V3: now also R89.1
- net ISO_GND: now also D17.1 (K); no longer R89.1 (K)
- net MCP4921_CS: now also TP29.1; no longer TP28.1
- net NTC_ADC: now also TP50.1; no longer TP49.1
- net PG_15V: now also TP46.1; no longer TP45.1
- net PWR_KILL: now also TP43.1; no longer TP42.1
- net SCL: now also TP39.1; no longer TP38.1
- net SDA: now also TP38.1; no longer TP37.1
- net SIG_SINE: now also TP49.1; no longer TP48.1
- net SPI_MISO: now also TP28.1; no longer TP27.1
- net SPI_MOSI: now also TP27.1; no longer TP26.1
- net SPI_SCK: now also TP26.1
- net STATUS_RGB: now also TP52.1; no longer TP51.1
- net at R88.1: now also D16.1 (K)
- net at R89.2: now also D17.2 (A)
- net at R86.2: now also D14.2 (A)
- net at R87.2: now also D15.2 (A)
Other:
- moved on the sheet: R86, R87, R88, R89, TP21, TP26, TP27, TP28, TP29, TP30, TP31, TP32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
