File: hardware/kicad/sheets/power_input.kicad_sch (KiCad schematic)
At the start: 5 parts, among them J2 12V IN

Commit message: WIP: restructure PCB for the Phoenix UCS 125-87 housing
Work in progress, layout not finished: about 90 parts still do not fit
their sections and the board is not routed.

- Right-angle connectors: Phoenix MSTBA 2,5 / MC 1,5, JST XH side entry,
  Hirose DF13, Molex 505448-0871 (new footprint from the Molex drawing)
- Datasheet and product links on every symbol (tools/part_links.py)
- Test points so every IC has one on its own nets
- gen_pcb.py: 100 x 62 mm two-sided board, housing holes and restricted
  corners, ESP32 antenna notch, one section per sheet, board ID block,
  ESP32 pin names, pin-1 marks, blue mask
- Housing drawings in hardware/housing/

Co-Authored-By: Claude Opus 5.5 <noreply@anthropic.com>
Parts:
- removed J2: 12V IN, TerminalBlock_Phoenix:TerminalBlock_Phoenix_MKDS-1,5-2-5.08_1x02_P5.08mm_Horizontal, symbol Connector:Screw_Terminal_01x02
- added F1: 5A backup, Fuse:Fuse_Littelfuse-NANO2-451_453, symbol Device:Fuse
- C6: Product (none) -> https://www.digikey.com/en/products/result?keywords=EEE-FK1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
- C7: Product (none) -> https://www.digikey.com/en/products/result?keywords=CL21B10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
- D1: Product (none) -> https://www.digikey.com/en/products/result?keywords=SMBJ16A
- J2: renamed from F1; value 5A backup -> 12V IN; footprint Fuse:Fuse_Littelfuse-NANO2-451_453 -> Connector_Phoenix_MSTB:PhoenixContact_MSTBA_2,5_2-G-5,08_1x02_P5.08mm_Horizontal; symbol Device:Fuse -> Connector:Screw_Terminal_01x02; Product (none) -> https://www.phoenixcontact.com/en-us/products/pcb-header-ms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
Connections:
- net GND: now also J2.2 (Pin_2)
- net VIN: now also F1.2; no longer J2.2
- net at J2.1 (Pin_1): now also F1.1
