File: hardware/kicad/sheets/supply_switches.kicad_sch (KiCad schematic)
At the start: 12 parts

Commit message: Split cooling into Water Cooling and Cold Head Temp sections, each with a supply jumper and LED
Water Cooling (EMC2303, SC18IS604 bridge, NTC, fan/pump/flow) sits behind JP4
on +3V3_COOL together with its pull-ups. Cold Head Temp (ADS1220, PT1000) gets
a new jumper JP5 and LED D22 on +3V3_CH. JP2 is relabelled for the +-15V rails
and moved into the RAILS +-15V box. PCB regenerated with two silk boxes, routed,
leftovers finished with a grid router; board render added to the main README.

Co-Authored-By: Claude Sonnet 5.5 <noreply@anthropic.com>
Parts:
- added D22: COLD HEAD +3V3 (ADS1220 RTD ADC) (green), LED_SMD:LED_0603_1608Metric, symbol Device:LED
- added JP5: EN CH, Connector_PinHeader_1.27mm:PinHeader_1x02_P1.27mm_Vertical, symbol Connector_Generic:Conn_01x02
- added R100: 1k, Resistor_SMD:R_0603_1608Metric, symbol Device:R_US
- D19: value +-15V SUPPLY +5V IN (green) -> +-15V RAILS ENABLE (+5V IN) (green)
- D21: value COOLING +3V3 (EMC2303, RTD ADC, I2C BRIDGE) (green) -> WATER COOLING +3V3 (EMC2303, I2C BRIDGE, NTC) (green)
Connections:
- net +3V3: now also JP5.1 (Pin_1)
- net GND: now also D22.1 (K)
- new net: D22.2 (A), R100.2
- new net +3V3_CH: JP5.2 (Pin_2), R100.1
Other:
- note added: "+-15V RAILS ENABLE (+5V IN)"
- note added: "COLD HEAD +3V3 (ADS1220 RTD ADC)"
- note added: "WATER COOLING +3V3 (EMC2303, I2C BRIDGE, NTC)"
- note removed: "+-15V SUPPLY +5V IN"
- note removed: "COOLING +3V3 (EMC2303, RTD ADC, I2C BRIDGE)"

Commit message: Log +-15 V power-good changes and add one LED per LT3097 PG pin
Firmware
- amplifier: configure PG_15V_N_PIN (GPIO43, active LOW), log the starting
  state and every debounced change (PowerGoodMonitor in power_good.h);
  amplifier::isPowerGood() reports the level. The lines reach the dashboard
  console through the logger ring buffer.
- dashboard: console colours for "power lost" (red), "power restored" and
  "power good: yes" (green), "power good: no" (yellow).
- native tests for the debounce logic and the amplifier stub.

Hardware
- power_good sheet: PGP and PGN each drive their own node (220k/62k from
  +15 V) and a green LED (D24 +15 V, D25 -15 V) through a BSS138W; a BAT54AW
  with a 10k pull-up ANDs the nodes into PG_15V, so the REM interlock and the
  PG_15V_N flag are unchanged.
- 0402 resistors, SOT-323 FETs and one BAT54AW so the stage fits the power
  box; Power Good parts are placed last in gen_pcb.py.
- Board re-routed with Freerouting 2.5.0 and cleaned with fix_route.py: DRC
  0 unconnected, no copper violations. Gerbers, JLCPCB zip, renders, BOM, CPL
  and schematic PDF regenerated; datasheet rules 193/193.

Co-Authored-By: Claude Sonnet 5.5 <noreply@anthropic.com>
Parts:
- removed D18: SIGNAL GEN +3V3 (green), LED_SMD:LED_0603_1608Metric, symbol Device:LED
- removed JP1: EN SG3, Connector_PinHeader_1.27mm:PinHeader_1x02_P1.27mm_Vertical, symbol Connector_Generic:Conn_01x02
- removed JP2: EN PS15, Connector_PinHeader_1.27mm:PinHeader_1x02_P1.27mm_Vertical, symbol Connector_Generic:Conn_01x02
- removed JP3: EN ISO5, Connector_PinHeader_1.27mm:PinHeader_1x02_P1.27mm_Vertical, symbol Connector_Generic:Conn_01x02
- removed JP4: EN COOL, Connector_PinHeader_1.27mm:PinHeader_1x02_P1.27mm_Vertical, symbol Connector_Generic:Conn_01x02
- added D21: WATER COOLING +3V3 (EMC2303, I2C BRIDGE, NTC) (gr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, LED_SMD:LED_0603_1608Metric, symbol Device:LED
- added D22: COLD HEAD +3V3 (ADS1220 RTD ADC) (green), LED_SMD:LED_0603_1608Metric, symbol Device:LED
- added R100, R98, R99: 1k, Resistor_SMD:R_0603_1608Metric, symbol Device:R_US
- D18: renamed from R98; value 1k -> SIGNAL GEN +3V3 (green); footprint Resistor_SMD:R_0603_1608Metric -> LED_SMD:LED_0603_1608Metric; symbol Device:R_US -> Device:LED
- D19: renamed from R99; value 1k -> +-15V RAILS ENABLE (+5V IN) (green); footprint Resistor_SMD:R_0603_1608Metric -> LED_SMD:LED_0603_1608Metric; symbol Device:R_US -> Device:LED
- D20: renamed from R100; value 1k -> ISOLATED SUPPLY +5V IN (green); footprint Resistor_SMD:R_0603_1608Metric -> LED_SMD:LED_0603_1608Metric; symbol Device:R_US -> Device:LED
- JP1: renamed from D19; value +-15V RAILS ENABLE (+5V IN) (green) -> EN SG3; footprint LED_SMD:LED_0603_1608Metric -> Connector_PinHeader_1.27mm:PinHeader_1x02_P1.27mm_Vertical; symbol Device:LED -> Connector_Generic:Conn_01x02
- JP2: renamed from D20; value ISOLATED SUPPLY +5V IN (green) -> EN PS15; footprint LED_SMD:LED_0603_1608Metric -> Connector_PinHeader_1.27mm:PinHeader_1x02_P1.27mm_Vertical; symbol Device:LED -> Connector_Generic:Conn_01x02
- JP3: renamed from D21; value WATER COOLING +3V3 (EMC2303, I2C BRIDGE, NTC) (green) -> EN ISO5; footprint LED_SMD:LED_0603_1608Metric -> Connector_PinHeader_1.27mm:PinHeader_1x02_P1.27mm_Vertical; symbol Device:LED -> Connector_Generic:Conn_01x02
- JP4: renamed from D22; value COLD HEAD +3V3 (ADS1220 RTD ADC) (green) -> EN COOL; footprint LED_SMD:LED_0603_1608Metric -> Connector_PinHeader_1.27mm:PinHeader_1x02_P1.27mm_Vertical; symbol Device:LED -> Connector_Generic:Conn_01x02
Connections:
- net +3V3: now also JP1.1 (Pin_1), JP4.1 (Pin_1)
- net +3V3_CH: now also R100.1; no longer D20.1
- net +3V3_COOL: now also JP4.2 (Pin_2), R99.1; no longer D19.1
- net +3V3_SG: now also JP1.2 (Pin_2)
- net +5V: now also JP2.1 (Pin_1), JP3.1 (Pin_1)
- net +5V_ISO: now also JP3.2 (Pin_2), R98.1; no longer D18.1
- net +5V_PS15: now also JP2.2 (Pin_2)
- net GND: now also D18.1 (K), D19.1 (K), D20.1 (K), D21.1 (K), D22.1 (K); no longer JP1.1 (K), JP2.1 (K), JP3.1 (K), JP4.1 (K)
- net at R97.2: now also D19.2 (A); no longer JP1.2 (A)
- net at D18.2 (A): now also R96.2; no longer JP2.2 (A)
- net at D20.2 (A): now also R98.2; no longer JP4.2 (A)
- new net: D21.2 (A), R99.2
- new net: D22.2 (A), R100.2
Other:
- moved on the sheet: D18, D19, D20

Commit message: WIP: restructure PCB for the Phoenix UCS 125-87 housing
Work in progress, layout not finished: about 90 parts still do not fit
their sections and the board is not routed.

- Right-angle connectors: Phoenix MSTBA 2,5 / MC 1,5, JST XH side entry,
  Hirose DF13, Molex 505448-0871 (new footprint from the Molex drawing)
- Datasheet and product links on every symbol (tools/part_links.py)
- Test points so every IC has one on its own nets
- gen_pcb.py: 100 x 62 mm two-sided board, housing holes and restricted
  corners, ESP32 antenna notch, one section per sheet, board ID block,
  ESP32 pin names, pin-1 marks, blue mask
- Housing drawings in hardware/housing/

Co-Authored-By: Claude Opus 5.5 <noreply@anthropic.com>
Parts:
- D18, D19, D20, D21, D22: Product (none) -> https://www.digikey.com/en/products/result?keywords=LTST-C1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
- R100, R96, R97, R98, R99: Product (none) -> https://www.digikey.com/en/products/result?keywords=RC0603F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

Commit message: Ground the M12 shield, order the ground loops, name the J14 cable parts
- J10: shielded symbol (Conn_01x04_Shielded); the M12 shield pin and its
  four shell legs are pad SH, tied to GND
- TP22-TP25: Keystone 5001 black miniature PC test points (KiCad
  TestPoint_Keystone_5000-5004 footprint, 1.02 mm hole per Keystone's
  drawing); now in the BOM, the bare pad test points stay out
- J14 BOM note: cable housing Molex 5054320801 with 505431 terminals, or
  tin pre-crimped leads 797581148 / 797581149 (from molex.com)

Only netlist change: GND gains J10 SH. DRC 0 errors, 0 unconnected, 0
schematic-parity issues; ERC 0; 193/193 datasheet rules.

Co-Authored-By: Claude Opus 5.5 <noreply@anthropic.com>
Parts:
- removed R100, R96, R97, R98, R99: 1k, Resistor_SMD:R_0603_1608Metric, symbol Device:R_US
- added D22: COLD HEAD +3V3 (ADS1220 RTD ADC) (green), LED_SMD:LED_0603_1608Metric, symbol Device:LED
- added JP2: EN PS15, Connector_PinHeader_1.27mm:PinHeader_1x02_P1.27mm_Vertical, symbol Connector_Generic:Conn_01x02
- added JP3: EN ISO5, Connector_PinHeader_1.27mm:PinHeader_1x02_P1.27mm_Vertical, symbol Connector_Generic:Conn_01x02
- added JP4: EN COOL, Connector_PinHeader_1.27mm:PinHeader_1x02_P1.27mm_Vertical, symbol Connector_Generic:Conn_01x02
- added JP5: EN CH, Connector_PinHeader_1.27mm:PinHeader_1x02_P1.27mm_Vertical, symbol Connector_Generic:Conn_01x02
- D18: renamed from JP2; value EN PS15 -> SIGNAL GEN +3V3 (green); footprint Connector_PinHeader_1.27mm:PinHeader_1x02_P1.27mm_Vertical -> LED_SMD:LED_0603_1608Metric; symbol Connector_Generic:Conn_01x02 -> Device:LED; Product (none) -> https://www.digikey.com/en/products/result?keywords=LTST-C1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
- D19: renamed from JP3; value EN ISO5 -> +-15V RAILS ENABLE (+5V IN) (green); footprint Connector_PinHeader_1.27mm:PinHeader_1x02_P1.27mm_Vertical -> LED_SMD:LED_0603_1608Metric; symbol Connector_Generic:Conn_01x02 -> Device:LED; Product (none) -> https://www.digikey.com/en/products/result?keywords=LTST-C1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
- D20: renamed from JP4; value EN COOL -> ISOLATED SUPPLY +5V IN (green); footprint Connector_PinHeader_1.27mm:PinHeader_1x02_P1.27mm_Vertical -> LED_SMD:LED_0603_1608Metric; symbol Connector_Generic:Conn_01x02 -> Device:LED; Product (none) -> https://www.digikey.com/en/products/result?keywords=LTST-C1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
- D21: renamed from JP5; value EN CH -> WATER COOLING +3V3 (EMC2303, I2C BRIDGE, NTC) (green); footprint Connector_PinHeader_1.27mm:PinHeader_1x02_P1.27mm_Vertical -> LED_SMD:LED_0603_1608Metric; symbol Connector_Generic:Conn_01x02 -> Device:LED; Product (none) -> https://www.digikey.com/en/products/result?keywords=LTST-C1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
- R100: renamed from D22; value COLD HEAD +3V3 (ADS1220 RTD ADC) (green) -> 1k; footprint LED_SMD:LED_0603_1608Metric -> Resistor_SMD:R_0603_1608Metric; symbol Device:LED -> Device:R_US; Product https://www.digikey.com/en/products/result?keywords=LTST-C1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 -> https://www.digikey.com/en/products/result?keywords=RC0603F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
- R96: renamed from D18; value SIGNAL GEN +3V3 (green) -> 1k; footprint LED_SMD:LED_0603_1608Metric -> Resistor_SMD:R_0603_1608Metric; symbol Device:LED -> Device:R_US; Product https://www.digikey.com/en/products/result?keywords=LTST-C1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 -> https://www.digikey.com/en/products/result?keywords=RC0603F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
- R97: renamed from D19; value +-15V RAILS ENABLE (+5V IN) (green) -> 1k; footprint LED_SMD:LED_0603_1608Metric -> Resistor_SMD:R_0603_1608Metric; symbol Device:LED -> Device:R_US; Product https://www.digikey.com/en/products/result?keywords=LTST-C1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 -> https://www.digikey.com/en/products/result?keywords=RC0603F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
- R98: renamed from D20; value ISOLATED SUPPLY +5V IN (green) -> 1k; footprint LED_SMD:LED_0603_1608Metric -> Resistor_SMD:R_0603_1608Metric; symbol Device:LED -> Device:R_US; Product https://www.digikey.com/en/products/result?keywords=LTST-C1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 -> https://www.digikey.com/en/products/result?keywords=RC0603F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
- R99: renamed from D21; value WATER COOLING +3V3 (EMC2303, I2C BRIDGE, NTC) (green) -> 1k; footprint LED_SMD:LED_0603_1608Metric -> Resistor_SMD:R_0603_1608Metric; symbol Device:LED -> Device:R_US; Product https://www.digikey.com/en/products/result?keywords=LTST-C1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 -> https://www.digikey.com/en/products/result?keywords=RC0603F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
Connections:
- net +3V3: now also JP4.1 (Pin_1), JP5.1 (Pin_1); no longer D20.1 (Pin_1), D21.1 (Pin_1)
- net +3V3_CH: now also R100.1, JP5.2 (Pin_2); no longer D21.2 (Pin_2)
- net +3V3_COOL: now also R99.1, JP4.2 (Pin_2); no longer D20.2 (Pin_2)
- net +3V3_SG: now also R96.1
- net +5V: now also JP2.1 (Pin_1), JP3.1 (Pin_1); no longer D18.1 (Pin_1), D19.1 (Pin_1)
- net +5V_ISO: now also R98.1, JP3.2 (Pin_2); no longer D19.2 (Pin_2)
- net +5V_PS15: now also R97.1, JP2.2 (Pin_2); no longer D18.2 (Pin_2)
- net GND: now also D18.1 (K), D19.1 (K), D20.1 (K), D21.1 (K), D22.1 (K); no longer R100.1 (K), R96.1 (K), R97.1 (K), R98.1 (K), R99.1 (K)
- net at R96.2: now also D18.2 (A)
- net at R97.2: now also D19.2 (A)
- net at R98.2: now also D20.2 (A)
- net at R99.2: now also D21.2 (A)
- net at R100.2: now also D22.2 (A)
Other:
- moved on the sheet: R100, R96, R97, R98, R99
