File: hardware/kicad/sheets/system_current.kicad_sch (KiCad schematic)
At the start: 15 parts, among them U23 INA239AIDGSR

Commit message: Replace the ±15 V LDOs with one LT3097 and add a power-good interlock
- rails_15v: ADP7142 + ADP7182 replaced by one LT3097 (±14.7 V, 147 k SET
  resistors); the ADP5071 output caps are now 22 uF / 50 V and double as the
  LT3097 inputs. PGP / PGN make the PG_15V node (fed from +15 V, so it reads
  0 V if a rail is missing).
- amp_control: a series BSS138 (Q9) gated by PG_15V blocks AMP_REM unless
  both rails are good. New power_good sheet: LED (D23) and the active-low
  PG_15V_N flag on GPIO43 (PG_15V_N_PIN).
- Tooling: LT3097 symbol, footprint and 3D envelope; datasheet rules (191),
  GPIO check, BOM tables, floor plan, PAD_BRIDGES and pre-placed GND vias in
  gen_pcb.py, new fix_route.py for post-route clean-up.
- Board regenerated and routed with Freerouting 2.5.0: DRC 0 unconnected,
  0 schematic-parity issues, no copper violations. Gerbers, JLCPCB zip,
  renders, BOM, CPL and schematic PDF regenerated.

Co-Authored-By: Claude Sonnet 5.5 <noreply@anthropic.com>
Parts:
- removed C72: 470nF, Capacitor_SMD:C_0805_2012Metric, symbol Device:C
- removed R65: 15m, Resistor_SMD:R_2512_6332Metric, symbol Device:R_US
- removed R67: 49.9, Resistor_SMD:R_0603_1608Metric, symbol Device:R_US
- added C73: 100nF, Capacitor_SMD:C_0603_1608Metric, symbol Device:C
- added C74: 1uF, Capacitor_SMD:C_0805_2012Metric, symbol Device:C
- added D8: PWR (green), LED_SMD:LED_0603_1608Metric, symbol Device:LED
- C72: renamed from C74; value 1uF -> 470nF
- R65: renamed from R69; value 10k -> 15m; footprint Resistor_SMD:R_0603_1608Metric -> Resistor_SMD:R_2512_6332Metric
- R67: renamed from C73; value 100nF -> 49.9; footprint Capacitor_SMD:C_0603_1608Metric -> Resistor_SMD:R_0603_1608Metric; symbol Device:C -> Device:R_US
- R69: renamed from D8; value PWR (green) -> 10k; footprint LED_SMD:LED_0603_1608Metric -> Resistor_SMD:R_0603_1608Metric; symbol Device:LED -> Device:R_US
Connections:
- net +12V: now also R65.2
- net +3V3: now also R69.2, C73.1, C74.1; no longer C72.1, R65.2, R67.1
- net GND: now also C73.2, C74.2, D8.1 (K); no longer C72.2, R67.2, R69.1 (K)
- net VSW: now also R65.1, R67.1
- net at R66.2, U23.8 (VBUS), U23.9 (IN-): now also C72.1
- net at R71.2: now also D8.2 (A); no longer R69.2 (A)
- net at U23.10 (IN+): now also C72.2, R67.2
- net at D7.1 (K), U23.3 (~{ALERT}): now also R69.1; no longer R65.1
Other:
- moved on the sheet: C72, R65, R69

Commit message: Log +-15 V power-good changes and add one LED per LT3097 PG pin
Firmware
- amplifier: configure PG_15V_N_PIN (GPIO43, active LOW), log the starting
  state and every debounced change (PowerGoodMonitor in power_good.h);
  amplifier::isPowerGood() reports the level. The lines reach the dashboard
  console through the logger ring buffer.
- dashboard: console colours for "power lost" (red), "power restored" and
  "power good: yes" (green), "power good: no" (yellow).
- native tests for the debounce logic and the amplifier stub.

Hardware
- power_good sheet: PGP and PGN each drive their own node (220k/62k from
  +15 V) and a green LED (D24 +15 V, D25 -15 V) through a BSS138W; a BAT54AW
  with a 10k pull-up ANDs the nodes into PG_15V, so the REM interlock and the
  PG_15V_N flag are unchanged.
- 0402 resistors, SOT-323 FETs and one BAT54AW so the stage fits the power
  box; Power Good parts are placed last in gen_pcb.py.
- Board re-routed with Freerouting 2.5.0 and cleaned with fix_route.py: DRC
  0 unconnected, no copper violations. Gerbers, JLCPCB zip, renders, BOM, CPL
  and schematic PDF regenerated; datasheet rules 193/193.

Co-Authored-By: Claude Sonnet 5.5 <noreply@anthropic.com>
Parts:
- removed C72: 470nF, Capacitor_SMD:C_0805_2012Metric, symbol Device:C
- removed R65: 15m, Resistor_SMD:R_2512_6332Metric, symbol Device:R_US
- removed R66: 49.9, Resistor_SMD:R_0603_1608Metric, symbol Device:R_US
- removed R68: 10k, Resistor_SMD:R_0603_1608Metric, symbol Device:R_US
- added C74: 1uF, Capacitor_SMD:C_0805_2012Metric, symbol Device:C
- added D7: ALERT (red), LED_SMD:LED_0603_1608Metric, symbol Device:LED
- added D8: PWR (green), LED_SMD:LED_0603_1608Metric, symbol Device:LED
- added R71: 470, Resistor_SMD:R_0603_1608Metric, symbol Device:R_US
- C72: renamed from R71; value 470 -> 470nF; footprint Resistor_SMD:R_0603_1608Metric -> Capacitor_SMD:C_0805_2012Metric; symbol Device:R_US -> Device:C
- R65: renamed from D7; value ALERT (red) -> 15m; footprint LED_SMD:LED_0603_1608Metric -> Resistor_SMD:R_2512_6332Metric; symbol Device:LED -> Device:R_US
- R66: renamed from C74; value 1uF -> 49.9; footprint Capacitor_SMD:C_0805_2012Metric -> Resistor_SMD:R_0603_1608Metric; symbol Device:C -> Device:R_US
- R68: renamed from D8; value PWR (green) -> 10k; footprint LED_SMD:LED_0603_1608Metric -> Resistor_SMD:R_0603_1608Metric; symbol Device:LED -> Device:R_US
Connections:
- net +12V: now also R65.2, R66.1
- net +3V3: now also R68.1, C74.1, R71.1; no longer C72.1, R66.1
- net GND: now also C74.2, D8.1 (K); no longer R66.2, R68.1 (K)
- net INA239_CS: now also R68.2
- net VSW: now also R65.1
- net at R70.1: now also D7.2 (A); no longer R65.2 (A)
- net at U23.8 (VBUS), U23.9 (IN-): now also C72.1, R66.2
- net at R67.2, U23.10 (IN+): now also C72.2
- net at R69.1, U23.3 (~{ALERT}): now also D7.1 (K); no longer R65.1 (K)
- new net: D8.2 (A), R71.2
Other:
- moved on the sheet: R65, R68

Commit message: WIP: restructure PCB for the Phoenix UCS 125-87 housing
Work in progress, layout not finished: about 90 parts still do not fit
their sections and the board is not routed.

- Right-angle connectors: Phoenix MSTBA 2,5 / MC 1,5, JST XH side entry,
  Hirose DF13, Molex 505448-0871 (new footprint from the Molex drawing)
- Datasheet and product links on every symbol (tools/part_links.py)
- Test points so every IC has one on its own nets
- gen_pcb.py: 100 x 62 mm two-sided board, housing holes and restricted
  corners, ESP32 antenna notch, one section per sheet, board ID block,
  ESP32 pin names, pin-1 marks, blue mask
- Housing drawings in hardware/housing/

Co-Authored-By: Claude Opus 5.5 <noreply@anthropic.com>
Parts:
- removed C71: 100uF/25V, Capacitor_SMD:CP_Elec_8x10, symbol Device:C_Polarized
- removed C72: 470nF, Capacitor_SMD:C_0805_2012Metric, symbol Device:C
- removed C73: 100nF, Capacitor_SMD:C_0603_1608Metric, symbol Device:C
- removed C74: 1uF, Capacitor_SMD:C_0805_2012Metric, symbol Device:C
- removed R66: 49.9, Resistor_SMD:R_0603_1608Metric, symbol Device:R_US
- added D8: PWR (green), LED_SMD:LED_0603_1608Metric, symbol Device:LED
- added R67: 49.9, Resistor_SMD:R_0603_1608Metric, symbol Device:R_US
- added R68: 10k, Resistor_SMD:R_0603_1608Metric, symbol Device:R_US
- added R70: 1k, Resistor_SMD:R_0603_1608Metric, symbol Device:R_US
- added R71: 470, Resistor_SMD:R_0603_1608Metric, symbol Device:R_US
- C70: Product (none) -> https://www.digikey.com/en/products/result?keywords=CL21B10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
- C71: renamed from R67; value 49.9 -> 100uF/25V; footprint Resistor_SMD:R_0603_1608Metric -> Capacitor_SMD:CP_Elec_8x10; symbol Device:R_US -> Device:C_Polarized; Product (none) -> https://www.digikey.com/en/products/result?keywords=EEE-FK1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
- C72: renamed from R69; value 10k -> 470nF; footprint Resistor_SMD:R_0603_1608Metric -> Capacitor_SMD:C_0805_2012Metric; symbol Device:R_US -> Device:C; Product (none) -> https://www.digikey.com/en/products/result?keywords=CL21B47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
- C73: renamed from R71; value 470 -> 100nF; footprint Resistor_SMD:R_0603_1608Metric -> Capacitor_SMD:C_0603_1608Metric; symbol Device:R_US -> Device:C; Product (none) -> https://www.digikey.com/en/products/result?keywords=C0603C1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
- C74: renamed from D8; value PWR (green) -> 1uF; footprint LED_SMD:LED_0603_1608Metric -> Capacitor_SMD:C_0805_2012Metric; symbol Device:LED -> Device:C; Product (none) -> https://www.digikey.com/en/products/result?keywords=08055C1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
- D7: Product (none) -> https://www.digikey.com/en/products/result?keywords=LTST-C1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
- R65: Product (none) -> https://www.digikey.com/en/products/result?keywords=WSL2512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
- R66: renamed from R68; value 10k -> 49.9; Product (none) -> https://www.digikey.com/en/products/result?keywords=RC0603F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
- R69: renamed from R70; value 1k -> 10k; Product (none) -> https://www.digikey.com/en/products/result?keywords=AR0603F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
- U23: Product (none) -> https://www.digikey.com/en/products/result?keywords=INA239A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
Connections:
- net +12V: now also C71.1, R66.1
- net +3V3: now also C74.1, R68.1, R70.2, R71.1; no longer C72.2, R66.1
- net GND: now also C71.2, C73.2, C74.2, D8.1 (K); no longer C74.1 (K)
- net INA239_CS: now also R68.2; no longer R66.2
- net VSW: now also R67.1; no longer C71.1
- net at D7.1 (K), U23.3 (~{ALERT}): now also R69.1; no longer C72.1
- net at D7.2 (A): now also R70.1; no longer R69.1
- net at U23.10 (IN+): now also C72.2, R67.2; no longer C71.2
- net at U23.8 (VBUS), U23.9 (IN-): now also C72.1, R66.2
- new net: D8.2 (A), R71.2
Other:
- moved on the sheet: C71, R66, R69

Commit message: Ground the M12 shield, order the ground loops, name the J14 cable parts
- J10: shielded symbol (Conn_01x04_Shielded); the M12 shield pin and its
  four shell legs are pad SH, tied to GND
- TP22-TP25: Keystone 5001 black miniature PC test points (KiCad
  TestPoint_Keystone_5000-5004 footprint, 1.02 mm hole per Keystone's
  drawing); now in the BOM, the bare pad test points stay out
- J14 BOM note: cable housing Molex 5054320801 with 505431 terminals, or
  tin pre-crimped leads 797581148 / 797581149 (from molex.com)

Only netlist change: GND gains J10 SH. DRC 0 errors, 0 unconnected, 0
schematic-parity issues; ERC 0; 193/193 datasheet rules.

Co-Authored-By: Claude Opus 5.5 <noreply@anthropic.com>
Parts:
- removed C73: 100nF, Capacitor_SMD:C_0603_1608Metric, symbol Device:C
- removed D7: ALERT (red), LED_SMD:LED_0603_1608Metric, symbol Device:LED
- removed R66: 49.9, Resistor_SMD:R_0603_1608Metric, symbol Device:R_US
- removed R71: 470, Resistor_SMD:R_0603_1608Metric, symbol Device:R_US
- removed U23: INA239AIDGSR, Package_SO:TSSOP-10_3x3mm_P0.5mm, symbol cryocooler:INA239AIDGSR
- added C74: 1uF, Capacitor_SMD:C_0805_2012Metric, symbol Device:C
- added D8: PWR (green), LED_SMD:LED_0603_1608Metric, symbol Device:LED
- added R65: 15m, Resistor_SMD:R_2512_6332Metric, symbol Device:R_US
- added R68: 10k, Resistor_SMD:R_0603_1608Metric, symbol Device:R_US
- added R70: 1k, Resistor_SMD:R_0603_1608Metric, symbol Device:R_US
- C72: renamed from R68; value 10k -> 470nF; footprint Resistor_SMD:R_0603_1608Metric -> Capacitor_SMD:C_0805_2012Metric; symbol Device:R_US -> Device:C; Product https://www.digikey.com/en/products/result?keywords=AR0603F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 -> https://www.digikey.com/en/products/result?keywords=CL21B47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
- C73: renamed from C74; value 1uF -> 100nF; footprint Capacitor_SMD:C_0805_2012Metric -> Capacitor_SMD:C_0603_1608Metric; Product https://www.digikey.com/en/products/result?keywords=08055C1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 -> https://www.digikey.com/en/products/result?keywords=C0603C1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
- D7: renamed from R70; value 1k -> ALERT (red); footprint Resistor_SMD:R_0603_1608Metric -> LED_SMD:LED_0603_1608Metric; symbol Device:R_US -> Device:LED; Product https://www.digikey.com/en/products/result?keywords=RC0603F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 -> https://www.digikey.com/en/products/result?keywords=LTST-C1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
- R67: renamed from C72; value 470nF -> 49.9; footprint Capacitor_SMD:C_0805_2012Metric -> Resistor_SMD:R_0603_1608Metric; symbol Device:C -> Device:R_US; Product https://www.digikey.com/en/products/result?keywords=CL21B47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 -> https://www.digikey.com/en/products/result?keywords=RC0603F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
- R71: renamed from D8; value PWR (green) -> 470; footprint LED_SMD:LED_0603_1608Metric -> Resistor_SMD:R_0603_1608Metric; symbol Device:LED -> Device:R_US; Product https://www.digikey.com/en/products/result?keywords=LTST-C1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 -> https://www.digikey.com/en/products/result?keywords=RC0603F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
- U23: renamed from R65; value 15m -> INA239AIDGSR; footprint Resistor_SMD:R_2512_6332Metric -> Package_SO:TSSOP-10_3x3mm_P0.5mm; symbol Device:R_US -> cryocooler:INA239AIDGSR; Product https://www.digikey.com/en/products/result?keywords=WSL2512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 -> https://www.digikey.com/en/products/result?keywords=INA239A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
- renumbered R67 to R66
Connections:
- net +12V: now also R66.1, R65.2; no longer U23.2
- net +3V3: now also R71.1, U23.6 (VS), C74.1, R68.1, R70.2; no longer C72.1, D7.2
- net GND: now also U23.7 (GND), C74.2, D8.1 (K); no longer R71.1 (K)
- net INA239_CS: now also U23.1 (~{CS}), R68.2; no longer C72.2
- net SPI_MISO: now also U23.4 (SDO)
- net SPI_MOSI: now also U23.2 (SDI)
- net SPI_SCK: now also U23.5 (SCLK)
- net VSW: now also R67.1, R65.1; no longer R66.1, U23.1
- net at D7.1 (K): now also R69.1, U23.3 (~{ALERT})
- net at R66.2: now also C72.1, U23.8 (VBUS), U23.9 (IN-); no longer R67.2
- net at R71.2: now also D8.2 (A)
- new net: D7.2 (A), R70.1
- new net: C72.2, R67.2, U23.10 (IN+)
Other:
- moved on the sheet: C73, D7, R66, R71
