File: hardware/kicad/sim/cryocooler_sim.kicad_sch (KiCad schematic)
At the start: 17 parts, among them U1 OPA1656ID, U2 AD633JRZ-R7, U3 OPA188ID

Commit message: Screenshots
Other:
- note added: ".param vdac=2.5"
- note removed: ".param vdac=1.25"
Changed lines of the file:
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@@
 		)
 	)
-	(text ".param vdac=1.25"
+	(text ".param vdac=2.5"
 		(exclude_from_sim no)
 		(at 20 36 0)
